File: simulation/power_supply_simulation.kicad_sch (KiCad schematic)
At the start: 12 parts, among them Q1 SSM6P69NU,LF, Q3 BC547

Commit message: some changes
Parts:
- U: renamed from V1; value PULSE(0 3.3 2 1m 1m 4 0) -> (none)
- U: renamed from Q3; value BC547 -> (none)
- U: renamed from R6; value 10k -> (none)
- U: renamed from Q1; value SSM6P69NU,LF -> (none); footprint footprints:SON65P200X200X80-8N -> (none)
- U: renamed from V3; value PULSE(0 3.3 4 1m 1m 1 0) -> (none)
- U: renamed from R2; value 0.06 -> (none)
- U: renamed from V4; value dc 3.3 -> (none)
- U: renamed from R4; value 1 -> (none)
- U: renamed from R3; value 0.05 -> (none)
- U: renamed from R1; value 2.4 -> (none)
- U: renamed from V2; value dc 5 -> (none)
- U: renamed from R5; value 2k -> (none)
