File: mainboard/mainboard/usb_connectors.kicad_sch (KiCad schematic)
At the start: 10 parts, among them U701 hs8836a

Commit message: some fixes for ERC
Connections:
- net +5V_USB_HUB: now also C703.1, C704.1, U701.13 (VCC); no longer F701.2
- new net: F701.2, R702.1
Changed lines of the file:
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@@
   (junction (at 60.96 44.45) (diameter 0) (color 0 0 0 0)
   )
+  (junction (at 242.57 96.52) (diameter 0) (color 0 0 0 0)
+  )
   (junction (at 60.96 106.68) (diameter 0) (color 0 0 0 0)
   )
@@
   )
   (junction (at 208.28 81.28) (diameter 0) (color 0 0 0 0)
-  )
-  (junction (at 242.57 96.52) (diameter 0) (color 0 0 0 0)
   )
   (no_connect (at 198.12 96.52))
@@
     (stroke (width 0) (type default))
   )
+  (wire (pts (xy 207.01 54.61) (xy 213.36 54.61))
+    (stroke (width 0) (type default))
+  )
   (wire (pts (xy 198.12 109.22) (xy 208.28 109.22))
     (stroke (width 0) (type default))
@@
     (stroke (width 0) (type default))
   )
+  (wire (pts (xy 210.82 96.52) (xy 231.14 96.52))
+    (stroke (width 0) (type default))
+  )
   (wire (pts (xy 60.96 48.26) (xy 60.96 44.45))
     (stroke (width 0) (type default))
@@
     (stroke (width 0) (type default))
   )
-  (wire (pts (xy 214.63 54.61) (xy 214.63 49.53))
+  (wire (pts (xy 228.6 54.61) (xy 228.6 49.53))
     (stroke (width 0) (type default))
   )
@@
     (stroke (width 0) (type default))
   )
-  (wire (pts (xy 231.14 96.52) (xy 210.82 96.52))
-    (stroke (width 0) (type default))
-  )
   (wire (pts (xy 60.96 119.38) (xy 66.04 119.38))
     (stroke (width 0) (type default))
@@
     (stroke (width 0) (type default))
   )
+  (wire (pts (xy 220.98 54.61) (xy 228.6 54.61))
+    (stroke (width 0) (type default))
+  )
   (wire (pts (xy 60.96 116.84) (xy 66.04 116.84))
     (stroke (width 0) (type default))
@@
     (stroke (width 0) (type default))
   )
-  (wire (pts (xy 207.01 54.61) (xy 214.63 54.61))
-    (stroke (width 0) (type default))
-  )
   (wire (pts (xy 203.2 81.28) (xy 208.28 81.28))
     (stroke (width 0) (type default))
@@
     (stroke (width 0) (type default))
   )
-  (wire (pts (xy 242.57 87.63) (xy 242.57 88.9))
+  (wire (pts (xy 242.57 87.63) (xy 242.57 96.52))
     (stroke (width 0) (type default))
   )
@@
     )
   )
-  (symbol (lib_id "project_power:+5V_USB_HUB") (at 214.63 49.53 0) (unit 1)
-    (in_bom yes) (on_board yes) (dnp no) (fields_autoplaced)
-    (property "Reference" "#PWR0709" (at 214.63 53.34 0)
-      (effects (font (size 1.27 1.27)) hide)
-    )
-    (property "Value" "+5V_USB_HUB" (at 214.63 44.45 0)
-      (effects (font (size 1.27 1.27)))
-    )
-    (property "Footprint" "" (at 214.63 49.53 0)
-      (effects (font (size 1.27 1.27)) hide)
-    )
-    (property "Datasheet" "" (at 214.63 49.53 0)
+  (symbol (lib_id "project_power:+5V_USB_HUB") (at 228.6 49.53 0) (unit 1)
+    (in_bom yes) (on_board yes) (dnp no) (fields_autoplaced)
+    (property "Reference" "#PWR0709" (at 228.6 53.34 0)
+      (effects (font (size 1.27 1.27)) hide)
+    )
+    (property "Value" "+5V_USB_HUB" (at 228.6 44.45 0)
+      (effects (font (size 1.27 1.27)))
+    )
+    (property "Footprint" "" (at 228.6 49.53 0)
+      (effects (font (size 1.27 1.27)) hide)
+    )
+    (property "Datasheet" "" (at 228.6 49.53 0)
       (effects (font (size 1.27 1.27)) hide)
     )
@@
   (symbol (lib_id "project_power:+5V_USB_HUB") (at 242.57 87.63 0) (unit 1)
     (in_bom yes) (on_board yes) (dnp no)
-    (property "Reference" "#PWR0155" (at 248.92 90.17 0)
+    (property "Reference" "#PWR0157" (at 248.92 90.17 0)
       (effects (font (size 1.27 1.27)) hide)
     )
@@
       (project "mainboard"
         (path "/e63e39d7-6ac0-4ffd-8aa3-1841a4541b55/b04c7282-7715-4444-b680-e16531d85cc8"
-          (reference "#PWR0155") (unit 1) (value "+5V_USB_HUB") (footprint "")
+          (reference "#PWR0157") (unit 1) (value "+5V_USB_HUB") (footprint "")
         )
       )
@@
     )
   )
+  (symbol (lib_id "Device:R") (at 217.17 54.61 90) (unit 1)
+    (in_bom yes) (on_board yes) (dnp no)
+    (property "Reference" "R702" (at 217.17 49.53 90)
+      (effects (font (size 1.27 1.27)))
+    )
+    (property "Value" "4.7" (at 217.17 52.07 90)
+      (effects (font (size 1.27 1.27)))
+    )
+    (property "Footprint" "Resistor_SMD:R_0603_1608Metric_Pad0.98x0.95mm_HandSolder" (at 217.17 56.388 90)
+      (effects (font (size 1.27 1.27)) hide)
+    )
+    (property "Datasheet" "~" (at 217.17 54.61 0)
+      (effects (font (size 1.27 1.27)) hide)
+    )
+    (pin "1")
+    (pin "2")
+    (instances
+      (project "mainboard"
+        (path "/e63e39d7-6ac0-4ffd-8aa3-1841a4541b55/b04c7282-7715-4444-b680-e16531d85cc8"
+          (reference "R702") (unit 1) (value "4.7") (footprint "Resistor_SMD:R_0603_1608Metric_Pad0.98x0.95mm_HandSolder")
+        )
+      )
+    )
+  )
   (symbol (lib_id "Connector:USB_A_Stacked") (at 50.8 116.84 0) (unit 1)
     (in_bom yes) (on_board yes) (dnp no) (fields_autoplaced)
@@
         )
       )
-    )
-  )
-  (symbol (lib_id "Device:R") (at 242.57 92.71 180) (unit 1)
-    (in_bom yes) (on_board yes) (dnp no)
-    (property "Reference" "R702" (at 237.49 92.71 90)
-      (effects (font (size 1.27 1.27)))
-    )
-    (property "Value" "4.7" (at 240.03 92.71 90)
-      (effects (font (size 1.27 1.27)))
-    )
-    (property "Footprint" "Resistor_SMD:R_0603_1608Metric_Pad0.98x0.95mm_HandSolder" (at 244.348 92.71 90)
-      (effects (font (size 1.27 1.27)) hide)
-    )
-    (property "Datasheet" "~" (at 242.57 92.71 0)
-      (effects (font (size 1.27 1.27)) hide)
-    )
-    (pin "1")
-    (pin "2")
-    (instances
-      (project "mainboard"
-        (path "/e63e39d7-6ac0-4ffd-8aa3-1841a4541b55/b04c7282-7715-4444-b680-e16531d85cc8"
-          (reference "R702") (unit 1) (value "4.7") (footprint "Resistor_SMD:R_0603_1608Metric_Pad0.98x0.95mm_HandSolder")
-        )
-      )

Commit message: gpu and motherboard passes tests, now time for fpga
Other:
- title: (none) -> MSPC
Changed lines of the file:
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@@
 (kicad_sch (version 20221004) (generator eeschema)
   (paper "A4")
+  (title_block
+    (title "MSPC")
+    (rev "1")
+  )
   (junction (at 60.96 48.26) (diameter 0) (color 0 0 0 0)
   )
