File: mainboard/mainboard/mainboard.kicad_pcb (KiCad board)
At the start: 4 copper layers, 99.2 x 94.1 mm, 172 parts, among them IC1 SN74HCS151PWR, IC2 SN74HCS151PWR, IC3 SN74HCS138PWR, IC4 SN74HCS138PWR, IC5 SN74HCS138PWR, J1 Barrel_Jack_Switch, J10 AudioJack4, J11 AudioJack4, J12 Conn_01x03_Female, J13 Connector 16-bit, J14 Connector A 8-bit, J15 Connector B 8-bit, J16 Connector A - 4 bit, J17 Connector B - 4 bit, J18 Connector A - 2 bit, J19 Connector B - 2 bit, J4 Micro_SD_Card, J5 I2C 2, J6 Conn_01x03_Female, J7 I2C 1, J8 I2C 3, J9 Conn_01x03_Female, U1 RP2040, U10 GD25D05CT, U11 W25Q128JVS, U2 LD1117S50TR_SOT223, U3 AP2210, U4 AP2210, U5 BD9D321EFJ, U6 BD9D321EFJ, U7 hs8836a, U8 RP2040, U9 TLV320DAC3203IRGET, Y1 ECS-120-8-36-CGN-TR, Y2 ECS-120-8-36-CGN-TR

Commit message: working on PCB
Parts:
- removed C203: 1u, Capacitor_SMD:C_0402_1005Metric_Pad0.74x0.62mm_HandSolder
- removed C205, C207, C77, C78: 100n, Capacitor_SMD:C_0402_1005Metric_Pad0.74x0.62mm_HandSolder
- removed the C45 at (70.0, 100.3)
- removed the C56 at (232.8, 103.5)
- removed the C66 at (236.0, 97.6)
- removed the C67 at (236.0, 99.6)
- removed the C68 at (236.0, 101.5)
- removed the C69 at (110.2, 97.4)
- removed the C72 at (249.1, 43.9)
- removed C74: 4.7u, Capacitor_SMD:C_0402_1005Metric_Pad0.74x0.62mm_HandSolder
- removed the D10 at (81.5, 131.1)
- removed the D10 at (28.2, 128.3)
- removed the D11 at (63.0, 123.4)
- removed the D2 at (59.1, 116.4)
- removed the D3 at (83.1, 131.1)
- removed the D4 at (59.1, 118.7)
- removed the D5 at (63.0, 116.4)
- removed the D6 at (24.3, 133.0)
- removed the D6 at (59.1, 121.1)
- removed the D7 at (63.0, 118.7)
- removed the D8 at (59.1, 123.4)
- removed the D8 at (28.2, 123.6)
- removed the D9 at (63.0, 121.1)
- removed IC2: SN74HCS151PWR, footprints:SOP65P640X120-16N
- removed IC3, IC4, IC5: SN74HCS138PWR, footprints:SOP65P640X120-16N
- removed J18: Connector A - 2 bit, Connector_PinHeader_1.27mm:PinHeader_2x05_P1.27mm_Vertical_SMD
- removed J19: Connector B - 2 bit, Connector_PinHeader_1.27mm:PinHeader_2x05_P1.27mm_Vertical_SMD
- removed the J7 at (273.7, 61.3)
- removed the R16 at (252.4, 43.9)
- removed S1, S2: PTS636_SM43J_SMTR_LFS, footprints:SW_PTS636_SM43J_SMTR_LFS
- removed the TP1 at (245.9, 88.2)
- added C44: 100n, Capacitor_SMD:C_0402_1005Metric_Pad0.74x0.62mm_HandSolder, F.Cu at (25.5, 105.4)
- added C46: 100n, Capacitor_SMD:C_0402_1005Metric_Pad0.74x0.62mm_HandSolder, F.Cu at (72.1, 101.1)
- added D10: LESD5D5.0CT1G, footprints:TVS_LESD5D5.0CT1G, F.Cu at (77.7, 137.5)
- added D6: LESD5D5.0CT1G, footprints:TVS_LESD5D5.0CT1G, F.Cu at (217.7, 137.9)
- added D8: LESD5D5.0CT1G, footprints:TVS_LESD5D5.0CT1G, F.Cu at (220.1, 137.9)
- added H1: MountingHole, MountingHole:MountingHole_2.2mm_M2_DIN965, F.Cu at (55.0, 130.0)
- added H2: MountingHole, MountingHole:MountingHole_2.2mm_M2_DIN965, F.Cu at (145.0, 130.0)
- added H3: MountingHole, MountingHole:MountingHole_2.2mm_M2_DIN965, F.Cu at (145.0, 55.0)
- added H4: MountingHole, MountingHole:MountingHole_2.2mm_M2_DIN965, F.Cu at (55.0, 55.0)
- added J1: Conn_01x02_Male, Connector_PinHeader_2.54mm:PinHeader_1x02_P2.54mm_Vertical, F.Cu at (59.6, 86.9)
- added R11: 0, Resistor_SMD:R_2512_6332Metric_Pad1.40x3.35mm_HandSolder, F.Cu at (135.9, 92.1)
- added R13: 0, Resistor_SMD:R_2512_6332Metric_Pad1.40x3.35mm_HandSolder, F.Cu at (140.5, 92.1)
- added R14: 0, Resistor_SMD:R_2512_6332Metric_Pad1.40x3.35mm_HandSolder, F.Cu at (128.4, 94.5)
- added R18: 4.7k, Resistor_SMD:R_0603_1608Metric_Pad0.98x0.95mm_HandSolder, F.Cu at (88.6, 101.1)
- added R2: 0, Resistor_SMD:R_1206_3216Metric_Pad1.30x1.75mm_HandSolder, F.Cu at (100.6, 102.0)
- added R21: 1k, Resistor_SMD:R_0402_1005Metric_Pad0.72x0.64mm_HandSolder, F.Cu at (59.4, 91.4)
- added R3: 0, Resistor_SMD:R_1206_3216Metric_Pad1.30x1.75mm_HandSolder, F.Cu at (94.8, 112.1)
- added R4: 0, Resistor_SMD:R_1206_3216Metric_Pad1.30x1.75mm_HandSolder, F.Cu at (113.5, 98.7)
- added TP2: TestPoint, TestPoint:TestPoint_Pad_D1.5mm, F.Cu at (200.8, 91.7)
- added TP3: TestPoint, TestPoint:TestPoint_Pad_D1.5mm, F.Cu at (200.8, 88.2)
- added U10: SN74LVC139APWR, Package_SO:TSSOP-16_4.4x5mm_P0.65mm, F.Cu at (94.7, 81.4)
- added U13: SN74LVC139APWR, Package_SO:TSSOP-16_4.4x5mm_P0.65mm, F.Cu at (75.7, 81.5)
- C57, C58: value 1u -> 100n
- C60: value 1u -> 10u; footprint Capacitor_SMD:C_0402_1005Metric_Pad0.74x0.62mm_HandSolder -> Capacitor_SMD:C_1206_3216Metric_Pad1.33x1.80mm_HandSolder
- C63: value 100n -> 1u
- C64: value 22u -> 47u; footprint Capacitor_SMD:C_0402_1005Metric_Pad0.74x0.62mm_HandSolder -> Capacitor_SMD:C_1206_3216Metric_Pad1.33x1.80mm_HandSolder
- C65: value 100n -> 47u; footprint Capacitor_SMD:C_0402_1005Metric_Pad0.74x0.62mm_HandSolder -> Capacitor_SMD:C_1206_3216Metric_Pad1.33x1.80mm_HandSolder
- C68: renamed from C72; moved to B.Cu
- IC1: footprint footprints:SOP65P640X120-16N -> Package_SO:TSSOP-16_4.4x5mm_P0.65mm
- J13: value Connector 16-bit -> Connector A 16-bit
- J5: value I2C 2 -> Conn_01x02_Male; footprint Connector_PinHeader_2.54mm:PinHeader_2x03_P2.54mm_Vertical -> Connector_PinHeader_2.54mm:PinHeader_1x02_P2.54mm_Vertical
- J6: renamed from J4; moved to B.Cu
- J8: value I2C 3 -> Conn_01x04_Female; footprint Connector_PinHeader_2.54mm:PinHeader_2x03_P2.54mm_Vertical -> Connector_PinHeader_2.54mm:PinHeader_1x04_P2.54mm_Vertical
- R12: value 1k -> 0; footprint Resistor_SMD:R_0402_1005Metric_Pad0.72x0.64mm_HandSolder -> Resistor_SMD:R_2512_6332Metric_Pad1.40x3.35mm_HandSolder
- R17: value 4.7 -> 4.7k; footprint Resistor_SMD:R_0402_1005Metric_Pad0.72x0.64mm_HandSolder -> Resistor_SMD:R_0603_1608Metric_Pad0.98x0.95mm_HandSolder
- R22: renamed from R13; moved to B.Cu
- R23: renamed from R14; moved to B.Cu
- TP4: renamed from TP3; footprint TestPoint:TestPoint_Pad_D1.0mm -> TestPoint:TestPoint_THTPad_D1.5mm_Drill0.7mm
- TP5: renamed from TP4; footprint TestPoint:TestPoint_Pad_D1.0mm -> TestPoint:TestPoint_THTPad_D1.5mm_Drill0.7mm
- moved R23 301.2 mm to (16.2, 142.2), turned to 180 degrees
- moved R22 297.4 mm to (15.1, 119.3)
- moved C68 284.5 mm to (28.7, 125.1)
- moved D11 268.6 mm to (30.6, 112.1), turned to -90 degrees
- moved J8 233.6 mm to (54.2, 118.1), turned to 180 degrees
- moved TP1 226.3 mm to (40.8, 138.3)
- moved J5 211.5 mm to (57.0, 91.1)
- moved TP4 210.5 mm to (43.6, 129.9)
- moved J6 190.4 mm to (17.5, 129.8), turned to -90 degrees
- moved R12 176.0 mm to (123.8, 94.5), turned to -90 degrees
- moved C73 176.0 mm to (78.0, 86.7), turned to -90 degrees
- moved R17 170.0 mm to (91.7, 101.3), turned to -90 degrees
- moved C20 156.2 mm to (101.6, 98.4), turned to 90 degrees
- moved C19 156.1 mm to (101.6, 96.0), turned to 90 degrees
- moved C17 155.6 mm to (99.6, 114.9)
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- renumbered C22 to C20, C20 to C21, C21 to C22, C44 to C45, C46 to C47, C47 to C48, C48 to C49, C49 to C50, C50 to C51, C51 to C52, C52 to C53, C53 to C54, C54 to C55, C55 to C56, C70 to C66, C71 to C67, C73 to C69, C74 to C70, C75 to C71, C76 to C72, J16 to J15, J17 to J16, J15 to J17, J1 to J2, J2 to J3, J3 to J4, J6 to J7, R7 to R10, R8 to R15, R9 to R16, R10 to R19, R11 to R20, R15 to R24, R16 to R25, R17 to R26, R18 to R27, R2 to R5, R3 to R6, R4 to R7, R5 to R8, R6 to R9, TP2 to TP1, TP5 to TP6, TP6 to TP7, U10 to U11, U11 to U12
Connections:
- C20 pad 1: +3V3_MCU -> Net-(U4-VOUT)
- C21 pad 1: +5V_VBUS -> Net-(U2-VO)
- C22 pad 1: +3V3_SOUTH -> Net-(U3-VOUT)
- C35 pad 1: +5V_BUS -> Net-(C35-Pad1)
- C36 pad 1: +3V3_BUS -> Net-(C36-Pad1)
- C37 pad 1: +5V_BUS -> Net-(C35-Pad1)
- C38 pad 1: +3V3_BUS -> Net-(C36-Pad1)
- C39 pad 1: +5V_BUS -> Net-(C35-Pad1)
- C40 pad 1: +3V3_BUS -> Net-(C36-Pad1)
- C41 pad 1: +3V3_SOUTH -> +3V3_USB_HUB
- C42 pad 1: +3V3_SOUTH -> +3V3_USB_HUB
- C57 pad 1: Net-(U9-AVDD) -> /South Bridge/Audio DAC/AUX_IN.L
- C57 pad 2: GND -> Net-(U9-INL)
- C59 pad 1: +3V3_SOUTH -> Net-(U9-AVDD)
- C60 pad 1: Net-(U9-AVDD) -> +3V3_SOUTH
- C61 pad 1: +3V3_SOUTH -> Net-(U9-AVDD)
- C62 pad 1: Net-(U9-AVDD) -> +3V3_SOUTH
- C63 pad 1: Net-(U9-AVDD) -> Net-(U9-REF)
- C64 pad 1: +3V3_SOUTH -> Net-(U9-HPR)
- C64 pad 2: GND -> /South Bridge/Audio DAC/AUDIO_OUT.R
- C65 pad 1: +3V3_SOUTH -> Net-(U9-HPL)
- C65 pad 2: GND -> /South Bridge/Audio DAC/AUDIO_OUT.L
- C66 pad 1: +3V3_MCU -> +3V3_SOUTH
- C67 pad 1: +3V3_MCU -> +3V3_SOUTH
- IC1 pad 1: /RP2040 Core/BUS_DET.IN1 -> /RP2040 Core/BUS_DET.IN2
- IC1 pad 12: /RP2040 Core/BUS_DET.IN3 -> /RP2040 Core/BUS_DET.IN4
- IC1 pad 13: /RP2040 Core/BUS_INT.IN3 -> /RP2040 Core/BUS_INT.IN2
- IC1 pad 14: /RP2040 Core/BUS_DET.IN2 -> /RP2040 Core/BUS_INT.IN1
- IC1 pad 15: /RP2040 Core/BUS_INT.IN2 -> /RP2040 Core/BUS_DET.IN3
- IC1 pad 16: +3V3_MCU -> +3V3_SOUTH
- IC1 pad 2: /RP2040 Core/BUS_INT.IN1 -> /RP2040 Core/BUS_DET.IN1
- IC1 pad 5: /South Bridge/BUS_INT.OUT -> /South Bridge/BUS_DET_OUT
- J13 pad 1: +5V_BUS -> GND
- J13 pad 10: /RP2040 Core/MCU Connectors/BUS_NORTH.D13 -> /RP2040 Core/MCU Connectors/BUS_NORTH.D8
- J13 pad 11: /RP2040 Core/MCU Connectors/BUS_NORTH.D12 -> /RP2040 Core/MCU Connectors/BUS_NORTH.D7
- J13 pad 12: /RP2040 Core/MCU Connectors/BUS_NORTH.D11 -> /RP2040 Core/MCU Connectors/BUS_NORTH.D6
- J13 pad 13: /RP2040 Core/MCU Connectors/BUS_NORTH.D10 -> /RP2040 Core/MCU Connectors/BUS_NORTH.D5
- J13 pad 14: /RP2040 Core/MCU Connectors/BUS_NORTH.D9 -> /RP2040 Core/MCU Connectors/BUS_NORTH.D4
- J13 pad 15: /RP2040 Core/MCU Connectors/BUS_NORTH.D8 -> /RP2040 Core/MCU Connectors/BUS_NORTH.D3
- J13 pad 16: /RP2040 Core/MCU Connectors/BUS_NORTH.D7 -> /RP2040 Core/MCU Connectors/BUS_NORTH.D2
- J13 pad 17: /RP2040 Core/MCU Connectors/BUS_NORTH.D6 -> /RP2040 Core/MCU Connectors/BUS_NORTH.D1
- J13 pad 18: /RP2040 Core/MCU Connectors/BUS_NORTH.D5 -> /RP2040 Core/MCU Connectors/BUS_NORTH.D0
- J13 pad 19: /RP2040 Core/MCU Connectors/BUS_NORTH.D4 -> /RP2040 Core/MCU Connectors/BUS_NORTH.RWDS
- J13 pad 2: +5V_BUS -> GND
- J13 pad 20: /RP2040 Core/MCU Connectors/BUS_NORTH.D3 -> /RP2040 Core/MCU Connectors/BUS_NORTH.CLK1
- J13 pad 21: /RP2040 Core/MCU Connectors/BUS_NORTH.D2 -> /RP2040 Core/MCU Connectors/BUS_CS#A0
- J13 pad 22: /RP2040 Core/MCU Connectors/BUS_NORTH.D1 -> /RP2040 Core/MCU Connectors/BUS_CS#A1
- J13 pad 23: /RP2040 Core/MCU Connectors/BUS_NORTH.D0 -> /RP2040 Core/BUS_DET.IN0
- J13 pad 24: /RP2040 Core/MCU Connectors/BUS_NORTH.CLK1 -> /RP2040 Core/BUS_RE#.OUT0
- J13 pad 25: /RP2040 Core/MCU Connectors/BUS_CS#A0 -> /RP2040 Core/BUS_INT.IN0
- J13 pad 26: /RP2040 Core/MCU Connectors/BUS_CS#A1 -> +5V_BUS
- J13 pad 27: /RP2040 Core/BUS_RE#.OUT0 -> +3V3_BUS
- J13 pad 28: /RP2040 Core/BUS_DET.IN0 -> GND
- J13 pad 29: /RP2040 Core/BUS_INT.IN0 -> GND
- J13 pad 3: +3V3_BUS -> /RP2040 Core/MCU Connectors/BUS_NORTH.D15
- J13 pad 4: +3V3_BUS -> /RP2040 Core/MCU Connectors/BUS_NORTH.D14
- J13 pad 5: GND -> /RP2040 Core/MCU Connectors/BUS_NORTH.D13
- J13 pad 6: GND -> /RP2040 Core/MCU Connectors/BUS_NORTH.D12
- J13 pad 7: /RP2040 Core/MCU Connectors/BUS_NORTH.RWDS -> /RP2040 Core/MCU Connectors/BUS_NORTH.D11
- J13 pad 8: /RP2040 Core/MCU Connectors/BUS_NORTH.D15 -> /RP2040 Core/MCU Connectors/BUS_NORTH.D10
- J13 pad 9: /RP2040 Core/MCU Connectors/BUS_NORTH.D14 -> /RP2040 Core/MCU Connectors/BUS_NORTH.D9
- J14 pad 1: +3V3_BUS -> /RP2040 Core/MCU Connectors/BUS_NORTH.D15
- J14 pad 10: /RP2040 Core/MCU Connectors/BUS_NORTH.D3 -> /RP2040 Core/MCU Connectors/BUS_NORTH.CLK1
- J14 pad 11: /RP2040 Core/MCU Connectors/BUS_NORTH.D2 -> /RP2040 Core/MCU Connectors/BUS_CS#A2
- J14 pad 12: /RP2040 Core/MCU Connectors/BUS_NORTH.D1 -> unconnected-(J14-Pin_12)
- J14 pad 13: /RP2040 Core/MCU Connectors/BUS_NORTH.D0 -> /RP2040 Core/BUS_DET.IN1
- J14 pad 14: /RP2040 Core/MCU Connectors/BUS_NORTH.CLK1 -> /RP2040 Core/BUS_RE#.OUT1
- J14 pad 15: /RP2040 Core/MCU Connectors/BUS_CS#A2 -> unconnected-(J14-Pin_15)
- J14 pad 16: /RP2040 Core/MCU Connectors/BUS_CS#A3 -> +5V_BUS
- J14 pad 17: /RP2040 Core/BUS_RE#.OUT4 -> +3V3_BUS
- J14 pad 18: /RP2040 Core/BUS_DET.IN4 -> GND
- J14 pad 19: /RP2040 Core/BUS_INT.IN4 -> GND
- J14 pad 2: +5V_BUS -> /RP2040 Core/MCU Connectors/BUS_NORTH.D14
- J14 pad 3: GND -> /RP2040 Core/MCU Connectors/BUS_NORTH.D13
- J14 pad 4: GND -> /RP2040 Core/MCU Connectors/BUS_NORTH.D12
- J14 pad 5: /RP2040 Core/MCU Connectors/BUS_NORTH.RWDS -> /RP2040 Core/MCU Connectors/BUS_NORTH.D11
- J14 pad 6: /RP2040 Core/MCU Connectors/BUS_NORTH.D7 -> /RP2040 Core/MCU Connectors/BUS_NORTH.D10
- J14 pad 7: /RP2040 Core/MCU Connectors/BUS_NORTH.D6 -> /RP2040 Core/MCU Connectors/BUS_NORTH.D9
- J14 pad 8: /RP2040 Core/MCU Connectors/BUS_NORTH.D5 -> /RP2040 Core/MCU Connectors/BUS_NORTH.D8
- J14 pad 9: /RP2040 Core/MCU Connectors/BUS_NORTH.D4 -> /RP2040 Core/MCU Connectors/BUS_NORTH.RWDS
- J15 pad 1: +3V3_BUS -> /RP2040 Core/MCU Connectors/BUS_NORTH.D11
- J15 pad 10: /RP2040 Core/MCU Connectors/BUS_NORTH.CLK1 -> /RP2040 Core/BUS_RE#.OUT2
- J15 pad 11: /RP2040 Core/MCU Connectors/BUS_CS#A4 -> unconnected-(J15-Pin_11)
- J15 pad 12: /RP2040 Core/MCU Connectors/BUS_CS#A5 -> +5V_BUS
- J15 pad 13: /RP2040 Core/BUS_RE#.OUT5 -> +3V3_BUS
- J15 pad 14: /RP2040 Core/BUS_DET.IN5 -> GND
- J15 pad 15: /RP2040 Core/BUS_INT.IN5 -> GND
- J15 pad 2: +5V_BUS -> /RP2040 Core/MCU Connectors/BUS_NORTH.D10
- J15 pad 3: GND -> /RP2040 Core/MCU Connectors/BUS_NORTH.D9
- J15 pad 4: GND -> /RP2040 Core/MCU Connectors/BUS_NORTH.D8
- J15 pad 6: /RP2040 Core/MCU Connectors/BUS_NORTH.D7 -> /RP2040 Core/MCU Connectors/BUS_NORTH.CLK1
- J15 pad 7: /RP2040 Core/MCU Connectors/BUS_NORTH.D6 -> /RP2040 Core/MCU Connectors/BUS_CS#A3
- J15 pad 8: /RP2040 Core/MCU Connectors/BUS_NORTH.D5 -> unconnected-(J15-Pin_8)
- J15 pad 9: /RP2040 Core/MCU Connectors/BUS_NORTH.D4 -> /RP2040 Core/BUS_DET.IN2
- J16 pad 1: +3V3_BUS -> /RP2040 Core/MCU Connectors/BUS_NORTH.D3
- J16 pad 10: /RP2040 Core/MCU Connectors/BUS_NORTH.CLK0 -> /RP2040 Core/BUS_RE#.OUT4
- J16 pad 11: /RP2040 Core/MCU Connectors/BUS_CS#B4 -> /RP2040 Core/BUS_INT.IN2
- J16 pad 12: /RP2040 Core/MCU Connectors/BUS_CS#B5 -> +5V_BUS
- J16 pad 13: /RP2040 Core/BUS_RE#.OUT2 -> +3V3_BUS
- J16 pad 14: /RP2040 Core/BUS_DET.IN2 -> GND
- J16 pad 15: /RP2040 Core/BUS_INT.IN2 -> GND
- J16 pad 2: +5V_BUS -> /RP2040 Core/MCU Connectors/BUS_NORTH.D2
- J16 pad 3: GND -> /RP2040 Core/MCU Connectors/BUS_NORTH.D1
- J16 pad 4: GND -> /RP2040 Core/MCU Connectors/BUS_NORTH.D0
- J16 pad 6: /RP2040 Core/MCU Connectors/BUS_NORTH.D15 -> /RP2040 Core/MCU Connectors/BUS_NORTH.CLK0
- J16 pad 7: /RP2040 Core/MCU Connectors/BUS_NORTH.D14 -> /RP2040 Core/MCU Connectors/BUS_CS#B2
- J16 pad 8: /RP2040 Core/MCU Connectors/BUS_NORTH.D13 -> /RP2040 Core/MCU Connectors/BUS_CS#B3
- J16 pad 9: /RP2040 Core/MCU Connectors/BUS_NORTH.D12 -> /RP2040 Core/BUS_DET.IN4
- J17 pad 1: +3V3_BUS -> /RP2040 Core/MCU Connectors/BUS_NORTH.D7
- J17 pad 10: /RP2040 Core/MCU Connectors/BUS_NORTH.D11 -> /RP2040 Core/MCU Connectors/BUS_NORTH.CLK0
- J17 pad 11: /RP2040 Core/MCU Connectors/BUS_NORTH.D10 -> /RP2040 Core/MCU Connectors/BUS_CS#B0
- J17 pad 12: /RP2040 Core/MCU Connectors/BUS_NORTH.D9 -> /RP2040 Core/MCU Connectors/BUS_CS#B1
- J17 pad 13: /RP2040 Core/MCU Connectors/BUS_NORTH.D8 -> /RP2040 Core/BUS_DET.IN3
- J17 pad 14: /RP2040 Core/MCU Connectors/BUS_NORTH.CLK0 -> /RP2040 Core/BUS_RE#.OUT3
- J17 pad 15: /RP2040 Core/MCU Connectors/BUS_CS#B2 -> /RP2040 Core/BUS_INT.IN1
- J17 pad 16: /RP2040 Core/MCU Connectors/BUS_CS#B3 -> +5V_BUS
- J17 pad 17: /RP2040 Core/BUS_RE#.OUT1 -> +3V3_BUS
- J17 pad 18: /RP2040 Core/BUS_DET.IN1 -> GND
- J17 pad 19: /RP2040 Core/BUS_INT.IN1 -> GND
- J17 pad 2: +5V_BUS -> /RP2040 Core/MCU Connectors/BUS_NORTH.D6
- J17 pad 3: GND -> /RP2040 Core/MCU Connectors/BUS_NORTH.D5
- J17 pad 4: GND -> /RP2040 Core/MCU Connectors/BUS_NORTH.D4
- J17 pad 5: /RP2040 Core/MCU Connectors/BUS_NORTH.RWDS -> /RP2040 Core/MCU Connectors/BUS_NORTH.D3
- J17 pad 6: /RP2040 Core/MCU Connectors/BUS_NORTH.D15 -> /RP2040 Core/MCU Connectors/BUS_NORTH.D2
- J17 pad 7: /RP2040 Core/MCU Connectors/BUS_NORTH.D14 -> /RP2040 Core/MCU Connectors/BUS_NORTH.D1
- J17 pad 8: /RP2040 Core/MCU Connectors/BUS_NORTH.D13 -> /RP2040 Core/MCU Connectors/BUS_NORTH.D0
- J17 pad 9: /RP2040 Core/MCU Connectors/BUS_NORTH.D12 -> /RP2040 Core/MCU Connectors/BUS_NORTH.RWDS
- J5 pad 1: +3V3_BUS -> Net-(J5-Pin_1)
- J5 pad 2: unconnected-(J5-Pin_2) -> /South Bridge/POWER_BUTTON
- J8 pad 2: unconnected-(J8-Pin_2) -> GND
- J8 pad 3: /South Bridge/Audio DAC/I2C.SCL -> /South Bridge/Audio DAC/I2C.SDA
- J8 pad 4: /South Bridge/Audio DAC/I2C.SDA -> /South Bridge/Audio DAC/I2C.SCL
- L1 pad 2: +5V_BUS -> Net-(C35-Pad1)
- L2 pad 2: +3V3_BUS -> Net-(C36-Pad1)
- R12 pad 1: Net-(R12-Pad1) -> +3V3_BUS
- R12 pad 2: +3V3_SOUTH -> Net-(C36-Pad1)
- R17 pad 1: Net-(U10-VCC) -> /South Bridge/Audio DAC/I2C.SCL
- R17 pad 2: +5V_VBUS -> +3V3_SOUTH
- R5 pad 1: +5V_BUS -> Net-(C35-Pad1)
- R8 pad 1: +3V3_BUS -> Net-(C36-Pad1)
- TP1 pad 1: +5V_VBUS -> Net-(U2-VO)
- TP6 pad 1: +5V_BUS -> Net-(C35-Pad1)
- TP7 pad 1: +3V3_BUS -> Net-(C36-Pad1)
- U1 pad 11: /RP2040 Core/MCU Connectors/BUS_NORTH.D6 -> /RP2040 Core/MCU Connectors/BUS_NORTH.D5
- U1 pad 12: /RP2040 Core/MCU Connectors/BUS_NORTH.D7 -> /RP2040 Core/MCU Connectors/BUS_NORTH.D6
- U1 pad 13: /RP2040 Core/MCU Connectors/BUS_NORTH.D8 -> /RP2040 Core/MCU Connectors/BUS_NORTH.D7
- U1 pad 14: /RP2040 Core/MCU Connectors/BUS_NORTH.D9 -> /RP2040 Core/MCU Connectors/BUS_NORTH.D8
- U1 pad 15: /RP2040 Core/MCU Connectors/BUS_NORTH.D10 -> /RP2040 Core/MCU Connectors/BUS_NORTH.D9
- U1 pad 16: /RP2040 Core/MCU Connectors/BUS_NORTH.D11 -> /RP2040 Core/MCU Connectors/BUS_NORTH.D10
- U1 pad 17: /RP2040 Core/MCU Connectors/BUS_NORTH.D12 -> /RP2040 Core/MCU Connectors/BUS_NORTH.D11
- U1 pad 18: /RP2040 Core/MCU Connectors/BUS_NORTH.D13 -> /RP2040 Core/MCU Connectors/BUS_NORTH.D12
- U1 pad 27: /RP2040 Core/MCU Connectors/BUS_NORTH.D14 -> /RP2040 Core/MCU Connectors/BUS_NORTH.D13
- U1 pad 28: /RP2040 Core/MCU Connectors/BUS_NORTH.D15 -> /RP2040 Core/MCU Connectors/BUS_NORTH.D14
- U1 pad 29: /RP2040 Core/MCU Connectors/BUS_NORTH.RWDS -> /RP2040 Core/MCU Connectors/BUS_NORTH.D15
- U1 pad 30: unconnected-(U1-GPIO19) -> /RP2040 Core/BUS_SOUTH.D0
- U1 pad 31: /RP2040 Core/BUS_SOUTH.CLK -> /RP2040 Core/BUS_SOUTH.D1
- U1 pad 32: /RP2040 Core/BUS_SOUTH.D0 -> /RP2040 Core/BUS_SOUTH.D2
- U1 pad 34: /RP2040 Core/BUS_SOUTH.D1 -> /RP2040 Core/BUS_SOUTH.D3
- U1 pad 35: /RP2040 Core/BUS_SOUTH.D2 -> /RP2040 Core/BUS_SOUTH.CLK
- U1 pad 36: /RP2040 Core/BUS_SOUTH.D3 -> /RP2040 Core/North Bridge BUS multiplexer/BUS_CTRL.CS#3
- U1 pad 37: /RP2040 Core/North Bridge BUS multiplexer/BUS_CTRL.CS#B_EN -> /RP2040 Core/North Bridge BUS multiplexer/BUS_CTRL.CS#2
- U1 pad 38: /RP2040 Core/North Bridge BUS multiplexer/BUS_CTRL.CS#2 -> /RP2040 Core/North Bridge BUS multiplexer/BUS_CTRL.CS#B_EN
- U1 pad 39: /RP2040 Core/North Bridge BUS multiplexer/BUS_CTRL.CS#1 -> /RP2040 Core/North Bridge BUS multiplexer/BUS_CTRL.CS#A_EN
- U1 pad 4: /RP2040 Core/MCU Connectors/BUS_NORTH.D0 -> /RP2040 Core/MCU Connectors/BUS_NORTH.RWDS
- U1 pad 41: /RP2040 Core/North Bridge BUS multiplexer/BUS_CTRL.CS#A_EN -> /RP2040 Core/North Bridge BUS multiplexer/BUS_CTRL.CS#1
- U1 pad 5: /RP2040 Core/MCU Connectors/BUS_NORTH.D1 -> /RP2040 Core/MCU Connectors/BUS_NORTH.D0
- U1 pad 6: /RP2040 Core/MCU Connectors/BUS_NORTH.D2 -> /RP2040 Core/MCU Connectors/BUS_NORTH.D1
- U1 pad 7: /RP2040 Core/MCU Connectors/BUS_NORTH.D3 -> /RP2040 Core/MCU Connectors/BUS_NORTH.D2
- U1 pad 8: /RP2040 Core/MCU Connectors/BUS_NORTH.D4 -> /RP2040 Core/MCU Connectors/BUS_NORTH.D3
- U1 pad 9: /RP2040 Core/MCU Connectors/BUS_NORTH.D5 -> /RP2040 Core/MCU Connectors/BUS_NORTH.D4
- U2 pad 2: +5V_VBUS -> Net-(U2-VO)
- U3 pad 5: +3V3_SOUTH -> Net-(U3-VOUT)
- U4 pad 5: +3V3_MCU -> Net-(U4-VOUT)
- U7 pad 12: +3V3_MCU -> +3V3_USB_HUB
- U7 pad 14: +3V3_SOUTH -> +3V3_USB_HUB
- U8 pad 13: /South Bridge/SD Card/SDIO.CMD -> /South Bridge/Main bus control/BUS.CONTROL0
- U8 pad 14: /South Bridge/SD Card/SDIO.D0 -> /South Bridge/Main bus control/BUS.CONTROL1
- U8 pad 15: /South Bridge/SD Card/SDIO.D1 -> /South Bridge/Main bus control/BUS.CONTROL2
- U8 pad 16: /South Bridge/SD Card/SDIO.D2 -> /South Bridge/BUS_RE#.IN
- U8 pad 17: /South Bridge/SD Card/SDIO.D3 -> /South Bridge/BUS_DET_OUT
- U8 pad 18: /South Bridge/POWER_BUTTON -> /power_supply/POWER_ENABLE
- U8 pad 27: /power_supply/POWER_ENABLE -> /South Bridge/POWER_BUTTON
- U8 pad 28: /South Bridge/POWER_LED_DATA -> /RP2040 Core/BUS_SOUTH.CLK
- U8 pad 29: /RP2040 Core/BUS_SOUTH.CLK -> /RP2040 Core/BUS_SOUTH.D0
- U8 pad 30: /RP2040 Core/BUS_SOUTH.D0 -> /RP2040 Core/BUS_SOUTH.D1
- U8 pad 31: /RP2040 Core/BUS_SOUTH.D1 -> /RP2040 Core/BUS_SOUTH.D2
- U8 pad 32: /RP2040 Core/BUS_SOUTH.D2 -> /RP2040 Core/BUS_SOUTH.D3
- U8 pad 34: /RP2040 Core/BUS_SOUTH.D3 -> /South Bridge/POWER_LED_DATA
- U8 pad 35: unconnected-(U8-GPIO23) -> /South Bridge/SD Card/SDIO.CLK
- U8 pad 36: /South Bridge/Main bus control/BUS.CONTROL0 -> /South Bridge/SD Card/SDIO.CMD
- U8 pad 37: /South Bridge/Main bus control/BUS.CONTROL1 -> /South Bridge/SD Card/SDIO.D0
- U8 pad 38: /South Bridge/Main bus control/BUS.CONTROL2 -> /South Bridge/SD Card/SDIO.D1
- U8 pad 39: /South Bridge/BUS_RE#.IN -> /South Bridge/SD Card/SDIO.D2
- U8 pad 4: unconnected-(U8-GPIO2) -> /South Bridge/Audio DAC/AUDIO.DOUT
- U8 pad 40: /South Bridge/BUS_DET.OUT -> /South Bridge/SD Card/SDIO.D3
- U8 pad 41: /South Bridge/BUS_INT.OUT -> unconnected-(U8-GPIO29/ADC3)
- U8 pad 5: unconnected-(U8-GPIO3) -> /South Bridge/Audio DAC/AUDIO.DIN
- U8 pad 6: unconnected-(U8-GPIO4) -> /South Bridge/Audio DAC/AUDIO.WCLK
- U8 pad 7: unconnected-(U8-GPIO5) -> /South Bridge/Audio DAC/AUDIO.BCLK
- U8 pad 8: unconnected-(U8-GPIO6) -> /South Bridge/Audio DAC/AUDIO.MCLK
- U8 pad 9: /South Bridge/SD Card/SDIO.CLK -> /South Bridge/Audio DAC/AUDIO.RESET#
Routing:
- net +3V3_BUS: track 25.1 -> 218.3 mm, vias 10 -> 36
- net Net-(C35-Pad1): track 0.00 -> 75.4 mm
- net /RP2040 Core/MCU Connectors/BUS_CS#B6: track 67.9 -> 0.00 mm, vias 2 -> 0
- net /RP2040 Core/MCU Connectors/BUS_NORTH.D10: track 19.0 -> 86.7 mm
- net /RP2040 Core/MCU Connectors/BUS_NORTH.D8: track 19.0 -> 86.6 mm
- net /RP2040 Core/MCU Connectors/BUS_NORTH.D11: track 19.0 -> 86.6 mm
- net /RP2040 Core/MCU Connectors/BUS_NORTH.D9: track 19.0 -> 86.5 mm
- net /RP2040 Core/MCU Connectors/BUS_NORTH.D1: track 28.8 -> 94.0 mm
- net /RP2040 Core/MCU Connectors/BUS_NORTH.D0: track 28.9 -> 94.0 mm
- net /RP2040 Core/MCU Connectors/BUS_NORTH.D2: track 28.8 -> 93.9 mm
- net /RP2040 Core/MCU Connectors/BUS_NORTH.D3: track 28.8 -> 93.9 mm
- net /RP2040 Core/BUS_INT.IN3: track 61.5 -> 0.00 mm, vias 2 -> 0
- net /RP2040 Core/BUS_INT.IN2: track 0.00 -> 60.2 mm, vias 0 -> 2
- net Net-(C36-Pad1): track 0.00 -> 60.0 mm
- net /RP2040 Core/MCU Connectors/BUS_CS#A6: track 59.7 -> 0.00 mm
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- added copper zone on F.Cu, net +3V3_BUS
- added copper zone on F.Cu, net +3V3_MCU
- added copper zone on F.Cu, net +5V_BUS
- added copper zone on F.Cu, net GND
Other:
- board size 99.2 x 94.1 mm -> 100 x 100 mm
- board text added: "J2"
