File: mainboard/mainboard/audio_dac.kicad_sch (KiCad schematic)
At the start: 14 parts, among them U2 TLV320DAC3203IRGET

Commit message: working on new pcb
Parts:
- C204: footprint Capacitor_SMD:C_0603_1608Metric_Pad1.08x0.95mm_HandSolder -> Capacitor_SMD:C_0402_1005Metric_Pad0.74x0.62mm_HandSolder

Commit message: working on PCB
Parts:
- removed C204 (x4): 1u, Capacitor_SMD:C_0402_1005Metric_Pad0.74x0.62mm_HandSolder, symbol Device:C
- C204: value 1u -> 100n
- C204: value 1u -> 10u; footprint Capacitor_SMD:C_0402_1005Metric_Pad0.74x0.62mm_HandSolder -> Capacitor_SMD:C_1206_3216Metric_Pad1.33x1.80mm_HandSolder
- C204: value 1u -> 47u; footprint Capacitor_SMD:C_0402_1005Metric_Pad0.74x0.62mm_HandSolder -> Capacitor_SMD:C_1206_3216Metric_Pad1.33x1.80mm_HandSolder
Other:
- moved on the sheet: C204

Commit message: Mainboard rev 1.0a prepared
Parts:
- U2: footprint Package_DFN_QFN:VQFN-24-1EP_4x4mm_P0.5mm_EP2.45x2.45mm_ThermalVias -> Package_DFN_QFN:VQFN-24-1EP_4x4mm_P0.5mm_EP2.45x2.45mm
Changed lines of the file:
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@@
       (effects (font (size 1.27 1.27)))
     )
-    (property "Footprint" "Package_DFN_QFN:VQFN-24-1EP_4x4mm_P0.5mm_EP2.45x2.45mm_ThermalVias" (at 120.65 135.89 0)
+    (property "Footprint" "Package_DFN_QFN:VQFN-24-1EP_4x4mm_P0.5mm_EP2.45x2.45mm" (at 120.65 135.89 0)
       (effects (font (size 1.27 1.27)) hide)
     )
@@
     (pin "23")
     (pin "24")
+    (pin "25")
     (pin "3")
     (pin "4")

Commit message: prepared first versions of PCBs
Parts:
- renumbered C204 to C19, C204 to C20, C204 to C22, C204 to C57, C204 to C58, C204 to C59, C204 to C60, C204 to C61, C204 to C62, U2 to U4
Connections:
- net +3V3_SOUTH renamed +3V3_BUS
