File: mainboard/mainboard/main_bus_control.kicad_sch (KiCad schematic)
At the start: 6 parts, among them IC504 SN74HCS138PWR, IC505 SN74HCS151PWR

Commit message: working on new pcb
Parts:
- C504, C505: footprint Capacitor_SMD:C_0603_1608Metric_Pad1.08x0.95mm_HandSolder -> Capacitor_SMD:C_0402_1005Metric_Pad0.74x0.62mm_HandSolder
- IC504, IC505: footprint SOP65P640X120-16N -> footprints:SOP65P640X120-16N
Connections:
- net BUS_DET.IN0: now also IC505.3 (D1); no longer IC505.4 (D0)
- net BUS_DET.IN1: now also IC505.1 (D3); no longer IC505.3 (D1)
- net BUS_DET.IN2: now also IC505.14 (D5); no longer IC505.2 (D2)
- net BUS_DET.IN3: now also IC505.12 (D7); no longer IC505.1 (D3)
- net BUS_DET.IN4: now also IC505.2 (D2); no longer IC505.15 (D4)
- net BUS_DET.IN5: now also IC505.4 (D0); no longer IC505.14 (D5)
- net BUS_DET.IN6: now also IC505.14 (D5); no longer IC505.13 (D6)
- net BUS_INT.IN1: now also IC505.2 (D2); no longer IC505.3 (D1)
- net BUS_INT.IN2: now also IC505.15 (D4); no longer IC505.2 (D2)
- net BUS_INT.IN3: now also IC505.13 (D6); no longer IC505.1 (D3)
- net BUS_INT.IN4: now also IC505.1 (D3); no longer IC505.15 (D4)
- net BUS_INT.IN5: now also IC505.3 (D1); no longer IC505.14 (D5)
- net BUS_INT.IN6: now also IC505.15 (D4); no longer IC505.13 (D6)

Commit message: working on PCB
Parts:
- removed C505: 100n, Capacitor_SMD:C_0402_1005Metric_Pad0.74x0.62mm_HandSolder, symbol Device:C
- removed IC504: SN74HCS138PWR, footprints:SOP65P640X120-16N, symbol SN74HCS138PWR:SN74HCS138PWR
- removed IC505 (x2): SN74HCS151PWR, footprints:SOP65P640X120-16N, symbol SN74HCS151PWR:SN74HCS151PWR
- added IC1: SN74HCS151PWR, Package_SO:TSSOP-16_4.4x5mm_P0.65mm, symbol sn74:SN74HCS151PWR
- added U10: SN74LVC139APWR, Package_SO:TSSOP-16_4.4x5mm_P0.65mm, symbol sn74:SN74LVC139APWR
Connections:
- net BUS.CONTROL0: now also IC1.11 (A), U10.14 (2A)
- net BUS.CONTROL1: now also IC1.10 (B), U10.13 (2B)
- net BUS.CONTROL2: now also IC1.9 (C), U10.1 (1G#)
- net BUS_DET.IN0: now also IC1.3 (D1)
- net BUS_DET.IN1: now also IC1.2 (D2)
- net BUS_DET.IN2: now also IC1.1 (D3)
- net BUS_DET.IN3: now also IC1.15 (D4)
- net BUS_DET.IN4: now also IC1.12 (D7)
- net BUS_DET_OUT: now also IC1.5 (Y)
- net BUS_INT.IN0: now also IC1.4 (D0)
- net BUS_INT.IN1: now also IC1.14 (D5)
- net BUS_INT.IN2: now also IC1.13 (D6)
- net BUS_RE#.OUT0: now also U10.12 (2Y0)
- net BUS_RE#.OUT1: now also U10.11 (2Y1)
- net BUS_RE#.OUT2: now also U10.10 (2Y2)
- net BUS_RE#.OUT3: now also U10.9 (2Y3)
- net BUS_RE#.OUT4: now also U10.4 (1Y0)
- net BUS_RE#_IN: now also U10.15 (2G#)
- net GND: now also IC1.7 (~{G}), IC1.8 (GND), U10.2 (1A), U10.3 (1B), U10.8 (GND)
- net +3V3_MCU renamed +3V3_SOUTH
- net +3V3_SOUTH: now also IC1.16 (VCC), U10.16 (VCC)
- no-connect marks 5 -> 4
Other:
- moved on the sheet: C504

Commit message: Mainboard rev 1.0a prepared
Connections:
- net +3V3_SOUTH renamed +3V3_BUS
Changed lines of the file:
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@@
-    )
-  )
-  (symbol (lib_id "project_power:+3V3_SOUTH") (at 170.18 87.63 0) (unit 1)
-    (in_bom yes) (on_board yes) (dnp no) (fields_autoplaced)
-    (property "Reference" "#PWR0156" (at 170.18 91.44 0)
-      (effects (font (size 1.27 1.27)) hide)
-    )
-    (property "Value" "+3V3_SOUTH" (at 170.18 83.82 0)
-      (effects (font (size 1.27 1.27)))
-    )
-    (property "Footprint" "" (at 170.18 87.63 0)
-      (effects (font (size 1.27 1.27)) hide)
-    )
-    (property "Datasheet" "" (at 170.18 87.63 0)
-      (effects (font (size 1.27 1.27)) hide)
-    )
-    (pin "1")
-    (instances
-      (project "mainboard"
-        (path "/e63e39d7-6ac0-4ffd-8aa3-1841a4541b55/ee636c63-5fee-42d9-b500-aef9f04ef5c4"
-          (reference "#PWR0156") (unit 1)
-        )
-        (path "/e63e39d7-6ac0-4ffd-8aa3-1841a4541b55/ee636c63-5fee-42d9-b500-aef9f04ef5c4/e2a0288b-5594-4970-9369-10c890ff0b60"
-          (reference "#PWR0111") (unit 1)
-        )
-      )
-    )
-  )
-  (symbol (lib_id "project_power:+3V3_SOUTH") (at 95.25 85.09 0) (unit 1)
-    (in_bom yes) (on_board yes) (dnp no) (fields_autoplaced)
-    (property "Reference" "#PWR0156" (at 95.25 88.9 0)
-      (effects (font (size 1.27 1.27)) hide)
-    )
-    (property "Value" "+3V3_SOUTH" (at 95.25 81.28 0)
-      (effects (font (size 1.27 1.27)))
-    )
-    (property "Footprint" "" (at 95.25 85.09 0)
-      (effects (font (size 1.27 1.27)) hide)
-    )
-    (property "Datasheet" "" (at 95.25 85.09 0)
-      (effects (font (size 1.27 1.27)) hide)
-    )
-    (pin "1")
-    (instances
-      (project "mainboard"
-        (path "/e63e39d7-6ac0-4ffd-8aa3-1841a4541b55/ee636c63-5fee-42d9-b500-aef9f04ef5c4"
-          (reference "#PWR0156") (unit 1)
-        )
-        (path "/e63e39d7-6ac0-4ffd-8aa3-1841a4541b55/ee636c63-5fee-42d9-b500-aef9f04ef5c4/e2a0288b-5594-4970-9369-10c890ff0b60"
-          (reference "#PWR0109") (unit 1)
-        )
-      )
     )
   )
@@
         (path "/e63e39d7-6ac0-4ffd-8aa3-1841a4541b55/ee636c63-5fee-42d9-b500-aef9f04ef5c4/e2a0288b-5594-4970-9369-10c890ff0b60"
           (reference "U10") (unit 1)
+        )
+      )
+    )
+  )
+  (symbol (lib_id "project_power:+3V3_BUS") (at 95.25 85.09 0) (unit 1)
+    (in_bom yes) (on_board yes) (dnp no) (fields_autoplaced)
+    (property "Reference" "#PWR0109" (at 95.25 88.9 0)
+      (effects (font (size 1.27 1.27)) hide)
+    )
+    (property "Value" "+3V3_BUS" (at 95.25 81.28 0)
+      (effects (font (size 1.27 1.27)))
+    )
+    (property "Footprint" "" (at 95.25 85.09 0)
+      (effects (font (size 1.27 1.27)) hide)
+    )
+    (property "Datasheet" "" (at 95.25 85.09 0)
+      (effects (font (size 1.27 1.27)) hide)
+    )
+    (pin "1")
+    (instances
+      (project "mainboard"
+        (path "/e63e39d7-6ac0-4ffd-8aa3-1841a4541b55/ee636c63-5fee-42d9-b500-aef9f04ef5c4/e2a0288b-5594-4970-9369-10c890ff0b60"
+          (reference "#PWR0109") (unit 1)
         )
       )
@@
         )
       )
+    )
+  )
+  (symbol (lib_id "project_power:+3V3_BUS") (at 170.18 87.63 0) (unit 1)
+    (in_bom yes) (on_board yes) (dnp no) (fields_autoplaced)
+    (property "Reference" "#PWR0111" (at 170.18 91.44 0)
+      (effects (font (size 1.27 1.27)) hide)
+    )
+    (property "Value" "+3V3_BUS" (at 170.18 83.82 0)
+      (effects (font (size 1.27 1.27)))
+    )
+    (property "Footprint" "" (at 170.18 87.63 0)
+      (effects (font (size 1.27 1.27)) hide)
+    )
+    (property "Datasheet" "" (at 170.18 87.63 0)
+      (effects (font (size 1.27 1.27)) hide)
+    )
+    (pin "1")
+    (instances
+      (project "mainboard"
+        (path "/e63e39d7-6ac0-4ffd-8aa3-1841a4541b55/ee636c63-5fee-42d9-b500-aef9f04ef5c4/e2a0288b-5594-4970-9369-10c890ff0b60"
+          (reference "#PWR0111") (unit 1)
+        )
+      )

Commit message: fixes
Parts:
- added R202 (x8): 10k, Resistor_SMD:R_0402_1005Metric_Pad0.72x0.64mm_HandSolder, symbol Device:R
Connections:
- net BUS_DET.IN0: now also R202.2
- net BUS_DET.IN1: now also R202.2
- net BUS_DET.IN2: now also R202.2
- net BUS_DET.IN3: now also R202.2
- net BUS_DET.IN4: now also R202.2
- net BUS_INT.IN0: now also R202.2
- net BUS_INT.IN1: now also R202.2
- net BUS_INT.IN2: now also R202.2
- net GND: now also R202.1, R202.1, R202.1, R202.1, R202.1, R202.1, R202.1, R202.1

Commit message: prepared first versions of PCBs
Parts:
- removed R202 (x2): 10k, Resistor_SMD:R_0402_1005Metric_Pad0.72x0.64mm_HandSolder, symbol Device:R
- renumbered C505 to C63, C504 to C64, R202 to R26, R202 to R30, R202 to R33, R202 to R34, R202 to R35, R202 to R4, U10 to U9
Connections:
- net BUS_DET.IN3 is gone; now on net BUS_INT.IN2: IC1.15 (D4)
- net BUS_DET.IN4 is gone; now on net BUS_DET.IN1: IC1.12 (D7)
- net BUS_DET.IN1: no longer IC1.2 (D2)
- net BUS_DET.IN2: now also IC1.14 (D5); no longer IC1.1 (D3)
- net BUS_INT.IN1: now also IC1.13 (D6); no longer IC1.14 (D5)
- net BUS_INT.IN2: no longer IC1.13 (D6)
- net BUS_RE#.OUT0: now also U9.10 (2Y2); no longer U9.12 (2Y0)
- net BUS_RE#.OUT2: now also U9.12 (2Y0); no longer U9.10 (2Y2)
- net BUS_RE#.OUT3 renamed AUDIO.RESET#
- net BUS_RE#.OUT4: no longer names the net of U9.4 (1Y0)
- no-connect marks 4 -> 7
