File: mainboard/mainboard/mainboard.kicad_sch (KiCad schematic)
At the start: 0 parts

Commit message: refactored mainboard schematic
Other:
- removed sheet Bus multiplexers & demultiplexers
- removed sheet Connectors
- removed sheet Flash memory
- removed sheet SD Card
- removed sheet Usb connectors
- added sheet South Bridge (south_bridge.kicad_sch)
- sheet RP2040 Core ports: added BUS_DET{IN[0..6]}, BUS_INT{IN[0..6]}, BUS_RE#{OUT[0..6]}, BUS_SOUTH{D[0..3] CLK RESET#}; removed BUS_CTRL[0..4], BUS_INTERRUPT, BUS_INTERRUPT{CTRL[0..2]}, BUS{D[0..7] SCLK RWDS}, DEBUG{SWCLK SWD}, FLASH{SD[0..3] SCLK CSN}, I2C{SDA SCL}, POWER_LED, SDIO{CMD CLK D[0..3]}, UART{TX RX}, USB{D-, D+}
- sheet power_supply ports: added POWER_ENABLE; removed none

Commit message: working on PCB
Parts:
- added H1, H2, H3, H4: MountingHole, MountingHole:MountingHole_2.2mm_M2_DIN965, symbol Mechanical:MountingHole
Other:
- sheet RP2040 Core ports: added BUS_DET{IN[0..4]}, BUS_INT{IN[0..2]}, BUS_RE#{OUT[0..4]}; removed BUS_DET{IN[0..6]}, BUS_INT{IN[0..6]}, BUS_RE#{OUT[0..6]}
- sheet South Bridge ports: added BUS_DET{IN[0..4]}, BUS_INT{IN[0..2]}, BUS_RE#{OUT[0..4]}; removed BUS_DET{IN[0..6]}, BUS_INT{IN[0..6]}, BUS_RE#{OUT[0..6]}
Changed lines of the file:
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@@
-(kicad_sch (version 20221004) (generator eeschema)
+(kicad_sch (version 20221206) (generator eeschema)
   (paper "A4")
   (title_block
@@
     (stroke (width 0) (type default))
   )
+  (symbol (lib_id "Mechanical:MountingHole") (at 30.48 26.67 0) (unit 1)
+    (in_bom yes) (on_board yes) (dnp no) (fields_autoplaced)
+    (property "Reference" "H1" (at 33.02 26.035 0)
+      (effects (font (size 1.27 1.27)) (justify left))
+    )
+    (property "Value" "MountingHole" (at 33.02 28.575 0)
+      (effects (font (size 1.27 1.27)) (justify left))
+    )
+    (property "Footprint" "MountingHole:MountingHole_2.2mm_M2_DIN965" (at 30.48 26.67 0)
+      (effects (font (size 1.27 1.27)) hide)
+    )
+    (property "Datasheet" "~" (at 30.48 26.67 0)
+      (effects (font (size 1.27 1.27)) hide)
+    )
+    (instances
+      (project "mainboard"
+        (path "/e63e39d7-6ac0-4ffd-8aa3-1841a4541b55"
+          (reference "H1") (unit 1)
+        )
+      )
+    )
+  )
+  (symbol (lib_id "Mechanical:MountingHole") (at 30.48 36.83 0) (unit 1)
+    (in_bom yes) (on_board yes) (dnp no) (fields_autoplaced)
+    (property "Reference" "H3" (at 33.02 36.195 0)
+      (effects (font (size 1.27 1.27)) (justify left))
+    )
+    (property "Value" "MountingHole" (at 33.02 38.735 0)
+      (effects (font (size 1.27 1.27)) (justify left))
+    )
+    (property "Footprint" "MountingHole:MountingHole_2.2mm_M2_DIN965" (at 30.48 36.83 0)
+      (effects (font (size 1.27 1.27)) hide)
+    )
+    (property "Datasheet" "~" (at 30.48 36.83 0)
+      (effects (font (size 1.27 1.27)) hide)
+    )
+    (instances
+      (project "mainboard"
+        (path "/e63e39d7-6ac0-4ffd-8aa3-1841a4541b55"
+          (reference "H3") (unit 1)
+        )
+      )
+    )
+  )
+  (symbol (lib_id "Mechanical:MountingHole") (at 30.48 41.91 0) (unit 1)
+    (in_bom yes) (on_board yes) (dnp no) (fields_autoplaced)
+    (property "Reference" "H4" (at 33.02 41.275 0)
+      (effects (font (size 1.27 1.27)) (justify left))
+    )
+    (property "Value" "MountingHole" (at 33.02 43.815 0)
+      (effects (font (size 1.27 1.27)) (justify left))
+    )
+    (property "Footprint" "MountingHole:MountingHole_2.2mm_M2_DIN965" (at 30.48 41.91 0)
+      (effects (font (size 1.27 1.27)) hide)
+    )
+    (property "Datasheet" "~" (at 30.48 41.91 0)
+      (effects (font (size 1.27 1.27)) hide)
+    )
+    (instances
+      (project "mainboard"
+        (path "/e63e39d7-6ac0-4ffd-8aa3-1841a4541b55"
+          (reference "H4") (unit 1)
+        )
+      )
+    )
+  )
+  (symbol (lib_id "Mechanical:MountingHole") (at 30.48 31.75 0) (unit 1)
+    (in_bom yes) (on_board yes) (dnp no) (fields_autoplaced)
+    (property "Reference" "H2" (at 33.02 31.115 0)
+      (effects (font (size 1.27 1.27)) (justify left))
+    )
+    (property "Value" "MountingHole" (at 33.02 33.655 0)
+      (effects (font (size 1.27 1.27)) (justify left))
+    )
+    (property "Footprint" "MountingHole:MountingHole_2.2mm_M2_DIN965" (at 30.48 31.75 0)
+      (effects (font (size 1.27 1.27)) hide)
+    )
+    (property "Datasheet" "~" (at 30.48 31.75 0)
+      (effects (font (size 1.27 1.27)) hide)
+    )
+    (instances
+      (project "mainboard"
+        (path "/e63e39d7-6ac0-4ffd-8aa3-1841a4541b55"
+          (reference "H2") (unit 1)
+        )
+      )
+    )
+  )
   (sheet (at 46.99 97.79) (size 36.83 31.75) (fields_autoplaced)
     (stroke (width 0.1524) (type solid))
@@
     (pin "POWER_ENABLE" input (at 74.93 97.79 90)
       (effects (font (size 1.27 1.27)) (justify right))
+    )
+    (instances
+      (project "mainboard"
+        (path "/e63e39d7-6ac0-4ffd-8aa3-1841a4541b55" (page "3"))
+      )
     )
   )
@@
       (effects (font (size 1.27 1.27)) (justify right))
     )
-    (pin "BUS_RE#{OUT[0..6]}" input (at 151.13 97.79 90)
+    (pin "BUS_INT{IN[0..2]}" output (at 143.51 97.79 90)
       (effects (font (size 1.27 1.27)) (justify right))
     )
-    (pin "BUS_DET{IN[0..6]}" output (at 147.32 97.79 90)
+    (pin "BUS_DET{IN[0..4]}" output (at 147.32 97.79 90)
       (effects (font (size 1.27 1.27)) (justify right))
     )
-    (pin "BUS_INT{IN[0..6]}" output (at 143.51 97.79 90)
+    (pin "BUS_RE#{OUT[0..4]}" input (at 151.13 97.79 90)
       (effects (font (size 1.27 1.27)) (justify right))
+    )
+    (instances
+      (project "mainboard"
+        (path "/e63e39d7-6ac0-4ffd-8aa3-1841a4541b55" (page "2"))
+      )
     )
   )
@@
       (effects (font (size 1.27 1.27)) (justify left top))
     )
-    (pin "BUS_DET{IN[0..6]}" input (at 147.32 90.17 270)
+    (pin "BUS_DET{IN[0..4]}" input (at 147.32 90.17 270)
       (effects (font (size 1.27 1.27)) (justify left))
     )
-    (pin "BUS_RE#{OUT[0..6]}" output (at 151.13 90.17 270)
+    (pin "BUS_RE#{OUT[0..4]}" output (at 151.13 90.17 270)
       (effects (font (size 1.27 1.27)) (justify left))
     )
@@
       (effects (font (size 1.27 1.27)) (justify left))
     )
-    (pin "BUS_INT{IN[0..6]}" bidirectional (at 143.51 90.17 270)
+    (pin "BUS_INT{IN[0..2]}" bidirectional (at 143.51 90.17 270)
       (effects (font (size 1.27 1.27)) (justify left))
+    )
+    (instances
+      (project "mainboard"
+        (path "/e63e39d7-6ac0-4ffd-8aa3-1841a4541b55" (page "9"))
+      )
     )
   )
   (sheet_instances
-    (path "/e63e39d7-6ac0-4ffd-8aa3-1841a4541b55" (page "1"))
-    (path "/e63e39d7-6ac0-4ffd-8aa3-1841a4541b55/90a5bc85-07ac-4ee1-af41-887c984cc4b9" (page "2"))
-    (path "/e63e39d7-6ac0-4ffd-8aa3-1841a4541b55/8c334f51-6a0b-406c-9f2c-47b0eaeba7c1" (page "3"))
-    (path "/e63e39d7-6ac0-4ffd-8aa3-1841a4541b55/ee636c63-5fee-42d9-b500-aef9f04ef5c4/5992df64-4101-4a52-b6a6-07d8f4453a45" (page "4"))
-    (path "/e63e39d7-6ac0-4ffd-8aa3-1841a4541b55/ee636c63-5fee-42d9-b500-aef9f04ef5c4" (page "9"))
-    (path "/e63e39d7-6ac0-4ffd-8aa3-1841a4541b55/ee636c63-5fee-42d9-b500-aef9f04ef5c4/82247a11-188e-40f6-a2f8-9149daba124e" (page "10"))
-    (path "/e63e39d7-6ac0-4ffd-8aa3-1841a4541b55/ee636c63-5fee-42d9-b500-aef9f04ef5c4/e2a0288b-5594-4970-9369-10c890ff0b60" (page "11"))
-    (path "/e63e39d7-6ac0-4ffd-8aa3-1841a4541b55/ee636c63-5fee-42d9-b500-aef9f04ef5c4/b34a86cb-f778-45af-b876-f75dc7b3f02d" (page "12"))
-    (path "/e63e39d7-6ac0-4ffd-8aa3-1841a4541b55/ee636c63-5fee-42d9-b500-aef9f04ef5c4/2f8d2ed3-bd82-4f8a-ae27-6fa7e5d02426" (page "13"))
-    (path "/e63e39d7-6ac0-4ffd-8aa3-1841a4541b55/ee636c63-5fee-42d9-b500-aef9f04ef5c4/9c458a31-8cc6-4b30-bfc6-26fedc686704" (page "14"))
-    (path "/e63e39d7-6ac0-4ffd-8aa3-1841a4541b55/ee636c63-5fee-42d9-b500-aef9f04ef5c4/e539fd0d-6f44-42c6-b17c-465bf8b74b11" (page "15"))
-    (path "/e63e39d7-6ac0-4ffd-8aa3-1841a4541b55/90a5bc85-07ac-4ee1-af41-887c984cc4b9/fda91f01-15e3-49e1-9dbc-660155d6725a" (page "16"))
-    (path "/e63e39d7-6ac0-4ffd-8aa3-1841a4541b55/90a5bc85-07ac-4ee1-af41-887c984cc4b9/78fa6cb9-f921-4861-9f70-f5ecadaf057b" (page "17"))
-    (path "/e63e39d7-6ac0-4ffd-8aa3-1841a4541b55/90a5bc85-07ac-4ee1-af41-887c984cc4b9/e8a0e619-f78c-4b86-bbf0-84ff0e9ddba1" (page "18"))
+    (path "/" (page "1"))
   )
 )

Commit message: prepared first versions of PCBs
Parts:
- added H5, H6, H7: MountingHole, MountingHole:MountingHole_2.2mm_M2_DIN965, symbol Mechanical:MountingHole
- H1, H2, H3, H4: footprint MountingHole:MountingHole_2.2mm_M2_DIN965 -> MountingHole:MountingHole_3.2mm_M3_DIN965
Other:
- removed sheet South Bridge
- sheet RP2040 Core ports: added POWER_ENABLE; removed BUS_DET{IN[0..4]}, BUS_INT{IN[0..2]}, BUS_RE#{OUT[0..4]}, BUS_SOUTH{D[0..3] CLK RESET#}
