File: mainboard/mainboard/mcu_connectors.kicad_sch (KiCad schematic)
At the start: 8 parts, among them J10 Connector B - 2 bit, J4 Connector 16-bit, J5 Connector A 8-bit, J6 Connector B 8-bit, J609 Conn_01x03_Female, J7 Connector A - 4 bit, J8 Connector B - 4 bit, J9 Connector A - 2 bit

Commit message: working on new pcb
Parts:
- renumbered J4 to J13, J5 to J14, J6 to J15, J7 to J16, J8 to J17, J9 to J18, J10 to J19
Connections:
- net BUS_CS#B0 is gone; now on net BUS_RE#.OUT1: J15.17 (Pin_17)
- net BUS_CS#B1 is gone; now on net BUS_INT.IN1: J15.19 (Pin_19)
- net BUS_CS#A0: now also J13.25 (Pin_25); no longer J13.27 (Pin_27)
- net BUS_CS#A1: now also J13.26 (Pin_26); no longer J13.29 (Pin_29)
- net BUS_CS#A2: now also J14.15 (Pin_15); no longer J14.17 (Pin_17)
- net BUS_CS#A3: now also J14.16 (Pin_16); no longer J14.19 (Pin_19)
- net BUS_CS#A4: now also J16.11 (Pin_11); no longer J16.13 (Pin_13)
- net BUS_CS#A5: now also J16.12 (Pin_12); no longer J16.15 (Pin_15)
- net BUS_CS#A6: now also J18.7 (Pin_7); no longer J18.10 (Pin_10)
- net BUS_CS#B2: now also J15.15 (Pin_15); no longer J17.13 (Pin_13)
- net BUS_CS#B3: now also J15.16 (Pin_16); no longer J17.15 (Pin_15)
- net BUS_CS#B4: now also J17.11 (Pin_11); no longer J19.10 (Pin_10)
- net BUS_DET.IN0: now also J13.28 (Pin_28); no longer J13.23 (Pin_23)
- net BUS_DET.IN1: now also J15.18 (Pin_18); no longer J14.13 (Pin_13)
- net BUS_DET.IN2: now also J17.14 (Pin_14); no longer J15.13 (Pin_13)
- net BUS_DET.IN3: now also J19.9 (Pin_9); no longer J16.9 (Pin_9)
- net BUS_DET.IN4: now also J14.18 (Pin_18); no longer J17.9 (Pin_9)
- net BUS_DET.IN5: now also J16.14 (Pin_14); no longer J18.7 (Pin_7)
- net BUS_DET.IN6: now also J18.9 (Pin_9); no longer J19.7 (Pin_7)
- net BUS_INT.IN0: now also J13.29 (Pin_29); no longer J13.28 (Pin_28)
- net BUS_INT.IN1: no longer J14.18 (Pin_18)
- net BUS_INT.IN2: now also J17.15 (Pin_15); no longer J15.18 (Pin_18)
- net BUS_INT.IN3: now also J19.10 (Pin_10); no longer J16.14 (Pin_14)
- net BUS_INT.IN4: now also J14.19 (Pin_19); no longer J17.14 (Pin_14)
- net BUS_INT.IN5: now also J16.15 (Pin_15); no longer J18.8 (Pin_8)
- net BUS_INT.IN6: now also J18.10 (Pin_10); no longer J19.8 (Pin_8)
- net BUS_NORTH.CLK0: now also J15.14 (Pin_14), J17.10 (Pin_10), J19.6 (Pin_6); no longer J13.25 (Pin_25), J14.15 (Pin_15), J16.11 (Pin_11)
- net BUS_NORTH.CLK1: now also J13.24 (Pin_24), J14.14 (Pin_14), J16.10 (Pin_10), J18.6 (Pin_6); no longer J15.15 (Pin_15), J17.11 (Pin_11)
- net BUS_NORTH.D0: now also J13.23 (Pin_23), J14.13 (Pin_13); no longer J13.24 (Pin_24), J14.14 (Pin_14), J16.10 (Pin_10), J18.5 (Pin_5)
- net BUS_NORTH.D1: now also J13.22 (Pin_22), J14.12 (Pin_12); no longer J13.21 (Pin_21), J14.11 (Pin_11), J16.7 (Pin_7), J18.4 (Pin_4)
- net BUS_NORTH.D10: now also J13.13 (Pin_13), J15.11 (Pin_11); no longer J13.14 (Pin_14), J15.12 (Pin_12), J17.8 (Pin_8)
- net BUS_NORTH.D11: now also J13.12 (Pin_12), J15.10 (Pin_10); no longer J13.11 (Pin_11), J15.9 (Pin_9), J17.5 (Pin_5)
- net BUS_NORTH.D12: now also J13.11 (Pin_11), J15.9 (Pin_9), J17.9 (Pin_9); no longer J13.12 (Pin_12), J15.10 (Pin_10)
- net BUS_NORTH.D13: now also J13.10 (Pin_10), J15.8 (Pin_8), J17.8 (Pin_8); no longer J13.9 (Pin_9), J15.7 (Pin_7)
- net BUS_NORTH.D14: now also J13.9 (Pin_9), J15.7 (Pin_7), J17.7 (Pin_7), J19.5 (Pin_5); no longer J13.10 (Pin_10), J15.8 (Pin_8)
- net BUS_NORTH.D15: now also J13.8 (Pin_8), J15.6 (Pin_6), J17.6 (Pin_6), J19.4 (Pin_4); no longer J13.7 (Pin_7), J15.5 (Pin_5)
- net BUS_NORTH.D2: now also J13.21 (Pin_21), J14.11 (Pin_11); no longer J13.22 (Pin_22), J14.12 (Pin_12), J16.8 (Pin_8)
- net BUS_NORTH.D3: now also J13.20 (Pin_20), J14.10 (Pin_10); no longer J13.19 (Pin_19), J14.9 (Pin_9), J16.5 (Pin_5)
- net BUS_NORTH.D4: now also J13.19 (Pin_19), J14.9 (Pin_9), J16.9 (Pin_9); no longer J13.20 (Pin_20), J14.10 (Pin_10)
- net BUS_NORTH.D5: now also J13.18 (Pin_18), J14.8 (Pin_8), J16.8 (Pin_8); no longer J13.17 (Pin_17), J14.7 (Pin_7)
- net BUS_NORTH.D6: now also J13.17 (Pin_17), J14.7 (Pin_7), J16.7 (Pin_7), J18.5 (Pin_5); no longer J13.18 (Pin_18), J14.8 (Pin_8)
- net BUS_NORTH.D7: now also J13.16 (Pin_16), J14.6 (Pin_6), J16.6 (Pin_6), J18.4 (Pin_4); no longer J13.15 (Pin_15), J14.5 (Pin_5)
- net BUS_NORTH.D8: now also J13.15 (Pin_15), J15.13 (Pin_13); no longer J13.16 (Pin_16), J15.14 (Pin_14), J17.10 (Pin_10), J19.5 (Pin_5)
- net BUS_NORTH.D9: now also J13.14 (Pin_14), J15.12 (Pin_12); no longer J13.13 (Pin_13), J15.11 (Pin_11), J17.7 (Pin_7), J19.4 (Pin_4)
- net BUS_NORTH.RWDS: now also J13.7 (Pin_7), J14.5 (Pin_5), J15.5 (Pin_5), J16.5 (Pin_5), J17.5 (Pin_5); no longer J13.8 (Pin_8), J14.6 (Pin_6), J15.6 (Pin_6), J16.6 (Pin_6), J17.6 (Pin_6)
- net BUS_RE#.OUT0: now also J13.27 (Pin_27); no longer J13.26 (Pin_26)
- net BUS_RE#.OUT1: no longer J14.16 (Pin_16)
- net BUS_RE#.OUT2: now also J17.13 (Pin_13); no longer J15.16 (Pin_16)
- net BUS_RE#.OUT3: now also J19.8 (Pin_8); no longer J16.12 (Pin_12)
- net BUS_RE#.OUT4: now also J14.17 (Pin_17); no longer J17.12 (Pin_12)
- net BUS_RE#.OUT5: now also J16.13 (Pin_13); no longer J18.6 (Pin_6)
- net BUS_RE#.OUT6: now also J18.8 (Pin_8); no longer J19.6 (Pin_6)
- removed net BUS.CLK0: J18.9 (Pin_9), J19.9 (Pin_9)
- new net BUS_CS#B5: J17.12 (Pin_12)
- new net BUS_CS#B6: J19.7 (Pin_7)

Commit message: working on PCB
Parts:
- removed J18: Connector A - 2 bit, Connector_PinHeader_1.27mm:PinHeader_2x05_P1.27mm_Vertical_SMD, symbol Connector_Generic:Conn_02x05_Odd_Even
- removed J19: Connector B - 2 bit, Connector_PinHeader_1.27mm:PinHeader_2x05_P1.27mm_Vertical_SMD, symbol Connector_Generic:Conn_02x05_Odd_Even
- J13: value Connector 16-bit -> Connector A 16-bit
- J609: footprint Connector_PinSocket_2.54mm:PinSocket_1x03_P2.54mm_Vertical -> Connector_PinHeader_2.54mm:PinHeader_1x03_P2.54mm_Vertical
- renumbered J16 to J15, J17 to J16, J15 to J17
Connections:
- net BUS_CS#A5 is gone; now on net +5V_BUS: J15.12 (Pin_12)
- net BUS_CS#B4 is gone; now on net BUS_INT.IN2: J16.11 (Pin_11)
- net BUS_CS#B5 is gone; now on net +5V_BUS: J16.12 (Pin_12)
- net BUS_DET.IN5 is gone; now on net GND: J15.14 (Pin_14)
- net BUS_INT.IN4 is gone; now on net GND: J14.19 (Pin_19)
- net BUS_INT.IN5 is gone; now on net GND: J15.15 (Pin_15)
- net BUS_RE#.OUT5 is gone; now on net +3V3_BUS: J15.13 (Pin_13)
- net +3V3_BUS: now also J13.27 (Pin_27), J14.17 (Pin_17), J16.13 (Pin_13), J17.17 (Pin_17); no longer J13.3 (Pin_3), J13.4 (Pin_4), J14.1 (Pin_1), J15.1 (Pin_1), J16.1 (Pin_1), J17.1 (Pin_1)
- net +5V_BUS: now also J13.26 (Pin_26), J14.16 (Pin_16), J17.16 (Pin_16); no longer J13.1 (Pin_1), J13.2 (Pin_2), J14.2 (Pin_2), J15.2 (Pin_2), J16.2 (Pin_2), J17.2 (Pin_2)
- net BUS_CS#A0: now also J13.21 (Pin_21); no longer J13.25 (Pin_25)
- net BUS_CS#A1: now also J13.22 (Pin_22); no longer J13.26 (Pin_26)
- net BUS_CS#A2: now also J14.11 (Pin_11); no longer J14.15 (Pin_15)
- net BUS_CS#A3: now also J15.7 (Pin_7); no longer J14.16 (Pin_16)
- net BUS_CS#B2: now also J16.7 (Pin_7); no longer J17.15 (Pin_15)
- net BUS_CS#B3: now also J16.8 (Pin_8); no longer J17.16 (Pin_16)
- net BUS_DET.IN0: now also J13.23 (Pin_23); no longer J13.28 (Pin_28)
- net BUS_DET.IN1: now also J14.13 (Pin_13); no longer J17.18 (Pin_18)
- net BUS_DET.IN2: now also J15.9 (Pin_9); no longer J16.14 (Pin_14)
- net BUS_DET.IN3: now also J17.13 (Pin_13)
- net BUS_DET.IN4: now also J16.9 (Pin_9); no longer J14.18 (Pin_18)
- net BUS_INT.IN0: now also J13.25 (Pin_25); no longer J13.29 (Pin_29)
- net BUS_INT.IN1: now also J17.15 (Pin_15); no longer J17.19 (Pin_19)
- net BUS_INT.IN2: no longer J16.15 (Pin_15)
- net BUS_NORTH.CLK0: now also J16.6 (Pin_6), J17.10 (Pin_10); no longer J16.10 (Pin_10), J17.14 (Pin_14)
- net BUS_NORTH.CLK1: now also J13.20 (Pin_20), J14.10 (Pin_10), J15.6 (Pin_6); no longer J13.24 (Pin_24), J14.14 (Pin_14), J15.10 (Pin_10)
- net BUS_NORTH.D0: now also J13.18 (Pin_18), J16.4 (Pin_4), J17.8 (Pin_8); no longer J13.23 (Pin_23), J14.13 (Pin_13)
- net BUS_NORTH.D1: now also J13.17 (Pin_17), J16.3 (Pin_3), J17.7 (Pin_7); no longer J13.22 (Pin_22), J14.12 (Pin_12)
- net BUS_NORTH.D10: now also J13.8 (Pin_8), J14.6 (Pin_6), J15.2 (Pin_2); no longer J13.13 (Pin_13), J17.11 (Pin_11)
- net BUS_NORTH.D11: now also J13.7 (Pin_7), J14.5 (Pin_5), J15.1 (Pin_1); no longer J13.12 (Pin_12), J17.10 (Pin_10)
- net BUS_NORTH.D12: now also J13.6 (Pin_6), J14.4 (Pin_4); no longer J13.11 (Pin_11), J16.9 (Pin_9), J17.9 (Pin_9)
- net BUS_NORTH.D13: now also J13.5 (Pin_5), J14.3 (Pin_3); no longer J13.10 (Pin_10), J16.8 (Pin_8), J17.8 (Pin_8)
- net BUS_NORTH.D14: now also J13.4 (Pin_4), J14.2 (Pin_2); no longer J13.9 (Pin_9), J16.7 (Pin_7), J17.7 (Pin_7)
- net BUS_NORTH.D15: now also J13.3 (Pin_3), J14.1 (Pin_1); no longer J13.8 (Pin_8), J16.6 (Pin_6), J17.6 (Pin_6)
- net BUS_NORTH.D2: now also J13.16 (Pin_16), J16.2 (Pin_2), J17.6 (Pin_6); no longer J13.21 (Pin_21), J14.11 (Pin_11)
- net BUS_NORTH.D3: now also J13.15 (Pin_15), J16.1 (Pin_1), J17.5 (Pin_5); no longer J13.20 (Pin_20), J14.10 (Pin_10)
- net BUS_NORTH.D4: now also J13.14 (Pin_14), J17.4 (Pin_4); no longer J13.19 (Pin_19), J14.9 (Pin_9), J15.9 (Pin_9)
- net BUS_NORTH.D5: now also J13.13 (Pin_13), J17.3 (Pin_3); no longer J13.18 (Pin_18), J14.8 (Pin_8), J15.8 (Pin_8)
- net BUS_NORTH.D6: now also J13.12 (Pin_12), J17.2 (Pin_2); no longer J13.17 (Pin_17), J14.7 (Pin_7), J15.7 (Pin_7)
- net BUS_NORTH.D7: now also J13.11 (Pin_11), J17.1 (Pin_1); no longer J13.16 (Pin_16), J14.6 (Pin_6), J15.6 (Pin_6)
- net BUS_NORTH.D8: now also J13.10 (Pin_10), J14.8 (Pin_8), J15.4 (Pin_4); no longer J13.15 (Pin_15), J17.13 (Pin_13)
- net BUS_NORTH.D9: now also J13.9 (Pin_9), J14.7 (Pin_7), J15.3 (Pin_3); no longer J13.14 (Pin_14), J17.12 (Pin_12)
- net BUS_NORTH.RWDS: now also J13.19 (Pin_19), J14.9 (Pin_9), J17.9 (Pin_9); no longer J13.7 (Pin_7), J14.5 (Pin_5), J17.5 (Pin_5)
- net BUS_RE#.OUT0: now also J13.24 (Pin_24); no longer J13.27 (Pin_27)
- net BUS_RE#.OUT1: now also J14.14 (Pin_14); no longer J17.17 (Pin_17)
- net BUS_RE#.OUT2: now also J15.10 (Pin_10); no longer J16.13 (Pin_13)
- net BUS_RE#.OUT3: now also J17.14 (Pin_14)
- net BUS_RE#.OUT4: now also J16.10 (Pin_10); no longer J14.17 (Pin_17)
- net GND: now also J13.1 (Pin_1), J13.2 (Pin_2), J13.28 (Pin_28), J13.29 (Pin_29), J14.18 (Pin_18), J16.14 (Pin_14), J16.15 (Pin_15), J17.18 (Pin_18), J17.19 (Pin_19); no longer J13.5 (Pin_5), J13.6 (Pin_6), J14.3 (Pin_3), J14.4 (Pin_4), J15.3 (Pin_3), J15.4 (Pin_4), J16.3 (Pin_3), J16.4 (Pin_4), J17.3 (Pin_3), J17.4 (Pin_4)
- net BUS_CS#A4: no longer names the net of J15.11 (Pin_11)
- new net BUS_CS#B0: J17.11 (Pin_11)
- new net BUS_CS#B1: J17.12 (Pin_12)
- no-connect marks 5 -> 9
Other:
- moved on the sheet: J13, J14, J15, J16, J17, J609

Commit message: Mainboard rev 1.0a prepared
Parts:
- J13: footprint Connector_PinHeader_1.27mm:PinHeader_2x15_P1.27mm_Vertical_SMD -> Connector_PinSocket_1.27mm:PinSocket_2x15_P1.27mm_Vertical_SMD
- J14, J17: footprint Connector_PinHeader_1.27mm:PinHeader_2x10_P1.27mm_Vertical_SMD -> Connector_PinSocket_1.27mm:PinSocket_2x10_P1.27mm_Vertical_SMD
- J15, J16: footprint Connector_PinHeader_1.27mm:PinHeader_2x08_P1.27mm_Vertical_SMD -> Connector_PinSocket_1.27mm:PinSocket_2x08_P1.27mm_Vertical_SMD
Connections:
- net +3V3_BUS: now also J13.28 (Pin_28), J14.18 (Pin_18), J15.14 (Pin_14), J16.14 (Pin_14), J17.18 (Pin_18); no longer J13.27 (Pin_27), J14.17 (Pin_17), J15.13 (Pin_13), J16.13 (Pin_13), J17.17 (Pin_17)
- net +5V_BUS: now also J13.25 (Pin_25), J14.15 (Pin_15), J15.11 (Pin_11), J16.11 (Pin_11), J17.15 (Pin_15); no longer J13.26 (Pin_26), J14.16 (Pin_16), J15.12 (Pin_12), J16.12 (Pin_12), J17.16 (Pin_16)
- net BUS_CS#A0: now also J13.22 (Pin_22); no longer J13.21 (Pin_21)
- net BUS_CS#A1: now also J13.21 (Pin_21); no longer J13.22 (Pin_22)
- net BUS_CS#A2: now also J14.12 (Pin_12); no longer J14.11 (Pin_11)
- net BUS_CS#A3: now also J15.8 (Pin_8); no longer J15.7 (Pin_7)
- net BUS_CS#B0: now also J17.12 (Pin_12); no longer J17.11 (Pin_11)
- net BUS_CS#B1: now also J17.11 (Pin_11); no longer J17.12 (Pin_12)
- net BUS_CS#B2: now also J16.8 (Pin_8); no longer J16.7 (Pin_7)
- net BUS_CS#B3: now also J16.7 (Pin_7); no longer J16.8 (Pin_8)
- net BUS_DET.IN0: now also J13.24 (Pin_24); no longer J13.23 (Pin_23)
- net BUS_DET.IN1: now also J14.14 (Pin_14); no longer J14.13 (Pin_13)
- net BUS_DET.IN2: now also J15.10 (Pin_10); no longer J15.9 (Pin_9)
- net BUS_DET.IN3: now also J17.14 (Pin_14); no longer J17.13 (Pin_13)
- net BUS_DET.IN4: now also J16.10 (Pin_10); no longer J16.9 (Pin_9)
- net BUS_INT.IN0: now also J13.26 (Pin_26); no longer J13.25 (Pin_25)
- net BUS_INT.IN1: now also J17.16 (Pin_16); no longer J17.15 (Pin_15)
- net BUS_INT.IN2: now also J16.12 (Pin_12); no longer J16.11 (Pin_11)
- net BUS_NORTH.CLK0: now also J16.5 (Pin_5), J17.9 (Pin_9); no longer J16.6 (Pin_6), J17.10 (Pin_10)
- net BUS_NORTH.CLK1: now also J13.19 (Pin_19), J14.9 (Pin_9), J15.5 (Pin_5); no longer J13.20 (Pin_20), J14.10 (Pin_10), J15.6 (Pin_6)
- net BUS_NORTH.D0: now also J13.17 (Pin_17), J16.3 (Pin_3), J17.7 (Pin_7); no longer J13.18 (Pin_18), J16.4 (Pin_4), J17.8 (Pin_8)
- net BUS_NORTH.D1: now also J13.18 (Pin_18), J16.4 (Pin_4), J17.8 (Pin_8); no longer J13.17 (Pin_17), J16.3 (Pin_3), J17.7 (Pin_7)
- net BUS_NORTH.D10: now also J13.7 (Pin_7), J14.5 (Pin_5), J15.1 (Pin_1); no longer J13.8 (Pin_8), J14.6 (Pin_6), J15.2 (Pin_2)
- net BUS_NORTH.D11: now also J13.8 (Pin_8), J14.6 (Pin_6), J15.2 (Pin_2); no longer J13.7 (Pin_7), J14.5 (Pin_5), J15.1 (Pin_1)
- net BUS_NORTH.D12: now also J13.5 (Pin_5), J14.3 (Pin_3); no longer J13.6 (Pin_6), J14.4 (Pin_4)
- net BUS_NORTH.D13: now also J13.6 (Pin_6), J14.4 (Pin_4); no longer J13.5 (Pin_5), J14.3 (Pin_3)
- net BUS_NORTH.D14: now also J13.3 (Pin_3), J14.1 (Pin_1); no longer J13.4 (Pin_4), J14.2 (Pin_2)
- net BUS_NORTH.D15: now also J13.4 (Pin_4), J14.2 (Pin_2); no longer J13.3 (Pin_3), J14.1 (Pin_1)
- net BUS_NORTH.D2: now also J13.15 (Pin_15), J16.1 (Pin_1), J17.5 (Pin_5); no longer J13.16 (Pin_16), J16.2 (Pin_2), J17.6 (Pin_6)
- net BUS_NORTH.D3: now also J13.16 (Pin_16), J16.2 (Pin_2), J17.6 (Pin_6); no longer J13.15 (Pin_15), J16.1 (Pin_1), J17.5 (Pin_5)
- net BUS_NORTH.D4: now also J13.13 (Pin_13), J17.3 (Pin_3); no longer J13.14 (Pin_14), J17.4 (Pin_4)
- net BUS_NORTH.D5: now also J13.14 (Pin_14), J17.4 (Pin_4); no longer J13.13 (Pin_13), J17.3 (Pin_3)
- net BUS_NORTH.D6: now also J13.11 (Pin_11), J17.1 (Pin_1); no longer J13.12 (Pin_12), J17.2 (Pin_2)
- net BUS_NORTH.D7: now also J13.12 (Pin_12), J17.2 (Pin_2); no longer J13.11 (Pin_11), J17.1 (Pin_1)
- net BUS_NORTH.D8: now also J13.9 (Pin_9), J14.7 (Pin_7), J15.3 (Pin_3); no longer J13.10 (Pin_10), J14.8 (Pin_8), J15.4 (Pin_4)
- net BUS_NORTH.D9: now also J13.10 (Pin_10), J14.8 (Pin_8), J15.4 (Pin_4); no longer J13.9 (Pin_9), J14.7 (Pin_7), J15.3 (Pin_3)
- net BUS_NORTH.RWDS: now also J13.20 (Pin_20), J14.10 (Pin_10), J15.6 (Pin_6), J16.6 (Pin_6), J17.10 (Pin_10); no longer J13.19 (Pin_19), J14.9 (Pin_9), J15.5 (Pin_5), J16.5 (Pin_5), J17.9 (Pin_9)
- net BUS_RE#.OUT0: now also J13.23 (Pin_23); no longer J13.24 (Pin_24)
- net BUS_RE#.OUT1: now also J14.13 (Pin_13); no longer J14.14 (Pin_14)
- net BUS_RE#.OUT2: now also J15.9 (Pin_9); no longer J15.10 (Pin_10)
- net BUS_RE#.OUT3: now also J17.13 (Pin_13); no longer J17.14 (Pin_14)
- net BUS_RE#.OUT4: now also J16.9 (Pin_9); no longer J16.10 (Pin_10)
- net GND: now also J13.27 (Pin_27), J13.30 (Pin_30), J14.17 (Pin_17), J14.20 (Pin_20), J15.13 (Pin_13), J15.16 (Pin_16), J16.13 (Pin_13), J16.16 (Pin_16), J17.17 (Pin_17), J17.20 (Pin_20); no longer J13.28 (Pin_28), J13.29 (Pin_29), J14.18 (Pin_18), J14.19 (Pin_19), J15.14 (Pin_14), J15.15 (Pin_15), J16.14 (Pin_14), J16.15 (Pin_15), J17.18 (Pin_18), J17.19 (Pin_19)

Commit message: prepared first versions of PCBs
Parts:
- removed J15: Connector A - 4 bit, Connector_PinSocket_1.27mm:PinSocket_2x08_P1.27mm_Vertical_SMD, symbol Connector_Generic:Conn_02x08_Odd_Even
- removed J16: Connector B - 4 bit, Connector_PinSocket_1.27mm:PinSocket_2x08_P1.27mm_Vertical_SMD, symbol Connector_Generic:Conn_02x08_Odd_Even
- removed J609: Conn_01x03_Female, Connector_PinHeader_2.54mm:PinHeader_1x03_P2.54mm_Vertical, symbol Connector:Conn_01x03_Female
- added J10, J9: AudioJack4, Connector_Audio:Jack_3.5mm_PJ320D_Horizontal, symbol Connector:AudioJack4
- added J11, J8: Conn_01x03_Female, Connector_PinHeader_2.54mm:PinHeader_1x03_P2.54mm_Vertical, symbol Connector:Conn_01x03_Female
- added J7: Conn_01x04_Female, Connector_PinHeader_2.54mm:PinHeader_1x04_P2.54mm_Vertical, symbol Connector:Conn_01x04_Female
- renumbered J17 to J15
Connections:
- net BUS_DET.IN3 is gone; now on net BUS_DET.IN2: J15.14 (Pin_14)
- net BUS_RE#.OUT3 is gone; now on net BUS_INT.IN2: J15.13 (Pin_13)
- net +3V3_BUS: now also J7.1 (Pin_1)
- net BUS_CS#A1: now also J13.20 (Pin_20); no longer J13.21 (Pin_21)
- net BUS_CS#A3: now also J14.10 (Pin_10)
- net BUS_CS#B1: now also J15.10 (Pin_10); no longer J15.11 (Pin_11)
- net BUS_INT.IN0: now also J13.23 (Pin_23); no longer J13.26 (Pin_26)
- net BUS_INT.IN1: now also J14.13 (Pin_13); no longer J15.16 (Pin_16)
- net BUS_NORTH.D0: now also J13.18 (Pin_18), J15.8 (Pin_8); no longer J13.17 (Pin_17), J15.7 (Pin_7)
- net BUS_NORTH.D1: now also J13.17 (Pin_17), J15.7 (Pin_7); no longer J13.18 (Pin_18), J15.8 (Pin_8)
- net BUS_NORTH.D10: now also J13.8 (Pin_8), J14.6 (Pin_6); no longer J13.7 (Pin_7), J14.5 (Pin_5)
- net BUS_NORTH.D11: now also J13.7 (Pin_7), J14.5 (Pin_5); no longer J13.8 (Pin_8), J14.6 (Pin_6)
- net BUS_NORTH.D12: now also J13.6 (Pin_6), J14.4 (Pin_4); no longer J13.5 (Pin_5), J14.3 (Pin_3)
- net BUS_NORTH.D13: now also J13.5 (Pin_5), J14.3 (Pin_3); no longer J13.6 (Pin_6), J14.4 (Pin_4)
- net BUS_NORTH.D14: now also J13.4 (Pin_4), J14.2 (Pin_2); no longer J13.3 (Pin_3), J14.1 (Pin_1)
- net BUS_NORTH.D15: now also J13.3 (Pin_3), J14.1 (Pin_1); no longer J13.4 (Pin_4), J14.2 (Pin_2)
- net BUS_NORTH.D2: now also J13.16 (Pin_16), J15.6 (Pin_6); no longer J13.15 (Pin_15), J15.5 (Pin_5)
- net BUS_NORTH.D3: now also J13.15 (Pin_15), J15.5 (Pin_5); no longer J13.16 (Pin_16), J15.6 (Pin_6)
- net BUS_NORTH.D4: now also J13.14 (Pin_14), J15.4 (Pin_4); no longer J13.13 (Pin_13), J15.3 (Pin_3)
- net BUS_NORTH.D5: now also J13.13 (Pin_13), J15.3 (Pin_3); no longer J13.14 (Pin_14), J15.4 (Pin_4)
- net BUS_NORTH.D6: now also J13.12 (Pin_12), J15.2 (Pin_2); no longer J13.11 (Pin_11), J15.1 (Pin_1)
- net BUS_NORTH.D7: now also J13.11 (Pin_11), J15.1 (Pin_1); no longer J13.12 (Pin_12), J15.2 (Pin_2)
- net BUS_NORTH.D8: now also J13.10 (Pin_10), J14.8 (Pin_8); no longer J13.9 (Pin_9), J14.7 (Pin_7)
- net BUS_NORTH.D9: now also J13.9 (Pin_9), J14.7 (Pin_7); no longer J13.10 (Pin_10), J14.8 (Pin_8)
- net BUS_RE#.OUT0: now also J13.26 (Pin_26); no longer J13.23 (Pin_23)
- net BUS_RE#.OUT1: now also J14.16 (Pin_16); no longer J14.13 (Pin_13)
- net BUS_RE#.OUT2: now also J15.16 (Pin_16)
- net DEBUG.SWCLK: now also J8.1 (Pin_1)
- net DEBUG.SWD: now also J8.3 (Pin_3)
- net GND: now also J10.R2, J10.S, J11.2 (Pin_2), J7.2 (Pin_2), J8.2 (Pin_2), J9.R2, J9.S
- removed net BUS_NORTH.RWDS: J13.20 (Pin_20), J14.10 (Pin_10), J15.10 (Pin_10)
- new net AUDIO_OUT.L: J9.T
- new net AUDIO_OUT.R: J9.R1
- new net AUX_IN.L: J10.T
- new net AUX_IN.R: J10.R1
- new net I2C.SCL: J7.4 (Pin_4)
- new net I2C.SDA: J7.3 (Pin_3)
- new net UART.RX: J11.3 (Pin_3)
- new net UART.TX: J11.1 (Pin_1)
- no-connect marks 9 -> 6
Other:
- moved on the sheet: J15
