File: mainboard/mainboard/mcu_flash.kicad_sch (KiCad schematic)
At the start: 3 parts, among them U401 W25Q128JVS

Commit message: working on new pcb
Parts:
- C76: renamed from C401; footprint Capacitor_SMD:C_0603_1608Metric_Pad1.08x0.95mm_HandSolder -> Capacitor_SMD:C_0402_1005Metric_Pad0.74x0.62mm_HandSolder
- R18: renamed from R402; footprint Resistor_SMD:R_0603_1608Metric_Pad0.98x0.95mm_HandSolder -> Resistor_SMD:R_0402_1005Metric_Pad0.72x0.64mm_HandSolder
- renumbered U401 to U11
Changed lines of the file:
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@@
   (symbol (lib_id "Device:R") (at 134.62 74.93 180) (unit 1)
     (in_bom yes) (on_board yes) (dnp no) (fields_autoplaced)
-    (property "Reference" "R402" (at 137.16 73.6599 0)
+    (property "Reference" "R18" (at 137.16 73.6599 0)
       (effects (font (size 1.27 1.27)) (justify right))
     )
@@
       (effects (font (size 1.27 1.27)) (justify right))
     )
-    (property "Footprint" "Resistor_SMD:R_0603_1608Metric_Pad0.98x0.95mm_HandSolder" (at 136.398 74.93 90)
+    (property "Footprint" "Resistor_SMD:R_0402_1005Metric_Pad0.72x0.64mm_HandSolder" (at 136.398 74.93 90)
       (effects (font (size 1.27 1.27)) hide)
     )
@@
       (project "mainboard"
         (path "/e63e39d7-6ac0-4ffd-8aa3-1841a4541b55/90a5bc85-07ac-4ee1-af41-887c984cc4b9/78fa6cb9-f921-4861-9f70-f5ecadaf057b"
-          (reference "R402") (unit 1) (value "10k") (footprint "Resistor_SMD:R_0603_1608Metric_Pad0.98x0.95mm_HandSolder")
+          (reference "R18") (unit 1) (value "10k") (footprint "Resistor_SMD:R_0402_1005Metric_Pad0.72x0.64mm_HandSolder")
         )
       )
@@
   (symbol (lib_id "Memory_Flash:W25Q128JVS") (at 147.32 90.17 0) (unit 1)
     (in_bom yes) (on_board yes) (dnp no) (fields_autoplaced)
-    (property "Reference" "U401" (at 149.3394 77.47 0)
+    (property "Reference" "U11" (at 149.3394 77.47 0)
       (effects (font (size 1.27 1.27)) (justify left))
     )
@@
       (project "mainboard"
         (path "/e63e39d7-6ac0-4ffd-8aa3-1841a4541b55/90a5bc85-07ac-4ee1-af41-887c984cc4b9/78fa6cb9-f921-4861-9f70-f5ecadaf057b"
-          (reference "U401") (unit 1) (value "W25Q128JVS") (footprint "Package_SO:SOIC-8_5.23x5.23mm_P1.27mm")
+          (reference "U11") (unit 1) (value "W25Q128JVS") (footprint "Package_SO:SOIC-8_5.23x5.23mm_P1.27mm")
         )
       )
@@
   (symbol (lib_id "Device:C") (at 165.1 72.39 0) (unit 1)
     (in_bom yes) (on_board yes) (dnp no) (fields_autoplaced)
-    (property "Reference" "C401" (at 168.91 71.1199 0)
+    (property "Reference" "C76" (at 168.91 71.1199 0)
       (effects (font (size 1.27 1.27)) (justify left))
     )
@@
       (effects (font (size 1.27 1.27)) (justify left))
     )
-    (property "Footprint" "Capacitor_SMD:C_0603_1608Metric_Pad1.08x0.95mm_HandSolder" (at 166.0652 76.2 0)
+    (property "Footprint" "Capacitor_SMD:C_0402_1005Metric_Pad0.74x0.62mm_HandSolder" (at 166.0652 76.2 0)
       (effects (font (size 1.27 1.27)) hide)
     )
@@
       (project "mainboard"
         (path "/e63e39d7-6ac0-4ffd-8aa3-1841a4541b55/90a5bc85-07ac-4ee1-af41-887c984cc4b9/78fa6cb9-f921-4861-9f70-f5ecadaf057b"
-          (reference "C401") (unit 1) (value "100n") (footprint "Capacitor_SMD:C_0603_1608Metric_Pad1.08x0.95mm_HandSolder")
+          (reference "C76") (unit 1) (value "100n") (footprint "Capacitor_SMD:C_0402_1005Metric_Pad0.74x0.62mm_HandSolder")
         )
       )

Commit message: working on PCB
Parts:
- renumbered C76 to C72, R18 to R27, U11 to U12
Changed lines of the file:
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@@
-(kicad_sch (version 20221004) (generator eeschema)
+(kicad_sch (version 20221206) (generator eeschema)
   (paper "A4")
   (junction (at 134.62 87.63) (diameter 0) (color 0 0 0 0)
@@
     (effects (font (size 1.27 1.27)) (justify right))
   )
-  (symbol (lib_id "power:GND") (at 147.32 100.33 0) (unit 1)
-    (in_bom yes) (on_board yes) (dnp no) (fields_autoplaced)
-    (property "Reference" "#PWR0190" (at 147.32 106.68 0)
-      (effects (font (size 1.27 1.27)) hide)
-    )
-    (property "Value" "GND" (at 147.32 105.41 0)
-      (effects (font (size 1.27 1.27)))
-    )
-    (property "Footprint" "" (at 147.32 100.33 0)
-      (effects (font (size 1.27 1.27)) hide)
-    )
-    (property "Datasheet" "" (at 147.32 100.33 0)
-      (effects (font (size 1.27 1.27)) hide)
-    )
-    (pin "1")
-    (instances
-      (project "mainboard"
-        (path "/e63e39d7-6ac0-4ffd-8aa3-1841a4541b55/90a5bc85-07ac-4ee1-af41-887c984cc4b9/78fa6cb9-f921-4861-9f70-f5ecadaf057b"
-          (reference "#PWR0190") (unit 1) (value "GND") (footprint "")
-        )
-      )
-    )
-  )
   (symbol (lib_id "Device:R") (at 134.62 74.93 180) (unit 1)
     (in_bom yes) (on_board yes) (dnp no) (fields_autoplaced)
-    (property "Reference" "R18" (at 137.16 73.6599 0)
+    (property "Reference" "R27" (at 137.16 73.6599 0)
       (effects (font (size 1.27 1.27)) (justify right))
     )
@@
       (project "mainboard"
         (path "/e63e39d7-6ac0-4ffd-8aa3-1841a4541b55/90a5bc85-07ac-4ee1-af41-887c984cc4b9/78fa6cb9-f921-4861-9f70-f5ecadaf057b"
-          (reference "R18") (unit 1) (value "10k") (footprint "Resistor_SMD:R_0402_1005Metric_Pad0.72x0.64mm_HandSolder")
+          (reference "R27") (unit 1)
         )
       )
@@
   (symbol (lib_id "Memory_Flash:W25Q128JVS") (at 147.32 90.17 0) (unit 1)
     (in_bom yes) (on_board yes) (dnp no) (fields_autoplaced)
-    (property "Reference" "U11" (at 149.3394 77.47 0)
+    (property "Reference" "U12" (at 149.3394 77.47 0)
       (effects (font (size 1.27 1.27)) (justify left))
     )
@@
       (project "mainboard"
         (path "/e63e39d7-6ac0-4ffd-8aa3-1841a4541b55/90a5bc85-07ac-4ee1-af41-887c984cc4b9/78fa6cb9-f921-4861-9f70-f5ecadaf057b"
-          (reference "U11") (unit 1) (value "W25Q128JVS") (footprint "Package_SO:SOIC-8_5.23x5.23mm_P1.27mm")
+          (reference "U12") (unit 1)
+        )
+      )
+    )
+  )
+  (symbol (lib_name "GND_1") (lib_id "power:GND") (at 147.32 100.33 0) (unit 1)
+    (in_bom yes) (on_board yes) (dnp no) (fields_autoplaced)
+    (property "Reference" "#PWR0182" (at 147.32 106.68 0)
+      (effects (font (size 1.27 1.27)) hide)
+    )
+    (property "Value" "GND" (at 147.32 105.41 0)
+      (effects (font (size 1.27 1.27)))
+    )
+    (property "Footprint" "" (at 147.32 100.33 0)
+      (effects (font (size 1.27 1.27)) hide)
+    )
+    (property "Datasheet" "" (at 147.32 100.33 0)
+      (effects (font (size 1.27 1.27)) hide)
+    )
+    (pin "1")
+    (instances
+      (project "mainboard"
+        (path "/e63e39d7-6ac0-4ffd-8aa3-1841a4541b55/90a5bc85-07ac-4ee1-af41-887c984cc4b9/78fa6cb9-f921-4861-9f70-f5ecadaf057b"
+          (reference "#PWR0182") (unit 1)
         )
       )
@@
   (symbol (lib_id "Device:C") (at 165.1 72.39 0) (unit 1)
     (in_bom yes) (on_board yes) (dnp no) (fields_autoplaced)
-    (property "Reference" "C76" (at 168.91 71.1199 0)
+    (property "Reference" "C72" (at 168.91 71.1199 0)
       (effects (font (size 1.27 1.27)) (justify left))
     )
@@
       (project "mainboard"
         (path "/e63e39d7-6ac0-4ffd-8aa3-1841a4541b55/90a5bc85-07ac-4ee1-af41-887c984cc4b9/78fa6cb9-f921-4861-9f70-f5ecadaf057b"
-          (reference "C76") (unit 1) (value "100n") (footprint "Capacitor_SMD:C_0402_1005Metric_Pad0.74x0.62mm_HandSolder")
+          (reference "C72") (unit 1)
         )
       )
@@
       (project "mainboard"
         (path "/e63e39d7-6ac0-4ffd-8aa3-1841a4541b55/90a5bc85-07ac-4ee1-af41-887c984cc4b9"
-          (reference "#PWR?") (unit 1) (value "+3V3_MCU") (footprint "")
-        )
-        (path "/e63e39d7-6ac0-4ffd-8aa3-1841a4541b55/90a5bc85-07ac-4ee1-af41-887c984cc4b9/78fa6cb9-f921-4861-9f70-f5ecadaf057b"
-          (reference "#PWR0201") (unit 1) (value "+3V3_MCU") (footprint "")
+          (reference "#PWR?") (unit 1)
+        )
+        (path "/e63e39d7-6ac0-4ffd-8aa3-1841a4541b55/90a5bc85-07ac-4ee1-af41-887c984cc4b9/78fa6cb9-f921-4861-9f70-f5ecadaf057b"
+          (reference "#PWR0201") (unit 1)
         )
       )
@@
       (project "mainboard"
         (path "/e63e39d7-6ac0-4ffd-8aa3-1841a4541b55/90a5bc85-07ac-4ee1-af41-887c984cc4b9/78fa6cb9-f921-4861-9f70-f5ecadaf057b"
-          (reference "#PWR0189") (unit 1) (value "GND") (footprint "")
-        )
-      )
+          (reference "#PWR0189") (unit 1)
+        )
+      )

Commit message: prepared first versions of PCBs
Parts:
- added C65: 100n, Capacitor_SMD:C_0402_1005Metric_Pad0.74x0.62mm_HandSolder, symbol Device:C
- added R31: 10k, Resistor_SMD:R_0402_1005Metric_Pad0.72x0.64mm_HandSolder, symbol Device:R
- added U10: W25Q128JVS, Package_SO:SOIC-8_5.23x5.23mm_P1.27mm, symbol Memory_Flash:W25Q128JVS
Connections:
- net +3V3_MCU: now also C65.1, R31.2, U10.8 (VCC)
- net GND: now also C65.2, U10.4 (GND)
- net FLASH.CSN renamed QSPI.CSN0
- net FLASH.SCLK renamed QSPI.SCLK
- net QSPI.SCLK: now also U10.6 (CLK)
- net FLASH.SD0 renamed QSPI.SD0
- net QSPI.SD0: now also U10.5 (DI(IO0))
- net FLASH.SD1 renamed QSPI.SD1
- net QSPI.SD1: now also U10.2 (DO(IO1))
- net FLASH.SD2 renamed QSPI.SD2
- net QSPI.SD2: now also U10.3 (IO2)
- net FLASH.SD3 renamed QSPI.SD3
- net QSPI.SD3: now also U10.7 (IO3)
- new net QSPI.CSN1: R31.1, U10.1 (~{CS})
