File: mainboard/mainboard/north_bridge_bus_multiplexer.kicad_sch (KiCad schematic)
At the start: 4 parts, among them IC502 SN74HCS138PWR, IC503 SN74HCS138PWR

Commit message: working on new pcb
Parts:
- C77: renamed from C502; footprint Capacitor_SMD:C_0603_1608Metric_Pad1.08x0.95mm_HandSolder -> Capacitor_SMD:C_0402_1005Metric_Pad0.74x0.62mm_HandSolder
- C78: renamed from C503; footprint Capacitor_SMD:C_0603_1608Metric_Pad1.08x0.95mm_HandSolder -> Capacitor_SMD:C_0402_1005Metric_Pad0.74x0.62mm_HandSolder
- IC4: renamed from IC502; footprint SOP65P640X120-16N -> footprints:SOP65P640X120-16N
- IC5: renamed from IC503; footprint SOP65P640X120-16N -> footprints:SOP65P640X120-16N
Connections:
- net BUS_CS#B1 is gone; now on net BUS_CS#B2: IC5.13 (Y2)
- net BUS_CTRL.CS10 is gone; now on net BUS_CTRL.CS#0: IC5.1 (A0)
- net BUS_CTRL.CS11 is gone; now on net BUS_CTRL.CS#1: IC5.2 (A1)
- net BUS_CTRL.CS12 is gone; now on net BUS_CTRL.CS#2: IC5.3 (A2)
- net +3V3_MCU: no longer IC4.6 (G2), IC5.6 (G2)
- net BUS_CS#A0: now also IC4.15 (Y0); no longer IC4.14 (Y1)
- net BUS_CS#A1: now also IC4.14 (Y1); no longer IC4.13 (Y2)
- net BUS_CS#A2: now also IC4.13 (Y2); no longer IC4.12 (Y3)
- net BUS_CS#A3: now also IC4.12 (Y3); no longer IC4.11 (Y4)
- net BUS_CS#A4: now also IC4.11 (Y4); no longer IC4.10 (Y5)
- net BUS_CS#A5: now also IC4.10 (Y5); no longer IC4.9 (Y6)
- net BUS_CS#A6: now also IC4.9 (Y6); no longer IC4.7 (Y7)
- net BUS_CS#B2: no longer IC5.12 (Y3)
- net BUS_CS#B3: now also IC5.12 (Y3); no longer IC5.11 (Y4)
- net BUS_CS#B4: now also IC5.11 (Y4); no longer IC5.10 (Y5)
- net BUS_CS#B6: now reaches IC5.9 (Y6)
- net BUS_CS#B0: no longer names the net of IC5.14 (Y1)
- net BUS_CTRL.CS00 renamed BUS_CTRL.CS#0
- net BUS_CTRL.CS01 renamed BUS_CTRL.CS#1
- net BUS_CTRL.CS02 renamed BUS_CTRL.CS#2
- new net BUS_CS#B5: IC5.10 (Y5)
- new net BUS_CTRL.CS#A_EN: IC4.6 (G2)
- new net BUS_CTRL.CS#B_EN: IC5.6 (G2)

Commit message: working on PCB
Parts:
- removed C77, C78: 100n, Capacitor_SMD:C_0402_1005Metric_Pad0.74x0.62mm_HandSolder, symbol Device:C
- removed IC4, IC5: SN74HCS138PWR, footprints:SOP65P640X120-16N, symbol SN74HCS138PWR:SN74HCS138PWR
- added C73: 100n, Capacitor_SMD:C_0402_1005Metric_Pad0.74x0.62mm_HandSolder, symbol Device:C
- added U10: SN74LVC139APWR, Package_SO:TSSOP-16_4.4x5mm_P0.65mm, symbol sn74:SN74LVC139APWR
Connections:
- net +3V3_MCU: now also C73.1, U10.16 (VCC)
- net BUS_CS#A0: now also U10.7 (1Y3)
- net BUS_CS#A1: now also U10.6 (1Y2)
- net BUS_CS#A2: now also U10.5 (1Y1)
- net BUS_CS#A3: now also U10.4 (1Y0)
- net BUS_CS#B2: now also U10.10 (2Y2)
- net BUS_CS#B3: now also U10.9 (2Y3)
- net BUS_CTRL.CS#0: now also U10.2 (1A)
- net BUS_CTRL.CS#1: now also U10.3 (1B)
- net BUS_CTRL.CS#2: now also U10.14 (2A)
- net BUS_CTRL.CS#A_EN: now also U10.1 (1G#)
- net BUS_CTRL.CS#B_EN: now also U10.15 (2G#)
- net GND: now also C73.2, U10.8 (GND)
- new net BUS_CS#B0: U10.12 (2Y0)
- new net BUS_CS#B1: U10.11 (2Y1)
- new net BUS_CTRL.CS#3: U10.13 (2B)
- no-connect marks 4 -> 0

Commit message: prepared first versions of PCBs
Parts:
- renumbered U10 to U13
