File: mainboard/mainboard/south_bridge.kicad_sch (KiCad schematic)
At the start: 15 parts, among them U201 RP2040

Commit message: working on new pcb
Parts:
- added C213: 100n, Capacitor_SMD:C_0402_1005Metric_Pad0.74x0.62mm_HandSolder, symbol Device:C
- added R2, R3: 27.4R, Resistor_SMD:R_0402_1005Metric_Pad0.72x0.64mm_HandSolder, symbol Device:R
- C203, C204, C205, C206, C207, C208, C209, C210, C211, C212, C213: footprint Capacitor_SMD:C_0603_1608Metric_Pad1.08x0.95mm_HandSolder -> Capacitor_SMD:C_0402_1005Metric_Pad0.74x0.62mm_HandSolder
- R202: footprint Resistor_SMD:R_0603_1608Metric_Pad0.98x0.95mm_HandSolder -> Resistor_SMD:R_0402_1005Metric_Pad0.72x0.64mm_HandSolder
- S201: footprint SW_PTS636_SM43J_SMTR_LFS -> footprints:SW_PTS636_SM43J_SMTR_LFS
- U201: footprint QFN40P700X700X90-57N -> footprints:QFN40P700X700X90-57N
- renumbered D1 to D11
Connections:
- net +3V3_SOUTH: now also C213.1
- net AUDIO.BCLK: no longer U201.32 (GPIO21)
- net AUDIO.DIN: no longer U201.29 (GPIO18)
- net AUDIO.DOUT: no longer U201.30 (GPIO19)
- net AUDIO.MCLK: no longer U201.31 (GPIO20)
- net AUDIO.RESET#: no longer U201.35 (GPIO23)
- net AUDIO.WCLK: no longer U201.34 (GPIO22)
- net BUS_SOUTH.CLK: now also U201.29 (GPIO18); no longer U201.4 (GPIO2)
- net BUS_SOUTH.D0: now also U201.30 (GPIO19); no longer U201.5 (GPIO3)
- net BUS_SOUTH.D1: now also U201.31 (GPIO20); no longer U201.6 (GPIO4)
- net BUS_SOUTH.D2: now also U201.32 (GPIO21); no longer U201.7 (GPIO5)
- net BUS_SOUTH.D3: now also U201.34 (GPIO22); no longer U201.8 (GPIO6)
- net GND: now also C213.2
- net USB_D-: now reaches U201.46 (USB_DM)
- net USB_D-: now also R2.1
- net USB_D+: now reaches U201.47 (USB_DP)
- net USB_D+: now also R3.1
- new net USB.D+: R3.2
- new net USB.D-: R2.2
- no-connect marks 5 -> 3
Other:
- added sheet USB Hub (usb_hub.kicad_sch)
- moved on the sheet: C203, C204, C205, C206, C207, C208, C209, C210, C211, C212, C213

Commit message: working on PCB
Parts:
- removed S201: PTS636_SM43J_SMTR_LFS, footprints:SW_PTS636_SM43J_SMTR_LFS, symbol PTS636_SM43J_SMTR_LFS:PTS636_SM43J_SMTR_LFS
- added C207: 100n, Capacitor_SMD:C_0402_1005Metric_Pad0.74x0.62mm_HandSolder, symbol Device:C
- added J5: Conn_01x02_Male, Connector_PinHeader_2.54mm:PinHeader_1x02_P2.54mm_Vertical, symbol Connector:Conn_01x02_Male
- added R2, R3: 4.7k, Resistor_SMD:R_0603_1608Metric_Pad0.98x0.95mm_HandSolder, symbol Device:R
Connections:
- net BUS_DET.OUT is gone; now on net SDIO.D3: U201.40 (GPIO28/ADC2)
- net +3V3_SOUTH: now also C207.1, R2.2, R3.2; no longer C205.1
- net +5V_VBUS: now also C205.1
- net AUDIO.BCLK: now also U201.7 (GPIO5)
- net AUDIO.DIN: now also U201.5 (GPIO3)
- net AUDIO.DOUT: now also U201.4 (GPIO2)
- net AUDIO.MCLK: now also U201.8 (GPIO6)
- net AUDIO.RESET#: now also U201.9 (GPIO7)
- net AUDIO.WCLK: now also U201.6 (GPIO4)
- net BUS.CONTROL0: now also U201.13 (GPIO10); no longer U201.36 (GPIO24)
- net BUS.CONTROL1: now also U201.14 (GPIO11); no longer U201.37 (GPIO25)
- net BUS.CONTROL2: now also U201.15 (GPIO12); no longer U201.38 (GPIO26/ADC0)
- net BUS_RE#.IN: now also U201.16 (GPIO13); no longer U201.39 (GPIO27/ADC1)
- net BUS_SOUTH.CLK: now also U201.28 (GPIO17); no longer U201.29 (GPIO18)
- net BUS_SOUTH.D0: now also U201.29 (GPIO18); no longer U201.30 (GPIO19)
- net BUS_SOUTH.D1: now also U201.30 (GPIO19); no longer U201.31 (GPIO20)
- net BUS_SOUTH.D2: now also U201.31 (GPIO20); no longer U201.32 (GPIO21)
- net BUS_SOUTH.D3: now also U201.32 (GPIO21); no longer U201.34 (GPIO22)
- net GND: now also C207.2
- net I2C.SCL: now also R2.1
- net I2C.SDA: now also R3.1
- net POWER_BUTTON: now also U201.27 (GPIO16), J5.2 (Pin_2); no longer U201.18 (GPIO15)
- net POWER_ENABLE: now also U201.18 (GPIO15); no longer U201.27 (GPIO16)
- net POWER_LED_DATA: now also U201.34 (GPIO22); no longer U201.28 (GPIO17)
- net SDIO.CLK: now also U201.35 (GPIO23); no longer U201.9 (GPIO7)
- net SDIO.CMD: now also U201.36 (GPIO24); no longer U201.13 (GPIO10)
- net SDIO.D0: now also U201.37 (GPIO25); no longer U201.14 (GPIO11)
- net SDIO.D1: now also U201.38 (GPIO26/ADC0); no longer U201.15 (GPIO12)
- net SDIO.D2: now also U201.39 (GPIO27/ADC1); no longer U201.16 (GPIO13)
- net SDIO.D3: no longer U201.17 (GPIO14)
- net at R202.1: now also J5.1 (Pin_1)
- net BUS_INT.OUT: no longer names the net of U201.41 (GPIO29/ADC3)
- new net BUS_DET_OUT: U201.17 (GPIO14)
- no-connect marks 3 -> 4
Other:
- sheet Main bus control ports: added BUS_DET{IN[0..4]}, BUS_INT{IN[0..2]}, BUS_RE#{OUT[0..4]}; removed BUS_DET{IN[0..6]}, BUS_INT_OUT, BUS_INT{IN[0..6]}, BUS_RE#{OUT[0..6]}
- moved on the sheet: R202

Commit message: Mainboard rev 1.0a prepared
Parts:
- removed D11: WS2812B, LED_SMD:LED_WS2812B_PLCC4_5.0x5.0mm_P3.2mm, symbol LED:WS2812B
- added J18: Conn_01x03_Male, Connector_PinHeader_2.54mm:PinHeader_1x03_P2.54mm_Vertical, symbol Connector:Conn_01x03_Male
- R2, R3: footprint Resistor_SMD:R_0603_1608Metric_Pad0.98x0.95mm_HandSolder -> Resistor_SMD:R_0402_1005Metric_Pad0.72x0.64mm_HandSolder
Connections:
- net +3V3_SOUTH: no longer R2.2, R3.2
- net +5V_VBUS: now also J18.2 (Pin_2)
- net GND: now also J18.1 (Pin_1)
- net POWER_LED_DATA: now also J18.3 (Pin_3)
- new net +3V3_BUS: R2.2, R3.2
- no-connect marks 4 -> 3
Other:
- moved on the sheet: C205

Commit message: version 1.0
Connections:
- net FLASH.SD3: now reaches U201.51 (QSPI_SD3)
- net FLASH.SD2: now reaches U201.54 (QSPI_SD2)
- no-connect marks 3 -> 1
Other:
- sheet South Bridge Flash ports: added FLASH{SD[0..3] SCLK CS#}; removed FLASH{SD0 SD1 SCLK CS#}
Changed lines of the file:
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@@
   (junction (at 265.43 35.56) (diameter 0) (color 0 0 0 0)
   )
-  (no_connect (at 134.62 104.14))
-  (no_connect (at 134.62 101.6))
   (no_connect (at 134.62 154.94))
   (bus_entry (at 148.59 93.98) (size -2.54 2.54)
@@
     (stroke (width 0) (type default))
   )
+  (bus_entry (at 148.59 101.6) (size -2.54 2.54)
+    (stroke (width 0) (type default))
+  )
   (bus_entry (at 52.07 154.94) (size 2.54 -2.54)
     (stroke (width 0) (type default))
@@
     (stroke (width 0) (type default))
   )
+  (bus_entry (at 148.59 99.06) (size -2.54 2.54)
+    (stroke (width 0) (type default))
+  )
   (bus_entry (at 243.84 151.13) (size -2.54 2.54)
     (stroke (width 0) (type default))
@@
     (stroke (width 0) (type default))
   )
+  (wire (pts (xy 134.62 104.14) (xy 146.05 104.14))
+    (stroke (width 0) (type default))
+  )
   (wire (pts (xy 69.85 128.27) (xy 71.12 128.27))
     (stroke (width 0) (type default))
@@
     (stroke (width 0) (type default))
   )
+  (bus (pts (xy 148.59 99.06) (xy 148.59 101.6))
+    (stroke (width 0) (type default))
+  )
   (wire (pts (xy 64.77 109.22) (xy 88.9 109.22))
     (stroke (width 0) (type default))
   )
-  (bus (pts (xy 148.59 96.52) (xy 148.59 104.14))
+  (bus (pts (xy 148.59 96.52) (xy 148.59 99.06))
     (stroke (width 0) (type default))
   )
@@
     (stroke (width 0) (type default))
   )
+  (bus (pts (xy 148.59 101.6) (xy 148.59 104.14))
+    (stroke (width 0) (type default))
+  )
   (wire (pts (xy 176.53 144.78) (xy 177.8 144.78))
     (stroke (width 0) (type default))
@@
     (stroke (width 0) (type default))
   )
+  (wire (pts (xy 134.62 101.6) (xy 146.05 101.6))
+    (stroke (width 0) (type default))
+  )
   (wire (pts (xy 139.7 165.1) (xy 134.62 165.1))
     (stroke (width 0) (type default))
@@
     (effects (font (size 1.27 1.27)) (justify right bottom))
   )
+  (label "FLASH.SD2" (at 134.62 101.6 0) (fields_autoplaced)
+    (effects (font (size 1.27 1.27)) (justify left bottom))
+  )
   (label "SDIO.D3" (at 134.62 152.4 0) (fields_autoplaced)
     (effects (font (size 1.27 1.27)) (justify left bottom))
@@
   )
   (label "POWER_BUTTON" (at 134.62 121.92 0) (fields_autoplaced)
+    (effects (font (size 1.27 1.27)) (justify left bottom))
+  )
+  (label "FLASH.SD3" (at 134.62 104.14 0) (fields_autoplaced)
     (effects (font (size 1.27 1.27)) (justify left bottom))
   )
@@
       (effects (font (size 1.27 1.27)) (justify left top))
     )
-    (pin "FLASH{SD0 SD1 SCLK CS#}" bidirectional (at 190.5 80.01 180)
-      (effects (font (size 1.27 1.27)) (justify left))
-    )
+    (pin "FLASH{SD[0..3] SCLK CS#}" bidirectional (at 190.5 80.01 180)
+      (effects (font (size 1.27 1.27)) (justify left))
+    )

Commit message: prepared first versions of PCBs
Parts:
- removed C205: 100n, Capacitor_SMD:C_0402_1005Metric_Pad0.74x0.62mm_HandSolder, symbol Device:C
- removed J18: Conn_01x03_Male, Connector_PinHeader_2.54mm:PinHeader_1x03_P2.54mm_Vertical, symbol Connector:Conn_01x03_Male
- removed J5: Conn_01x02_Male, Connector_PinHeader_2.54mm:PinHeader_1x02_P2.54mm_Vertical, symbol Connector:Conn_01x02_Male
- removed R2, R3: 27.4R, Resistor_SMD:R_0402_1005Metric_Pad0.72x0.64mm_HandSolder, symbol Device:R
- removed R202: 1k, Resistor_SMD:R_0402_1005Metric_Pad0.72x0.64mm_HandSolder, symbol Device:R
- renumbered C203 to C45, C207 to C46, C207 to C47, C204 to C48, C209 to C49, C206 to C50, C210 to C51, C208 to C52, C211 to C53, C212 to C54, C213 to C55, C213 to C56, R2 to R17, R3 to R18, U201 to U8
Connections:
- net BUS_SOUTH.CLK: no longer U8.28 (GPIO17)
- net BUS_SOUTH.D0: no longer U8.29 (GPIO18)
- net BUS_SOUTH.D1: no longer U8.30 (GPIO19)
- net BUS_SOUTH.D2: no longer U8.31 (GPIO20)
- net BUS_SOUTH.D3: no longer U8.32 (GPIO21)
- net USB_D+: no longer names the net of U8.47 (USB_DP)
- net USB_D-: no longer names the net of U8.46 (USB_DM)
Other:
- removed sheet Audio DAC
- removed sheet Bus south connectors
- removed sheet Main bus control
- removed sheet SD Card
- removed sheet USB Hub
- note removed: "Board Input/Output"
