File: mainboard/mainboard/usb_hub.kicad_sch (KiCad schematic)
At the start: 18 parts, among them U10 hs8836a

Commit message: working on new pcb
Parts:
- renumbered C72 to C41, C73 to C42, C74 to C43, D2 to D1, D11 to D10, D3 to D2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

Commit message: working on PCB
Parts:
- renumbered J2 to J3, J3 to J4, R8 to R15, R9 to R16
Connections:
- net +3V3_SOUTH is gone; now on net +3V3_USB_HUB: C41.1, C42.1, U7.14 (V33)
- net +3V3_MCU renamed +3V3_USB_HUB

Commit message: prepared first versions of PCBs
Parts:
- renumbered R15 to R19, R16 to R20
