File: mainboard/mainboard/rp2350_core.kicad_sch (KiCad schematic)
At the start: 29 parts, among them J1 Conn_01x02_Male, J16 Conn_01x02_Male, J5 Conn_01x03_Male, U11 RP2350_80QFN, Y1 ECS-120-8-36-CGN-TR

Commit message: bumped up kicad to v10
Parts:
- Y1: DESCRIPTION The minature ECX-2236 is a compact SMD Crystal. The industr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 -> (none)
