File: mainboard/mainboard/rp2350_core.kicad_sch (KiCad schematic)
At the start: 29 parts, among them J1 Conn_01x02_Male, J16 Conn_01x02_Male, J5 Conn_01x03_Male, U11 RP2350_80QFN, Y1 ECS-120-8-36-CGN-TR

Commit message: Share KiCad libraries, update v2.5 mainboard schematics
- Move every board's symbols, footprints and 3D models into libs/ and point
  the projects' lib tables there; add the mspc design-block library.
- Mainboard: new debug probe, MSPC bus and power connector sheets; drop the
  old shared-bus, south/north bridge and SD card sheets.
- Remove orphaned sheets from the GPU cards and the simulation sandbox.
- Rewrite the v2.5 plan, document libs/ in the README, ignore KiCad 10
  restore backups.

Co-Authored-By: Claude Opus 5 (1M context) <noreply@anthropic.com>
Parts:
- removed J1, J16: Conn_01x02_Male, Connector_PinHeader_2.54mm:PinHeader_1x02_P2.54mm_Vertical, symbol Connector:Conn_01x02_Male
- removed J5: Conn_01x03_Male, Connector_PinHeader_2.54mm:PinHeader_1x03_P2.54mm_Vertical, symbol Connector:Conn_01x03_Male
- removed R21: 1k, Resistor_SMD:R_0402_1005Metric_Pad0.72x0.64mm_HandSolder, symbol Device:R
- removed Y1: ECS-120-8-36-CGN-TR, footprints:XTAL_ECS-120-8-36-CGN-TR, symbol ECS-120-8-36-CGN-TR:ECS-120-8-36-CGN-TR
- added C207: 10u, Capacitor_SMD:C_0402_1005Metric_Pad0.74x0.62mm_HandSolder, symbol Device:C
- added C213, C220: 100n, Capacitor_SMD:C_0402_1005Metric_Pad0.74x0.62mm_HandSolder, symbol Device:C
- added J201, J202: JST_SH_BM02B-SRSS-TB, footprints:JST_SH_BM02B-SRSS-TB_1x02-1MP_P1.00mm_Vertical, symbol mspc_connectors:JST_SH_BM02B-SRSS-TB
- added J203: JST_SH_BM03B-SRSS-TB, footprints:JST_SH_BM03B-SRSS-TB_1x03-1MP_P1.00mm_Vertical, symbol mspc_connectors:JST_SH_BM03B-SRSS-TB
- added J204: Micro_SD_Card, Connector_Card:microSD_HC_Wuerth_693072010801, symbol Connector:Micro_SD_Card
- added R201: 1k, Resistor_SMD:R_0402_1005Metric_Pad0.72x0.64mm_HandSolder, symbol Device:R
- added R206, R207, R208, R209: 10k, Resistor_SMD:R_0402_1005Metric_Pad0.72x0.64mm_HandSolder, symbol Device:R
- added U202: W25Q128JVS, Package_SO:SOIC-8_5.3x5.3mm_P1.27mm, symbol Memory_Flash:W25Q128JVS
- added U203: ESP_PSRAM64, Package_SO:SOIC-8_5.3x5.3mm_P1.27mm, symbol Memory_Flash:W25Q128JVS
- added Y201: ABM8-272-T3, Crystal:Crystal_SMD_3225-4Pin_3.2x2.5mm, symbol mspc_xtal:ABM8-272-T3
- renumbered C74 to C201, C44 to C202, C75 to C203, C1 to C204, C71 to C205, C2 to C206, C3 to C208, C4 to C209, C5 to C210, C6 to C211, C7 to C212, C8 to C214, C9 to C215, C10 to C216, C11 to C217, C12 to C218, C13 to C219, C14 to C221, L3 to L201, R25 to R202, R1 to R203, R15 to R204, R16 to R205, U11 to U201
Connections:
- net BUS.CONTROL2 is gone; now on net POWER_LED_DATA: U201.53 (GPIO42_ADC2)
- net BUS_NORTH.CLK0 is gone; now on net AUDIO.DIN: U201.13 (GPIO14)
- net POWER_ENABLE is gone; now on net POWER_BUTTON: U201.54 (GPIO43_ADC3)
- net +5V_VBUS: now also J203.2 (Pin_2)
- net AUDIO.DIN: no longer U201.1 (GPIO4)
- net GND: now also C207.2, C213.2, C220.2, J201.2 (Pin_2), J201.MP (MountPin), J203.3 (Pin_3), J203.MP (MountPin), J204.6 (VSS), J204.SH (SHIELD), U202.4 (GND), U203.4 (GND), Y201.2 (G), Y201.4 (G)
- net MCU_RESET#: now also J201.1 (Pin_1)
- net OSC_IN: now also Y201.1
- net POWER_BUTTON: now also J202.2 (Pin_2); no longer U201.47 (GPIO38)
- net POWER_LED_DATA: now also J203.1 (Pin_1); no longer U201.48 (GPIO39)
- net SDIO.CLK: now also J204.5 (CLK)
- net SDIO.CMD: now also J204.3 (CMD)
- net SDIO.D0: now also J204.7 (DAT0)
- net SDIO.D1: now also J204.8 (DAT1), R208.2
- net SDIO.D2: now also J204.1 (DAT2), R207.2
- net SDIO.D3: now also J204.2 (DAT3/CD)
- net USB.D+: now also R204.2; no longer R205.2
- net USB.D-: now also R205.2; no longer R204.2
- net USB_D+: now also R204.1, U201.67 (USB_DP); no longer R205.1, U201.66 (USB_DM)
- net USB_D-: now also R205.1, U201.66 (USB_DM); no longer R204.1, U201.67 (USB_DP)
- net at C206.1, R203.1: now also Y201.3
- net +3V3_MCU renamed +3V3
- net +3V3: now also C207.1, C213.1, C220.1, J204.4 (VDD), R201.1, R206.2, R207.1, R208.1, R209.2, U202.8 (VCC), U203.8 (VCC)
- net AUDIO.BCLK renamed BUS_CARD0.D6
- net AUDIO.DOUT renamed BUS_CARD0.D2
- net AUDIO.MCLK renamed BUS_CARD0.D5
- net AUDIO.WCLK renamed BUS_CARD0.D4
- net BUS.CONTROL0 renamed CARD_2_EN
- net BUS.CONTROL1 renamed VBUS_EN
- net BUS_CS#A0 renamed BUS_CARD0.CS#
- net BUS_CS#A1 renamed AUDIO.BCK
- net BUS_CS#A2 renamed BUS_CARD0.INT#
- net BUS_CS#A3 renamed BUS_CARD0.RST#
- net BUS_CS#B0 renamed BUS_CARD0.D7
- net BUS_CS#B1 renamed BUS_CARD0.CLK
- net BUS_DET_OUT: no longer names the net of U201.57 (GPIO46_ADC6)
- net BUS_NORTH.CLK1 renamed AUDIO.LRCK
- net BUS_NORTH.D0 renamed BUS_CARD1.D0
- net BUS_NORTH.D1 renamed BUS_CARD1.CS#
- net BUS_NORTH.D10 renamed BUS_CARD2.CLK
- net BUS_NORTH.D11 renamed BUS_CARD2.INT#
- net BUS_NORTH.D12 renamed BUS_CARD2.RST#
- net BUS_NORTH.D13 renamed BUS_CARD2.CS#
- net BUS_NORTH.D14 renamed PRIMARY_POWER_FAULT#
- net BUS_NORTH.D15 renamed SECONDARY_POWER_FAULT#
- net BUS_NORTH.D2 renamed BUS_CARD1.CLK
- net BUS_NORTH.D3 renamed BUS_CARD1.D1
- net BUS_NORTH.D4 renamed BUS_CARD1.INT#
- net BUS_NORTH.D5 renamed BUS_CARD1.RST#
- net BUS_NORTH.D6 renamed BUS_CARD2.D0
- net BUS_NORTH.D7 renamed BUS_CARD2.D1
- net BUS_NORTH.D8 renamed BUS_CARD2.D2
- net BUS_NORTH.D9 renamed BUS_CARD2.D3
- net BUS_RE#.IN: no longer names the net of U201.58 (GPIO47_ADC7)
- net DEBUG.SWCLK renamed SWD.CLK
- net DEBUG.SWD renamed SWD.DIO
- net I2C.SCL renamed BUS_CARD0.D0
- net I2C.SDA renamed BUS_CARD0.D1
- net QSPI.CSN0 renamed QSPI_CSN0
- net QSPI_CSN0: now also R206.1, U202.1 (~{CS})
- net QSPI.CSN1 renamed QSPI_CSN1
- net QSPI_CSN1: now also R209.1, U203.1 (~{CS})
- net QSPI.SCLK renamed QSPI_SCLK
- net QSPI_SCLK: now also U202.6 (CLK), U203.6 (CLK)
- net QSPI.SD0 renamed QSPI_SD0
- net QSPI_SD0: now also U202.5 (DI/IO_{0}), U203.5 (DI/IO_{0})
- net QSPI.SD1 renamed QSPI_SD1
- net QSPI_SD1: now also U202.2 (DO/IO_{1}), U203.2 (DO/IO_{1})
- net QSPI.SD2 renamed QSPI_SD2
- net QSPI_SD2: now also U202.3 (~{WP}/IO_{2}), U203.3 (~{WP}/IO_{2})
- net QSPI.SD3 renamed QSPI_SD3
- net QSPI_SD3: now also U202.7 (~{HOLD}/~{RESET}/IO_{3}), U203.7 (~{HOLD}/~{RESET}/IO_{3})
- net UART.RX renamed UART_DEBUG.TX
- net UART.TX renamed UART_DEBUG.RX
- new net: J202.1 (Pin_1), R201.2
- new net BUS_CARD0.D3: U201.1 (GPIO4)
- new net CARD_0_EN: U201.47 (GPIO38)
- new net CARD_1_EN: U201.48 (GPIO39)
- no-connect marks 0 -> 3
Other:
- removed sheet Audio DAC
- removed sheet MCU Connectors
- removed sheet MCU flash
- removed sheet Main bus control
- removed sheet SD Card
- removed sheet USB Hub
- moved on the sheet: C204, C206, R203

Commit message: Mainboard v3: schematic review fixes
New sheets for the housekeeping bus: TCA6408A expander, INA226/INA3221
power measurement and the MCP7940N RTC with a CR1220 backup cell.

Correctness:
- RTC load caps C241/C242 are 6.8 pF C0G 0402 (were a relay footprint).
- L50 is the AOTA-B201610S3R3-101-T with pin 1 on +1V1_MCU; U52 is an
  APS1604M-3SQR-SN on a 150-mil SOP-8.
- I2S is DIN=GPIO13, BCK=GPIO14, LRCK=GPIO15, as pico-extras audio_i2s
  expects. Expander INT# goes to GPIO42.
- ADC_AVDD filter (FB50, C74, C75), 33 ohm on SDIO CLK, SD ESD (U53/U54),
  PSRAM 1 uF, POWER_BUTTON 10 k pull-up, 10 uF at the SY6280 inputs.
- J_DBG: USBLC6-4SC6 on the probe USB, 47 uF polymer on +5V_DBG against
  charger overvoltage spikes, and bleeders on both USB-C VBUS inputs and
  on +5V_DBG.
- Power symbols point at their matching project_power symbols.

Parts and fields:
- Part numbers and LCSC codes for the purchased parts: push-push microSD
  J53, HRO USB-C J1/J2, stacked USB-A J90/J91, TLV70033DDCR, and others.
- Voltage, dielectric and tolerance fields on every capacitor and a
  tolerance on every resistor; the field is named "LCSC" everywhere.
- Hand-solder footprint variants where KiCad has one.

Drawing:
- References renumbered into the per-sheet ranges.
- Net names on the USB, crystal, DAC, CC and ISET nets; netclass
  patterns updated.
- No four-way junctions left.
- Notes for the slot pin 1 marking, J120 and firmware bring-up.

ERC is clean with all rules enabled.

Co-Authored-By: Claude Opus 5 (1M context) <noreply@anthropic.com>
Parts:
- removed C202: 100n, Capacitor_SMD:C_0402_1005Metric_Pad0.74x0.62mm_HandSolder, symbol Device:C
- removed L201: 3.3u, Inductor_SMD:L_0805_2012Metric, symbol Device:L
- removed R201: 1k, Resistor_SMD:R_0402_1005Metric_Pad0.72x0.64mm_HandSolder, symbol Device:R
- removed U203: ESP_PSRAM64, Package_SO:SOIC-8_5.3x5.3mm_P1.27mm, symbol Memory_Flash:W25Q128JVS
- added C52, C53, C54, C73, C74, C76, C77, C78, C79: 100n, Capacitor_SMD:C_0402_1005Metric_Pad0.74x0.62mm_HandSolder, symbol Device:C
- added C75, C80: 1u, Capacitor_SMD:C_0402_1005Metric_Pad0.74x0.62mm_HandSolder, symbol Device:C
- added FB50: 600R@100MHz, Inductor_SMD:L_0402_1005Metric_Pad0.77x0.64mm_HandSolder, symbol Device:FerriteBead
- added L50: AOTA-B201610S3R3-101-T, footprints:L_Abracon_AOTA-B201610S_Polarity, symbol mspc_power:AOTA-B201610S3R3-101-T
- added R50, R51: 100, Resistor_SMD:R_0402_1005Metric_Pad0.72x0.64mm_HandSolder, symbol Device:R
- added R58, R59, R60, R65, R69: 10k, Resistor_SMD:R_0402_1005Metric_Pad0.72x0.64mm_HandSolder, symbol Device:R
- added R63, R64: 4.7k, Resistor_SMD:R_0402_1005Metric_Pad0.72x0.64mm_HandSolder, symbol Device:R
- added R66, R67: 220, Resistor_SMD:R_0402_1005Metric_Pad0.72x0.64mm_HandSolder, symbol Device:R
- added R68: 33, Resistor_SMD:R_0402_1005Metric_Pad0.72x0.64mm_HandSolder, symbol Device:R
- added TP50: TestPoint, TestPoint:TestPoint_THTPad_D1.5mm_Drill0.7mm, symbol Connector:TestPoint
- added U52: APS1604M-3SQRx-SN, Package_SO:SOIC-8_3.9x4.9mm_P1.27mm, symbol Memory_RAM:APS1604M-3SQRx-SN
- added U53, U54: USBLC6-4SC6, Package_TO_SOT_SMD:SOT-23-6_Handsoldering, symbol Power_Protection:USBLC6-4SC6
- C50: renamed from C201; Dielectric (none) -> X5R; Tolerance (none) -> 10%; Voltage (none) -> 10V
- C51: renamed from C203; Dielectric (none) -> X5R; Tolerance (none) -> 10%; Voltage (none) -> 10V
- C55: renamed from C204; Dielectric (none) -> C0G; Tolerance (none) -> 5%; Voltage (none) -> 10V
- C56: renamed from C205; Dielectric (none) -> X5R; Tolerance (none) -> 10%; Voltage (none) -> 10V
- C57: renamed from C206; Dielectric (none) -> C0G; Tolerance (none) -> 5%; Voltage (none) -> 10V
- C58: renamed from C207; footprint Capacitor_SMD:C_0402_1005Metric_Pad0.74x0.62mm_HandSolder -> Capacitor_SMD:C_1206_3216Metric_Pad1.33x1.80mm_HandSolder; Dielectric (none) -> X5R; LCSC (none) -> C9807; MPN (none) -> CL31A106KAHNNNE; Tolerance (none) -> 10%; Voltage (none) -> 25V
- C59: renamed from C208; Dielectric (none) -> X7R; Tolerance (none) -> 10%; Voltage (none) -> 16V
- C60: renamed from C209; Dielectric (none) -> X7R; Tolerance (none) -> 10%; Voltage (none) -> 16V
- C61: renamed from C210; Dielectric (none) -> X5R; Tolerance (none) -> 10%; Voltage (none) -> 10V
- C62: renamed from C213; Dielectric (none) -> X7R; Tolerance (none) -> 10%; Voltage (none) -> 16V
- C63: renamed from C211; Dielectric (none) -> X7R; Tolerance (none) -> 10%; Voltage (none) -> 16V
- C64: renamed from C212; Dielectric (none) -> X7R; Tolerance (none) -> 10%; Voltage (none) -> 16V
- C65: renamed from C214; Dielectric (none) -> X7R; Tolerance (none) -> 10%; Voltage (none) -> 16V
- C66: renamed from C215; Dielectric (none) -> X7R; Tolerance (none) -> 10%; Voltage (none) -> 16V
- C67: renamed from C216; Dielectric (none) -> X7R; Tolerance (none) -> 10%; Voltage (none) -> 16V
- C68: renamed from C217; Dielectric (none) -> X7R; Tolerance (none) -> 10%; Voltage (none) -> 16V
- C69: renamed from C218; Dielectric (none) -> X7R; Tolerance (none) -> 10%; Voltage (none) -> 16V
- C70: renamed from C220; Dielectric (none) -> X7R; Tolerance (none) -> 10%; Voltage (none) -> 16V
- C71: renamed from C219; Dielectric (none) -> X7R; Tolerance (none) -> 10%; Voltage (none) -> 16V
- C72: renamed from C221; Dielectric (none) -> X7R; Tolerance (none) -> 10%; Voltage (none) -> 16V
- J53: renamed from J204; value Micro_SD_Card -> DM3AT-SF-PEJM5; footprint Connector_Card:microSD_HC_Wuerth_693072010801 -> Connector_Card:microSD_HC_Hirose_DM3AT-SF-PEJM5; LCSC (none) -> C114218; MPN (none) -> DM3AT-SF-PEJM5; Manufacturer (none) -> Hirose
- R52: renamed from R202; LCSC (none) -> C25105; MPN (none) -> 0402WGF330JTCE; Tolerance (none) -> 1%
- R53: renamed from R203; Tolerance (none) -> 1%
- R54: renamed from R204; value 27.4R -> 27.4; Tolerance (none) -> 1%
- R55: renamed from R205; value 27.4R -> 27.4; Tolerance (none) -> 1%
- R56: renamed from R206; Tolerance (none) -> 1%
- R57: renamed from R207; Tolerance (none) -> 1%
- R61: renamed from R208; Tolerance (none) -> 1%
- R62: renamed from R209; Tolerance (none) -> 1%
- U50: renamed from U201; LCSC (none) -> C42415655; MPN (none) -> RP2350B; Manufacturer (none) -> Raspberry Pi
- U51: renamed from U202; LCSC (none) -> C97521; MPN (none) -> W25Q128JVSIQ; Manufacturer (none) -> Winbond
- Y50: renamed from Y201; footprint Crystal:Crystal_SMD_3225-4Pin_3.2x2.5mm -> Crystal:Crystal_SMD_3225-4Pin_3.2x2.5mm_HandSoldering; LCSC (none) -> C20625731
- renumbered J201 to J50, J202 to J51, J203 to J52
Connections:
- net +1V1_MCU: now also C52.1, L50.1, TP50.1
- net +3V3: now also C73.1, C76.1, C77.1, C78.2, C79.2, C80.1, FB50.1, R58.1, R59.1, R60.1, R63.2, R64.2, R65.2, R69.1, U52.8 (VDD), U53.5 (VBUS), U54.5 (VBUS); no longer U50.59 (ADC_AVDD)
- net AUDIO.BCK: now also U50.13 (GPIO14); no longer U50.12 (GPIO13)
- net AUDIO.DIN: now also U50.12 (GPIO13); no longer U50.13 (GPIO14)
- net GND: now also J51.2 (Pin_2), J51.MP (MountPin), C52.2, C53.2, C54.2, C73.2, C74.2, C75.2, C76.2, C77.2, C78.1, C79.1, C80.2, U52.4 (VSS), U53.2 (GND), U54.2 (GND)
- net MCU_RESET#: now also C53.1, R50.2; no longer J50.1 (Pin_1)
- net POWER_BUTTON: now also C54.1, R51.2, R69.2; no longer J51.2 (Pin_2)
- net QSPI_CSN1: now also U52.1 (~{CE})
- net QSPI_SCLK: now also U52.6 (SCLK)
- net QSPI_SD0: now also U52.5 (SI/SIO0)
- net QSPI_SD1: now also U52.2 (SO/SIO1)
- net QSPI_SD2: now also U52.3 (SIO2)
- net QSPI_SD3: now also U52.7 (SIO3)
- net SDIO.CLK: now also R68.2, U54.3 (I/O2); no longer U50.40 (GPIO32)
- net SDIO.CMD: now also R60.2, U54.1 (I/O1)
- net SDIO.D0: now also R58.2, U53.1 (I/O1)
- net SDIO.D1: now also U53.3 (I/O2)
- net SDIO.D2: now also U53.4 (I/O3)
- net SDIO.D3: now also R59.2, U53.6 (I/O4)
- net VREG_LX: now also L50.2
- net POWER_BTN: now reaches J51.1 (Pin_1)
- net POWER_BTN: now also R51.1
- net OSC_XO: now reaches C57.1, R53.1, Y50.3
- net I2C.SDA: now reaches U50.57 (GPIO46_ADC6)
- net I2C.SDA: now also R63.1
- net I2C.SCL: now reaches U50.58 (GPIO47_ADC7)
- net I2C.SCL: now also R64.1
- net +5V_VBUS renamed PANEL_LED2
- net PANEL_LED2: now also R67.1
- net CARD_0_EN renamed POWER_LED
- net POWER_LED: now also R66.2
- net CARD_1_EN renamed STATUS_LED
- net STATUS_LED: now also R67.2
- net CARD_2_EN renamed USB1_CC
- net POWER_LED_DATA renamed EXPANDER.INT#
- net EXPANDER.INT#: now also R65.1; no longer J52.1 (Pin_1)
- net PRIMARY_POWER_FAULT# renamed PWR_CARD.PV
- net SECONDARY_POWER_FAULT# renamed PWR_CARD.TC
- net UART_DEBUG.RX renamed UART_DEBUG.MCU_TX
- net UART_DEBUG.TX renamed UART_DEBUG.MCU_RX
- net USB_D+ renamed USB_MCU_D+
- net USB_D- renamed USB_MCU_D-
- net VBUS_EN renamed USB2_CC
- new net: R68.1, U50.40 (GPIO32)
- new net ADC_AVDD: C74.1, C75.1, FB50.2, U50.59 (ADC_AVDD)
- new net PANEL_LED1: J52.1 (Pin_1), R66.1
- new net RESET_BTN: J50.1 (Pin_1), R50.1
- no-connect marks 3 -> 2
Other:
- note added: "Firmware notes: GPIO40/41 ADC: disable digital input (RP2350-E9) GPIO43 POWER_BUTTON: R69 10k pull-up (pin resets pulled down) I2S: DATA=GPIO13, BCK=GPIO14, LRCK=GPIO15"
- moved on the sheet: C58, C62, C70, J51, R57, R61, R62

Commit message: Mainboard: title blocks for v3
Every schematic sheet and the PCB carry the same title block: "MSPC
mainboard", rev 3, 2026-09-13. The root sheet still said rev 1 from
2022, and most sheets had none.

Co-Authored-By: Claude Opus 5 (1M context) <noreply@anthropic.com>
Other:
- company: (none) -> Mateusz Stadnik
- title: MSPC -> MSPC mainboard
Changed lines of the file:
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@@
 	(paper "A4")
 	(title_block
-		(title "MSPC")
-		(rev "1")
+		(title "MSPC mainboard")
+		(date "2026-09-13")
+		(rev "3")
+		(company "Mateusz Stadnik")
 	)
 	(rectangle
