File: mainboard/mainboard/debug_probe.kicad_sch (KiCad schematic)
At the start: 48 parts, among them J801 JST_SH_BM03B-SRSS-TB, SW801 USB_BOOT, SW802 PROBE_RESET#, U801 TLV70033_SOT23-5, U802 W25Q128JVS, U803 RP2040, U804 74AUP1T17GW, U805 74AUP1T17GW, Y801 ABM8-272-T3

Commit message: Mainboard v3: schematic review fixes
New sheets for the housekeeping bus: TCA6408A expander, INA226/INA3221
power measurement and the MCP7940N RTC with a CR1220 backup cell.

Correctness:
- RTC load caps C241/C242 are 6.8 pF C0G 0402 (were a relay footprint).
- L50 is the AOTA-B201610S3R3-101-T with pin 1 on +1V1_MCU; U52 is an
  APS1604M-3SQR-SN on a 150-mil SOP-8.
- I2S is DIN=GPIO13, BCK=GPIO14, LRCK=GPIO15, as pico-extras audio_i2s
  expects. Expander INT# goes to GPIO42.
- ADC_AVDD filter (FB50, C74, C75), 33 ohm on SDIO CLK, SD ESD (U53/U54),
  PSRAM 1 uF, POWER_BUTTON 10 k pull-up, 10 uF at the SY6280 inputs.
- J_DBG: USBLC6-4SC6 on the probe USB, 47 uF polymer on +5V_DBG against
  charger overvoltage spikes, and bleeders on both USB-C VBUS inputs and
  on +5V_DBG.
- Power symbols point at their matching project_power symbols.

Parts and fields:
- Part numbers and LCSC codes for the purchased parts: push-push microSD
  J53, HRO USB-C J1/J2, stacked USB-A J90/J91, TLV70033DDCR, and others.
- Voltage, dielectric and tolerance fields on every capacitor and a
  tolerance on every resistor; the field is named "LCSC" everywhere.
- Hand-solder footprint variants where KiCad has one.

Drawing:
- References renumbered into the per-sheet ranges.
- Net names on the USB, crystal, DAC, CC and ISET nets; netclass
  patterns updated.
- No four-way junctions left.
- Notes for the slot pin 1 marking, J120 and firmware bring-up.

ERC is clean with all rules enabled.

Co-Authored-By: Claude Opus 5 (1M context) <noreply@anthropic.com>
Parts:
- removed R801: 0, Resistor_SMD:R_0402_1005Metric_Pad0.72x0.64mm_HandSolder, symbol Device:R
- removed R812: 100, Resistor_SMD:R_0402_1005Metric_Pad0.72x0.64mm_HandSolder, symbol Device:R
- removed U802: W25Q128JVS, Package_SO:SOIC-8_5.3x5.3mm_P1.27mm, symbol Memory_Flash:W25Q128JVS
- added Q120, Q121: 2N7002, Package_TO_SOT_SMD:SOT-23_Handsoldering, symbol Transistor_FET:2N7002
- added R136, R137, R138, R139: 100k, Resistor_SMD:R_0402_1005Metric_Pad0.72x0.64mm_HandSolder, symbol Device:R
- added R140: 2.2k, Resistor_SMD:R_0402_1005Metric_Pad0.72x0.64mm_HandSolder, symbol Device:R
- added TP122, TP124: TestPoint, TestPoint:TestPoint_THTPad_D1.5mm_Drill0.7mm, symbol Connector:TestPoint
- added U121: W25Q16JVSS, Package_SO:SOIC-8_5.3x5.3mm_P1.27mm, symbol Memory_Flash:W25Q16JVSS
- C120: renamed from C802; footprint Capacitor_SMD:C_0402_1005Metric -> Capacitor_SMD:C_0402_1005Metric_Pad0.74x0.62mm_HandSolder; Dielectric (none) -> C0G; Tolerance (none) -> 5%; Voltage (none) -> 10V
- C121: renamed from C801; Dielectric (none) -> X5R; Tolerance (none) -> 10%; Voltage (none) -> 16V
- C122: renamed from C803; footprint Capacitor_SMD:C_0402_1005Metric -> Capacitor_SMD:C_0402_1005Metric_Pad0.74x0.62mm_HandSolder; Dielectric (none) -> X7R; Tolerance (none) -> 10%; Voltage (none) -> 16V
- C123: renamed from C805; footprint Capacitor_SMD:C_0402_1005Metric -> Capacitor_SMD:C_0402_1005Metric_Pad0.74x0.62mm_HandSolder; Dielectric (none) -> X7R; Tolerance (none) -> 10%; Voltage (none) -> 16V
- C124: renamed from C804; footprint Capacitor_SMD:C_0402_1005Metric -> Capacitor_SMD:C_0402_1005Metric_Pad0.74x0.62mm_HandSolder; Dielectric (none) -> C0G; Tolerance (none) -> 5%; Voltage (none) -> 10V
- C125: renamed from C806; footprint Capacitor_SMD:C_0402_1005Metric -> Capacitor_SMD:C_0402_1005Metric_Pad0.74x0.62mm_HandSolder; Dielectric (none) -> X7R; Tolerance (none) -> 10%; Voltage (none) -> 16V
- C126: renamed from C807; Dielectric (none) -> X5R; Tolerance (none) -> 10%; Voltage (none) -> 16V
- C127: renamed from C808; footprint Capacitor_SMD:C_0402_1005Metric -> Capacitor_SMD:C_0402_1005Metric_Pad0.74x0.62mm_HandSolder; Dielectric (none) -> X5R; Tolerance (none) -> 10%; Voltage (none) -> 10V
- C128: renamed from C809; footprint Capacitor_SMD:C_0402_1005Metric -> Capacitor_SMD:C_0402_1005Metric_Pad0.74x0.62mm_HandSolder; Dielectric (none) -> X7R; Tolerance (none) -> 10%; Voltage (none) -> 16V
- C129: renamed from C810; footprint Capacitor_SMD:C_0402_1005Metric -> Capacitor_SMD:C_0402_1005Metric_Pad0.74x0.62mm_HandSolder; Dielectric (none) -> X5R; Tolerance (none) -> 10%; Voltage (none) -> 10V
- C130: renamed from C811; footprint Capacitor_SMD:C_0402_1005Metric -> Capacitor_SMD:C_0402_1005Metric_Pad0.74x0.62mm_HandSolder; Dielectric (none) -> X7R; Tolerance (none) -> 10%; Voltage (none) -> 16V
- C131: renamed from C812; footprint Capacitor_SMD:C_0402_1005Metric -> Capacitor_SMD:C_0402_1005Metric_Pad0.74x0.62mm_HandSolder; Dielectric (none) -> X7R; Tolerance (none) -> 10%; Voltage (none) -> 16V
- C132: renamed from C813; footprint Capacitor_SMD:C_0402_1005Metric -> Capacitor_SMD:C_0402_1005Metric_Pad0.74x0.62mm_HandSolder; Dielectric (none) -> X5R; Tolerance (none) -> 10%; Voltage (none) -> 10V
- C133: renamed from C814; footprint Capacitor_SMD:C_0402_1005Metric -> Capacitor_SMD:C_0402_1005Metric_Pad0.74x0.62mm_HandSolder; Dielectric (none) -> X7R; Tolerance (none) -> 10%; Voltage (none) -> 16V
- C134: renamed from C815; footprint Capacitor_SMD:C_0402_1005Metric -> Capacitor_SMD:C_0402_1005Metric_Pad0.74x0.62mm_HandSolder; Dielectric (none) -> X7R; Tolerance (none) -> 10%; Voltage (none) -> 16V
- C135: renamed from C816; footprint Capacitor_SMD:C_0402_1005Metric -> Capacitor_SMD:C_0402_1005Metric_Pad0.74x0.62mm_HandSolder; Dielectric (none) -> X7R; Tolerance (none) -> 10%; Voltage (none) -> 16V
- R121: renamed from R802; Tolerance (none) -> 1%
- R122: renamed from R803; Tolerance (none) -> 1%
- R123: renamed from R804; Tolerance (none) -> 1%
- R124: renamed from R805; Tolerance (none) -> 1%
- R125: renamed from R806; Tolerance (none) -> 1%
- R126: renamed from R807; Tolerance (none) -> 1%
- R127: renamed from R808; value 1K -> 1k; Tolerance (none) -> 1%
- R128: renamed from R809; Tolerance (none) -> 1%
- R129: renamed from R810; Tolerance (none) -> 1%
- R130: renamed from R814; Tolerance (none) -> 1%
- R131: renamed from R815; Tolerance (none) -> 1%
- R132: renamed from R816; Tolerance (none) -> 1%
- R133: renamed from R811; Tolerance (none) -> 1%
- R135: renamed from R813; Tolerance (none) -> 1%
- SW120: renamed from SW801; LCSC (none) -> C720477; MPN (none) -> TS-1088-AR02016
- SW121: renamed from SW802; LCSC (none) -> C720477; MPN (none) -> TS-1088-AR02016
- U120: renamed from U801; footprint Package_TO_SOT_SMD:SOT-23-5 -> Package_TO_SOT_SMD:SOT-23-5_HandSoldering; LCSC (none) -> C11337; MPN (none) -> TLV70033DDCR; Manufacturer (none) -> Texas Instruments
- U122: renamed from U803; LCSC (none) -> C2040; MPN (none) -> RP2040; Manufacturer (none) -> Raspberry Pi
- Y120: renamed from Y801; footprint Crystal:Crystal_SMD_3225-4Pin_3.2x2.5mm -> Crystal:Crystal_SMD_3225-4Pin_3.2x2.5mm_HandSoldering; LCSC (none) -> C20625731
- renumbered D801 to D120, D802 to D121, D803 to D122, D804 to D123, D805 to D124, J801 to J120, TP801 to TP120, TP802 to TP121, U805 to U123, U804 to U124
Connections:
- net +3V3_PROBE: now also TP122.1, U121.8 (VCC)
- net +5V_DBG: now also U120.3 (EN), R140.2, TP124.1
- net GND: now also Q120.2 (S), Q121.2 (S), R137.1, R138.1, R139.1, R140.1, U121.4 (GND)
- net QSPI_SCLK: now also U121.6 (CLK)
- net QSPI_SD0: now also U121.5 (DI/IO_{0})
- net QSPI_SD1: now also U121.2 (DO/IO_{1})
- net QSPI_SD2: now also U121.3 (~{WP}/IO_{2})
- net QSPI_SD3: now also U121.7 (~{HOLD}/~{RESET}/IO_{3})
- net QSPI_SS: now also U121.1 (~{CS})
- net XO_XTAL: now reaches C124.2, R126.1, Y120.3
- net MCU_TX_BUF_IN: now reaches R135.2, U124.2 (A)
- net GPIO10: now reaches U122.13 (GPIO10)
- net GPIO10: now also Q120.1 (G), R138.2
- net GPIO11: now reaches U122.14 (GPIO11)
- net GPIO11: now also Q121.1 (G), R139.2
- net at U122.38 (GPIO26/ADC0): now also R136.1, R137.2
- net SWDIO_BUF_IN: now reaches R132.2, U123.2 (A)
- net BOOTSEL: now reaches R127.2, SW120.2 (B), TP121.1
- net GPIO6: no longer names the net of U122.8 (GPIO6)
- net UART_DEBUG.RX renamed UART_DEBUG.MCU_TX
- net UART_DEBUG.TX renamed UART_DEBUG.MCU_RX
- new net +3V3: R136.2
- new net MCU_RESET#: Q121.3 (D)
- new net POWER_OFF#: Q120.3 (D)
- no-connect marks 19 -> 17
Other:
- note added: "J120: RP2040 UART0 1 TX (GPIO0), 2 GND, 3 RX (GPIO1)"

Commit message: Mainboard: title blocks for v3
Every schematic sheet and the PCB carry the same title block: "MSPC
mainboard", rev 3, 2026-09-13. The root sheet still said rev 1 from
2022, and most sheets had none.

Co-Authored-By: Claude Opus 5 (1M context) <noreply@anthropic.com>
Other:
- company: (none) -> Mateusz Stadnik
- title: (none) -> MSPC mainboard
Changed lines of the file:
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@@
 	(generator_version "10.0")
 	(paper "A4")
+	(title_block
+		(title "MSPC mainboard")
+		(date "2026-09-13")
+		(rev "3")
+		(company "Mateusz Stadnik")
+	)
 	(text "J120: RP2040 UART0\n1 TX (GPIO0), 2 GND, 3 RX (GPIO1)"
 		(exclude_from_sim no)
