File: mainboard/mainboard/expander.kicad_sch (KiCad schematic)
At the start: 3 parts, among them U200 TCA6408APW

Commit message: Mainboard: title blocks for v3
Every schematic sheet and the PCB carry the same title block: "MSPC
mainboard", rev 3, 2026-09-13. The root sheet still said rev 1 from
2022, and most sheets had none.

Co-Authored-By: Claude Opus 5 (1M context) <noreply@anthropic.com>
Other:
- company: (none) -> Mateusz Stadnik
- title: (none) -> MSPC mainboard
Changed lines of the file:
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@@
 	(generator_version "10.0")
 	(paper "A4")
+	(title_block
+		(title "MSPC mainboard")
+		(date "2026-09-13")
+		(rev "3")
+		(company "Mateusz Stadnik")
+	)
 	(junction
 		(at 146.05 90.17)
