File: mainboard/mainboard/mspc_bus.kicad_sch (KiCad schematic)
At the start: 9 parts, among them J1101 Card 0 8-bit, J1102 Card 1 2-bit, J1103 Card 2 4-bit

Commit message: Mainboard v3: schematic review fixes
New sheets for the housekeeping bus: TCA6408A expander, INA226/INA3221
power measurement and the MCP7940N RTC with a CR1220 backup cell.

Correctness:
- RTC load caps C241/C242 are 6.8 pF C0G 0402 (were a relay footprint).
- L50 is the AOTA-B201610S3R3-101-T with pin 1 on +1V1_MCU; U52 is an
  APS1604M-3SQR-SN on a 150-mil SOP-8.
- I2S is DIN=GPIO13, BCK=GPIO14, LRCK=GPIO15, as pico-extras audio_i2s
  expects. Expander INT# goes to GPIO42.
- ADC_AVDD filter (FB50, C74, C75), 33 ohm on SDIO CLK, SD ESD (U53/U54),
  PSRAM 1 uF, POWER_BUTTON 10 k pull-up, 10 uF at the SY6280 inputs.
- J_DBG: USBLC6-4SC6 on the probe USB, 47 uF polymer on +5V_DBG against
  charger overvoltage spikes, and bleeders on both USB-C VBUS inputs and
  on +5V_DBG.
- Power symbols point at their matching project_power symbols.

Parts and fields:
- Part numbers and LCSC codes for the purchased parts: push-push microSD
  J53, HRO USB-C J1/J2, stacked USB-A J90/J91, TLV70033DDCR, and others.
- Voltage, dielectric and tolerance fields on every capacitor and a
  tolerance on every resistor; the field is named "LCSC" everywhere.
- Hand-solder footprint variants where KiCad has one.

Drawing:
- References renumbered into the per-sheet ranges.
- Net names on the USB, crystal, DAC, CC and ISET nets; netclass
  patterns updated.
- No four-way junctions left.
- Notes for the slot pin 1 marking, J120 and firmware bring-up.

ERC is clean with all rules enabled.

Co-Authored-By: Claude Opus 5 (1M context) <noreply@anthropic.com>
Parts:
- added R150, R151, R152, R153, R154, R161, R174, R175, R176: 7.5k, Resistor_SMD:R_0402_1005Metric_Pad0.72x0.64mm_HandSolder, symbol Device:R
- added R155, R156, R157, R158, R159, R160, R162, R163, R164, R165, R166, R167, R168, R169, R170, R171, R172, R173, R177, R178, R179, R180, R181, R182, R183, R184: 33, Resistor_SMD:R_0402_1005Metric_Pad0.72x0.64mm_HandSolder, symbol Device:R
- C150: renamed from C1101; Dielectric (none) -> X5R; LCSC (none) -> C9807; MPN (none) -> CL31A106KAHNNNE; Tolerance (none) -> 10%; Voltage (none) -> 25V
- C151: renamed from C1102; Dielectric (none) -> X7R; Tolerance (none) -> 10%; Voltage (none) -> 16V
- C152: renamed from C1103; Dielectric (none) -> X5R; LCSC (none) -> C9807; MPN (none) -> CL31A106KAHNNNE; Tolerance (none) -> 10%; Voltage (none) -> 25V
- C153: renamed from C1104; Dielectric (none) -> X7R; Tolerance (none) -> 10%; Voltage (none) -> 16V
- C154: renamed from C1105; Dielectric (none) -> X5R; LCSC (none) -> C9807; MPN (none) -> CL31A106KAHNNNE; Tolerance (none) -> 10%; Voltage (none) -> 25V
- C155: renamed from C1106; Dielectric (none) -> X7R; Tolerance (none) -> 10%; Voltage (none) -> 16V
- renumbered J1101 to J150, J1102 to J151, J1103 to J152
Connections:
- net BUS_CARD0.CLK: now also R166.1; no longer J150.18 (Pin_18)
- net BUS_CARD0.CS#: now also R150.2, R159.1; no longer J150.15 (Pin_15)
- net BUS_CARD0.D0: now also R162.1; no longer J150.14 (Pin_14)
- net BUS_CARD0.D1: now also R155.1; no longer J150.13 (Pin_13)
- net BUS_CARD0.D2: now also R163.1; no longer J150.12 (Pin_12)
- net BUS_CARD0.D3: now also R156.1; no longer J150.11 (Pin_11)
- net BUS_CARD0.D4: now also R164.1; no longer J150.8 (Pin_8)
- net BUS_CARD0.D5: now also R157.1; no longer J150.7 (Pin_7)
- net BUS_CARD0.D6: now also R165.1; no longer J150.6 (Pin_6)
- net BUS_CARD0.D7: now also R158.1; no longer J150.5 (Pin_5)
- net BUS_CARD0.INT#: now also R152.2, R160.1; no longer J150.20 (Pin_20)
- net BUS_CARD0.RST#: now also R151.2, R167.1; no longer J150.19 (Pin_19)
- net BUS_CARD1.CLK: now also R170.1; no longer J151.14 (Pin_14)
- net BUS_CARD1.CS#: now also R153.2, R171.1; no longer J151.11 (Pin_11)
- net BUS_CARD1.D0: now also R168.1; no longer J151.8 (Pin_8)
- net BUS_CARD1.D1: now also R169.1; no longer J151.7 (Pin_7)
- net BUS_CARD1.INT#: now also R161.2, R173.1; no longer J151.16 (Pin_16)
- net BUS_CARD1.RST#: now also R154.2, R172.1; no longer J151.15 (Pin_15)
- net BUS_CARD2.CLK: now also R183.1; no longer J152.14 (Pin_14)
- net BUS_CARD2.CS#: now also R174.2, R179.1; no longer J152.11 (Pin_11)
- net BUS_CARD2.D0: now also R181.1; no longer J152.8 (Pin_8)
- net BUS_CARD2.D1: now also R177.1; no longer J152.7 (Pin_7)
- net BUS_CARD2.D2: now also R182.1; no longer J152.6 (Pin_6)
- net BUS_CARD2.D3: now also R178.1; no longer J152.5 (Pin_5)
- net BUS_CARD2.INT#: now also R176.2, R180.1; no longer J152.16 (Pin_16)
- net BUS_CARD2.RST#: now also R175.2, R184.1; no longer J152.15 (Pin_15)
- net GND: now also R150.1, R151.1, R152.1, R153.1, R154.1, R161.1, R174.1, R175.1, R176.1
- new net BUS_CARD0_CLK: J150.18 (Pin_18), R166.2
- new net BUS_CARD0_CS#: J150.15 (Pin_15), R159.2
- new net BUS_CARD0_D0: J150.14 (Pin_14), R162.2
- new net BUS_CARD0_D1: J150.13 (Pin_13), R155.2
- new net BUS_CARD0_D2: J150.12 (Pin_12), R163.2
- new net BUS_CARD0_D3: J150.11 (Pin_11), R156.2
- new net BUS_CARD0_D4: J150.8 (Pin_8), R164.2
- new net BUS_CARD0_D5: J150.7 (Pin_7), R157.2
- new net BUS_CARD0_D6: J150.6 (Pin_6), R165.2
- new net BUS_CARD0_D7: J150.5 (Pin_5), R158.2
- new net BUS_CARD0_INT#: J150.20 (Pin_20), R160.2
- new net BUS_CARD0_RST#: J150.19 (Pin_19), R167.2
- new net BUS_CARD1_CLK: J151.14 (Pin_14), R170.2
- new net BUS_CARD1_CS#: J151.11 (Pin_11), R171.2
- new net BUS_CARD1_D0: J151.8 (Pin_8), R168.2
- new net BUS_CARD1_D1: J151.7 (Pin_7), R169.2
- new net BUS_CARD1_INT#: J151.16 (Pin_16), R173.2
- new net BUS_CARD1_RST#: J151.15 (Pin_15), R172.2
- new net BUS_CARD2_CLK: J152.14 (Pin_14), R183.2
- new net BUS_CARD2_CS#: J152.11 (Pin_11), R179.2
- new net BUS_CARD2_D0: J152.8 (Pin_8), R181.2
- new net BUS_CARD2_D1: J152.7 (Pin_7), R177.2
- new net BUS_CARD2_D2: J152.6 (Pin_6), R182.2
- new net BUS_CARD2_D3: J152.5 (Pin_5), R178.2
- new net BUS_CARD2_INT#: J152.16 (Pin_16), R180.2
- new net BUS_CARD2_RST#: J152.15 (Pin_15), R184.2
Other:
- note added: "v3 slot pinout - not compatible with v2 cards. Sockets are unkeyed: mark pin 1 on the board and card silkscreen."

Commit message: Mainboard: title blocks for v3
Every schematic sheet and the PCB carry the same title block: "MSPC
mainboard", rev 3, 2026-09-13. The root sheet still said rev 1 from
2022, and most sheets had none.

Co-Authored-By: Claude Opus 5 (1M context) <noreply@anthropic.com>
Other:
- company: (none) -> Mateusz Stadnik
- title: (none) -> MSPC mainboard
Changed lines of the file:
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@@
 	(generator_version "10.0")
 	(paper "A4")
+	(title_block
+		(title "MSPC mainboard")
+		(date "2026-09-13")
+		(rev "3")
+		(company "Mateusz Stadnik")
+	)
 	(rectangle
 		(start 19.05 24.13)
