File: fpga_extension/fpga_extension/fpga_qspi.kicad_sch (KiCad schematic)
At the start: 4 parts

Commit message: refactored mainboard schematic
Parts:
- removed U?: LFE5U-25F-6BG381x, Package_BGA:Lattice_caBGA-381_17.0x17.0mm_Layout20x20_P0.8mm_Ball0.4mm_Pad0.4mm_NSMD, symbol fpga_extension_library:LFE5U-25F-6BG381x
- added U6: LFE5UM-85F-6BG381x, Package_BGA:Lattice_caBGA-381_17.0x17.0mm_Layout20x20_P0.8mm_Ball0.4mm_Pad0.4mm_NSMD, symbol FPGA_Lattice:LFE5UM-85F-6BG381x
Connections:
- net VCC: now also U6.F10 (VCCIO0), U6.F9 (VCCIO0)
- new net QSPI1.CE#: U6.A6 (PT4A)
- new net QSPI1.IO0: U6.E6 (PT6A)
- new net QSPI1.IO1: U6.D6 (PT6B)
- new net QSPI1.IO2: U6.E7 (PT9A)
- new net QSPI1.IO3: U6.D7 (PT9B)
- new net QSPI1.SCLK: U6.B6 (PT4B)
- new net QSPI2.CE#: U6.C6 (PT11A)
- new net QSPI2.IO0: U6.E8 (PT13A)
- new net QSPI2.IO1: U6.D8 (PT13B)
- new net QSPI2.IO2: U6.C8 (PT15A)
- new net QSPI2.IO3: U6.B8 (PT15B)
- new net QSPI2.SCLK: U6.C7 (PT11B)
