File: fpga_extension/fpga_extension/fpga_unused.kicad_sch (KiCad schematic)
At the start: 10 parts

Commit message: refactored mainboard schematic
Parts:
- removed U? (x2): LFE5U-25F-6BG381x, Package_BGA:Lattice_caBGA-381_17.0x17.0mm_Layout20x20_P0.8mm_Ball0.4mm_Pad0.4mm_NSMD, symbol fpga_extension_library:LFE5U-25F-6BG381x
- added U6: LFE5UM-85F-6BG381x, Package_BGA:Lattice_caBGA-381_17.0x17.0mm_Layout20x20_P0.8mm_Ball0.4mm_Pad0.4mm_NSMD, symbol FPGA_Lattice:LFE5UM-85F-6BG381x
Connections:
- net VCC: now also U6.H6 (VCCIO7), U6.H7 (VCCIO7), U6.J6 (VCCIO7), U6.L6 (VCCIO6), U6.L7 (VCCIO6), U6.M6 (VCCIO6)
- no-connect marks 66 -> 65
