File: fpga_extension/fpga_extension/connector.kicad_sch (KiCad schematic)
At the start: 1 part, among them J1 Conn_02x16_Odd_Even

Commit message: prepared first versions of PCBs
Parts:
- removed J1: Conn_02x16_Odd_Even, Connector_PinHeader_2.00mm:PinHeader_2x16_P2.00mm_Vertical, symbol Connector_Generic:Conn_02x16_Odd_Even
- added J4: Connector A 16-bit, Connector_PinHeader_1.27mm:PinHeader_2x15_P1.27mm_Vertical_SMD, symbol Connector_Generic:Conn_02x15_Odd_Even
- added R28: <10k, Resistor_SMD:R_0402_1005Metric_Pad0.72x0.64mm_HandSolder, symbol Device:R
Connections:
- net GND: now also J4.1 (Pin_1), J4.2 (Pin_2), J4.27 (Pin_27), J4.30 (Pin_30)
- new net +3V3_BUS: J4.28 (Pin_28), R28.1
- new net +5V_BUS: J4.25 (Pin_25)
- new net BUS.CLK: J4.19 (Pin_19)
- new net BUS.CS#A0: J4.22 (Pin_22)
- new net BUS.CS#A1: J4.20 (Pin_20)
- new net BUS.D0: J4.18 (Pin_18)
- new net BUS.D1: J4.17 (Pin_17)
- new net BUS.D10: J4.8 (Pin_8)
- new net BUS.D11: J4.7 (Pin_7)
- new net BUS.D12: J4.6 (Pin_6)
- new net BUS.D13: J4.5 (Pin_5)
- new net BUS.D14: J4.4 (Pin_4)
- new net BUS.D15: J4.3 (Pin_3)
- new net BUS.D2: J4.16 (Pin_16)
- new net BUS.D3: J4.15 (Pin_15)
- new net BUS.D4: J4.14 (Pin_14)
- new net BUS.D5: J4.13 (Pin_13)
- new net BUS.D6: J4.12 (Pin_12)
- new net BUS.D7: J4.11 (Pin_11)
- new net BUS.D8: J4.10 (Pin_10)
- new net BUS.D9: J4.9 (Pin_9)
- new net BUS.DET: J4.24 (Pin_24), R28.2
- new net BUS.INT: J4.23 (Pin_23)
- new net BUS.RE#: J4.26 (Pin_26)
- no-connect marks 10 -> 2
