File: gpu_extension/bus_connector.kicad_sch (KiCad schematic)
At the start: 1 part, among them J1 Conn_02x10_Odd_Even

Commit message: prepared first versions of PCBs
Parts:
- added R29: < 10k, Resistor_SMD:R_0402_1005Metric_Pad0.72x0.64mm_HandSolder, symbol Device:R
- renumbered J1 to J3
Connections:
- net +3V3: now also J3.3 (Pin_3), R29.1; no longer J3.14 (Pin_14), J3.18 (Pin_18)
- net +5V: now also J3.6 (Pin_6); no longer J3.15 (Pin_15)
- net BUS.CLK: now also J3.12 (Pin_12); no longer J3.9 (Pin_9)
- net BUS.CS#: now also J3.11 (Pin_11); no longer J3.12 (Pin_12)
- net BUS.D0: now also J3.13 (Pin_13); no longer J3.7 (Pin_7)
- net BUS.D1: now also J3.14 (Pin_14); no longer J3.8 (Pin_8)
- net BUS.D2: now also J3.15 (Pin_15); no longer J3.5 (Pin_5)
- net BUS.D3: now also J3.16 (Pin_16); no longer J3.6 (Pin_6)
- net BUS.D4: now also J3.17 (Pin_17); no longer J3.3 (Pin_3)
- net BUS.D5: now also J3.18 (Pin_18); no longer J3.4 (Pin_4)
- net BUS.D6: now also J3.19 (Pin_19); no longer J3.1 (Pin_1)
- net BUS.D7: now also J3.20 (Pin_20); no longer J3.2 (Pin_2)
- net BUS.RE#: now also J3.5 (Pin_5); no longer J3.13 (Pin_13)
- net GND: now also J3.1 (Pin_1), J3.4 (Pin_4); no longer J3.17 (Pin_17), J3.20 (Pin_20)
- new net BUS.DET#: J3.7 (Pin_7), R29.2
