File: gpu_extension/dvi.kicad_sch (KiCad schematic)
At the start: 9 parts, among them J302 NOT_HDMI_A

Commit message: fixes
Parts:
- added J2: DB15_Female_HighDensity_MountingHoles, Connector_Dsub:DSUB-15-HD_Female_Horizontal_P2.29x1.98mm_EdgePinOffset3.03mm_Housed_MountingHolesOffset4.94mm, symbol Connector:DB15_Female_HighDensity_MountingHoles
- added Q1, Q2, Q3, Q4: BS170F, Package_TO_SOT_SMD:SOT-23, symbol Transistor_FET:BS170F
- added R17, R19, R21, R23, R24, R25, R26, R27: 619, Resistor_SMD:R_0603_1608Metric_Pad0.98x0.95mm_HandSolder, symbol Device:R
- added R18, R20, R28, R29: 309, Resistor_SMD:R_0603_1608Metric_Pad0.98x0.95mm_HandSolder, symbol Device:R
- added R22, R30: 97.6, Resistor_SMD:R_0603_1608Metric_Pad0.98x0.95mm_HandSolder, symbol Device:R
- added R31, R32, R34: 536, Resistor_SMD:R_0603_1608Metric_Pad0.98x0.95mm_HandSolder, symbol Device:R
- added R33, R36: 47, Resistor_SMD:R_0603_1608Metric_Pad0.98x0.95mm_HandSolder, symbol Device:R
- added R35: 267, Resistor_SMD:R_0603_1608Metric_Pad0.98x0.95mm_HandSolder, symbol Device:R
- added R37: 105, Resistor_SMD:R_0603_1608Metric_Pad0.98x0.95mm_HandSolder, symbol Device:R
- added R38, R39, R40, R41: 10k, Resistor_SMD:R_0603_1608Metric_Pad0.98x0.95mm_HandSolder, symbol Device:R
- added R42, R43, R44, R45: 0, Resistor_SMD:R_0402_1005Metric_Pad0.72x0.64mm_HandSolder, symbol Device:R
- R315, R316, R317, R318, R319, R320, R321, R322: footprint Resistor_SMD:R_0603_1608Metric_Pad0.98x0.95mm_HandSolder -> Resistor_SMD:R_0402_1005Metric_Pad0.72x0.64mm_HandSolder
Connections:
- net +5V: now also J2.9, Q2.1 (G), Q4.1 (G), R40.2, R41.2
- net GND: now also J2.0, J2.10, J2.5, J2.6, J2.7, J2.8, R17.1, R22.2, R27.1, R30.2, R34.1, R37.2
- net at J302.15 (SCL): now also R44.1
- net at J302.16 (SDA): now also R45.1
- new net: R17.2, R18.1, R19.2
- new net: R24.2, R27.2, R28.1
- new net: R18.2, R20.1, R21.2
- new net: R25.2, R28.2, R29.1
- new net: J2.12, R42.2
- new net: Q3.3 (D), Q4.3 (D)
- new net: J2.15, R43.2
- new net: Q1.3 (D), Q2.3 (D)
- new net: R31.2, R34.2, R35.1
- new net +3V3: Q1.1 (G), Q3.1 (G), R38.2, R39.2
- new net CEC_I2C_CLOCK: Q4.2 (S), R41.1, R43.1, R44.2
- new net CEC_I2C_DATA: Q2.2 (S), R40.1, R42.1, R45.2
- new net MCU_I2C.CLOCK: Q3.2 (S), R38.1
- new net MCU_I2C.DATA: Q1.2 (S), R39.1
- new net VGA.B0: R31.1
- new net VGA.B1: R32.1
- new net VGA.G0: R24.1
- new net VGA.G1: R25.1
- new net VGA.G2: R26.1
- new net VGA.HSYNC: R33.2
- new net VGA.R0: R19.1
- new net VGA.R1: R21.1
- new net VGA.R2: R23.1
- new net VGA.VSYNC: R36.2
- new net VGA_B: J2.3, R32.2, R35.2, R37.1
- new net VGA_G: J2.2, R26.2, R29.2, R30.1
- new net VGA_HSYNC: J2.13, R33.1
- new net VGA_R: J2.1, R20.2, R22.1, R23.2
- new net VGA_VSYNC: J2.14, R36.1

Commit message: version 1.0
Parts:
- R17, R18, R19, R20, R21, R22, R23, R24, R25, R26, R27, R28, R29, R30, R31, R32, R33, R34, R35, R36, R37, R38, R39, R40, R41: footprint Resistor_SMD:R_0603_1608Metric_Pad0.98x0.95mm_HandSolder -> Resistor_SMD:R_0402_1005Metric_Pad0.72x0.64mm_HandSolder
Changed lines of the file:
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@@
       (effects (font (size 1.27 1.27)))
     )
-    (property "Footprint" "Resistor_SMD:R_0603_1608Metric_Pad0.98x0.95mm_HandSolder" (at 149.86 34.798 90)
+    (property "Footprint" "Resistor_SMD:R_0402_1005Metric_Pad0.72x0.64mm_HandSolder" (at 149.86 34.798 90)
       (effects (font (size 1.27 1.27)) hide)
     )
@@
       (effects (font (size 1.27 1.27)) (justify left))
     )
-    (property "Footprint" "Resistor_SMD:R_0603_1608Metric_Pad0.98x0.95mm_HandSolder" (at 151.892 74.93 90)
+    (property "Footprint" "Resistor_SMD:R_0402_1005Metric_Pad0.72x0.64mm_HandSolder" (at 151.892 74.93 90)
       (effects (font (size 1.27 1.27)) hide)
     )
@@
       (effects (font (size 1.27 1.27)))
     )
-    (property "Footprint" "Resistor_SMD:R_0603_1608Metric_Pad0.98x0.95mm_HandSolder" (at 149.86 44.958 90)
+    (property "Footprint" "Resistor_SMD:R_0402_1005Metric_Pad0.72x0.64mm_HandSolder" (at 149.86 44.958 90)
       (effects (font (size 1.27 1.27)) hide)
     )
@@
       (effects (font (size 1.27 1.27)) (justify left))
     )
-    (property "Footprint" "Resistor_SMD:R_0603_1608Metric_Pad0.98x0.95mm_HandSolder" (at 151.892 85.09 90)
+    (property "Footprint" "Resistor_SMD:R_0402_1005Metric_Pad0.72x0.64mm_HandSolder" (at 151.892 85.09 90)
       (effects (font (size 1.27 1.27)) hide)
     )
@@
       (effects (font (size 1.27 1.27)))
     )
-    (property "Footprint" "Resistor_SMD:R_0603_1608Metric_Pad0.98x0.95mm_HandSolder" (at 148.59 102.108 90)
+    (property "Footprint" "Resistor_SMD:R_0402_1005Metric_Pad0.72x0.64mm_HandSolder" (at 148.59 102.108 90)
       (effects (font (size 1.27 1.27)) hide)
     )
@@
       (effects (font (size 1.27 1.27)) (justify right))
     )
-    (property "Footprint" "Resistor_SMD:R_0603_1608Metric_Pad0.98x0.95mm_HandSolder" (at 102.108 135.89 90)
+    (property "Footprint" "Resistor_SMD:R_0402_1005Metric_Pad0.72x0.64mm_HandSolder" (at 102.108 135.89 90)
       (effects (font (size 1.27 1.27)) hide)
     )
@@
       (effects (font (size 1.27 1.27)) (justify left))
     )
-    (property "Footprint" "Resistor_SMD:R_0603_1608Metric_Pad0.98x0.95mm_HandSolder" (at 151.892 105.41 90)
+    (property "Footprint" "Resistor_SMD:R_0402_1005Metric_Pad0.72x0.64mm_HandSolder" (at 151.892 105.41 90)
       (effects (font (size 1.27 1.27)) hide)
     )
@@
       (effects (font (size 1.27 1.27)))
     )
-    (property "Footprint" "Resistor_SMD:R_0603_1608Metric_Pad0.98x0.95mm_HandSolder" (at 148.59 91.948 90)
+    (property "Footprint" "Resistor_SMD:R_0402_1005Metric_Pad0.72x0.64mm_HandSolder" (at 148.59 91.948 90)
       (effects (font (size 1.27 1.27)) hide)
     )
@@
       (effects (font (size 1.27 1.27)))
     )
-    (property "Footprint" "Resistor_SMD:R_0603_1608Metric_Pad0.98x0.95mm_HandSolder" (at 148.59 81.788 90)
+    (property "Footprint" "Resistor_SMD:R_0402_1005Metric_Pad0.72x0.64mm_HandSolder" (at 148.59 81.788 90)
       (effects (font (size 1.27 1.27)) hide)
     )
@@
       (effects (font (size 1.27 1.27)) (justify left))
     )
-    (property "Footprint" "Resistor_SMD:R_0603_1608Metric_Pad0.98x0.95mm_HandSolder" (at 151.892 95.25 90)
+    (property "Footprint" "Resistor_SMD:R_0402_1005Metric_Pad0.72x0.64mm_HandSolder" (at 151.892 95.25 90)
       (effects (font (size 1.27 1.27)) hide)
     )
@@
       (effects (font (size 1.27 1.27)) (justify left))
     )
-    (property "Footprint" "Resistor_SMD:R_0603_1608Metric_Pad0.98x0.95mm_HandSolder" (at 153.162 48.26 90)
+    (property "Footprint" "Resistor_SMD:R_0402_1005Metric_Pad0.72x0.64mm_HandSolder" (at 153.162 48.26 90)
       (effects (font (size 1.27 1.27)) hide)
     )
@@
       (effects (font (size 1.27 1.27)) (justify left))
     )
-    (property "Footprint" "Resistor_SMD:R_0603_1608Metric_Pad0.98x0.95mm_HandSolder" (at 149.352 121.92 90)
+    (property "Footprint" "Resistor_SMD:R_0402_1005Metric_Pad0.72x0.64mm_HandSolder" (at 149.352 121.92 90)
       (effects (font (size 1.27 1.27)) hide)
     )
@@
       (effects (font (size 1.27 1.27)) (justify left))
     )
-    (property "Footprint" "Resistor_SMD:R_0603_1608Metric_Pad0.98x0.95mm_HandSolder" (at 153.162 38.1 90)
+    (property "Footprint" "Resistor_SMD:R_0402_1005Metric_Pad0.72x0.64mm_HandSolder" (at 153.162 38.1 90)
       (effects (font (size 1.27 1.27)) hide)
     )
@@
       (effects (font (size 1.27 1.27)))
     )
-    (property "Footprint" "Resistor_SMD:R_0603_1608Metric_Pad0.98x0.95mm_HandSolder" (at 146.05 128.778 90)
+    (property "Footprint" "Resistor_SMD:R_0402_1005Metric_Pad0.72x0.64mm_HandSolder" (at 146.05 128.778 90)
       (effects (font (size 1.27 1.27)) hide)
     )
@@
       (effects (font (size 1.27 1.27)))
     )
-    (property "Footprint" "Resistor_SMD:R_0603_1608Metric_Pad0.98x0.95mm_HandSolder" (at 204.47 102.362 90)
+    (property "Footprint" "Resistor_SMD:R_0402_1005Metric_Pad0.72x0.64mm_HandSolder" (at 204.47 102.362 90)
       (effects (font (size 1.27 1.27)) hide)
     )
@@
       (effects (font (size 1.27 1.27)) (justify left))
     )
-    (property "Footprint" "Resistor_SMD:R_0603_1608Metric_Pad0.98x0.95mm_HandSolder" (at 153.162 58.42 90)
+    (property "Footprint" "Resistor_SMD:R_0402_1005Metric_Pad0.72x0.64mm_HandSolder" (at 153.162 58.42 90)
       (effects (font (size 1.27 1.27)) hide)
     )
@@
       (effects (font (size 1.27 1.27)) (justify right))
     )
-    (property "Footprint" "Resistor_SMD:R_0603_1608Metric_Pad0.98x0.95mm_HandSolder" (at 90.678 135.89 90)
+    (property "Footprint" "Resistor_SMD:R_0402_1005Metric_Pad0.72x0.64mm_HandSolder" (at 90.678 135.89 90)
       (effects (font (size 1.27 1.27)) hide)
     )
@@
       (effects (font (size 1.27 1.27)))
     )
-    (property "Footprint" "Resistor_SMD:R_0603_1608Metric_Pad0.98x0.95mm_HandSolder" (at 146.05 138.938 90)
+    (property "Footprint" "Resistor_SMD:R_0402_1005Metric_Pad0.72x0.64mm_HandSolder" (at 146.05 138.938 90)
       (effects (font (size 1.27 1.27)) hide)
     )
@@
       (effects (font (size 1.27 1.27)) (justify left))
     )
-    (property "Footprint" "Resistor_SMD:R_0603_1608Metric_Pad0.98x0.95mm_HandSolder" (at 149.352 142.24 90)
+    (property "Footprint" "Resistor_SMD:R_0402_1005Metric_Pad0.72x0.64mm_HandSolder" (at 149.352 142.24 90)
       (effects (font (size 1.27 1.27)) hide)
     )
@@
       (effects (font (size 1.27 1.27)) (justify right))
     )
-    (property "Footprint" "Resistor_SMD:R_0603_1608Metric_Pad0.98x0.95mm_HandSolder" (at 42.418 135.89 90)
+    (property "Footprint" "Resistor_SMD:R_0402_1005Metric_Pad0.72x0.64mm_HandSolder" (at 42.418 135.89 90)
       (effects (font (size 1.27 1.27)) hide)
     )
@@
       (effects (font (size 1.27 1.27)))
     )
-    (property "Footprint" "Resistor_SMD:R_0603_1608Metric_Pad0.98x0.95mm_HandSolder" (at 204.47 97.282 90)
+    (property "Footprint" "Resistor_SMD:R_0402_1005Metric_Pad0.72x0.64mm_HandSolder" (at 204.47 97.282 90)
       (effects (font (size 1.27 1.27)) hide)
     )
@@
       (effects (font (size 1.27 1.27)))
     )
-    (property "Footprint" "Resistor_SMD:R_0603_1608Metric_Pad0.98x0.95mm_HandSolder" (at 149.86 55.118 90)
+    (property "Footprint" "Resistor_SMD:R_0402_1005Metric_Pad0.72x0.64mm_HandSolder" (at 149.86 55.118 90)
       (effects (font (size 1.27 1.27)) hide)
     )
@@
       (effects (font (size 1.27 1.27)) (justify right))
     )
-    (property "Footprint" "Resistor_SMD:R_0603_1608Metric_Pad0.98x0.95mm_HandSolder" (at 33.528 135.89 90)
+    (property "Footprint" "Resistor_SMD:R_0402_1005Metric_Pad0.72x0.64mm_HandSolder" (at 33.528 135.89 90)
       (effects (font (size 1.27 1.27)) hide)
     )
@@
       (effects (font (size 1.27 1.27)) (justify left))
     )
-    (property "Footprint" "Resistor_SMD:R_0603_1608Metric_Pad0.98x0.95mm_HandSolder" (at 153.162 27.94 90)
+    (property "Footprint" "Resistor_SMD:R_0402_1005Metric_Pad0.72x0.64mm_HandSolder" (at 153.162 27.94 90)
       (effects (font (size 1.27 1.27)) hide)
     )
@@
       (effects (font (size 1.27 1.27)) (justify left))
     )
-    (property "Footprint" "Resistor_SMD:R_0603_1608Metric_Pad0.98x0.95mm_HandSolder" (at 149.352 132.08 90)
-      (effects (font (size 1.27 1.27)) hide)
-    )
+    (property "Footprint" "Resistor_SMD:R_0402_1005Metric_Pad0.72x0.64mm_HandSolder" (at 149.352 132.08 90)
+      (effects (font (size 1.27 1.27)) hide)
+    )

Commit message: prepared first versions of PCBs
Parts:
- removed J302: NOT_HDMI_A, Connector_HDMI:HDMI_A_Molex_208658-1001_Horizontal, symbol Connector:HDMI_A
- removed R315, R316, R317, R318, R319, R320, R321, R322: 270, Resistor_SMD:R_0402_1005Metric_Pad0.72x0.64mm_HandSolder, symbol Device:R
- removed R42, R43, R44, R45: 0, Resistor_SMD:R_0402_1005Metric_Pad0.72x0.64mm_HandSolder, symbol Device:R
- added J1: Conn_02x06_Odd_Even, Connector_PinHeader_1.27mm:PinHeader_2x06_P1.27mm_Vertical_SMD, symbol Connector_Generic:Conn_02x06_Odd_Even
- added R26, R27: 0, Resistor_SMD:R_0402_1005Metric_Pad0.72x0.64mm_HandSolder, symbol Device:R
- renumbered Q3 to Q1, Q1 to Q2, Q4 to Q3, Q2 to Q4, R38 to R1, R19 to R10, R21 to R11, R23 to R12, R34 to R13, R35 to R14, R37 to R15, R27 to R16, R28 to R17, R29 to R18, R30 to R19, R39 to R2, R17 to R20, R18 to R21, R20 to R22, R22 to R23, R33 to R24, R36 to R25, R40 to R3, R41 to R4, R31 to R5, R32 to R6, R24 to R7, R25 to R8, R26 to R9
Connections:
- net +5V: now also J1.1 (Pin_1)
- net CEC_I2C_CLOCK: now also J2.15, J1.9 (Pin_9), R27.1; no longer Q3.2 (S), R4.1
- net CEC_I2C_DATA: now also J2.12, J1.7 (Pin_7), R26.1; no longer Q4.2 (S), R3.1
- net DVI.CK+: now also J1.5 (Pin_5)
- net DVI.CK-: now also J1.3 (Pin_3)
- net DVI.D0+: now also J1.2 (Pin_2)
- net DVI.D0-: now also J1.4 (Pin_4)
- net DVI.D1+: now also J1.6 (Pin_6)
- net DVI.D1-: now also J1.8 (Pin_8)
- net DVI.D2+: now also J1.10 (Pin_10)
- net DVI.D2-: now also J1.12 (Pin_12)
- net GND: now also J1.11 (Pin_11)
- new net: Q3.2 (S), R27.2, R4.1
- new net: Q4.2 (S), R26.2, R3.1
- no-connect marks 5 -> 2
Other:
- note removed: "NOT"
