File: gpu_extension/gpu_extension.kicad_sch (KiCad schematic)
At the start: 18 parts, among them J201 Conn_01x03_Male, U4 RP2040, Y201 ECS-120-8-36-CGN-TR

Commit message: version 1.0
Connections:
- net FLASH.IO3: now reaches U4.51 (QSPI_SD3)
- net FLASH.IO2: now reaches U4.54 (QSPI_SD2)
- no-connect marks 5 -> 3
Other:
- sheet Memory ports: added FLASH{CS# CLK IO[0..3]}; removed FLASH{CS# CLK IO[0..1]}
Changed lines of the file:
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@@
   (junction (at 168.91 34.29) (diameter 0) (color 0 0 0 0)
   )
-  (no_connect (at 179.07 77.47))
   (no_connect (at 179.07 90.17))
-  (no_connect (at 179.07 80.01))
   (no_connect (at 179.07 125.73))
   (no_connect (at 179.07 87.63))
@@
     (stroke (width 0) (type default))
   )
+  (bus_entry (at 62.23 111.76) (size 2.54 2.54)
+    (stroke (width 0) (type default))
+  )
   (bus_entry (at 62.23 109.22) (size 2.54 2.54)
     (stroke (width 0) (type default))
@@
     (stroke (width 0) (type default))
   )
+  (bus_entry (at 62.23 114.3) (size 2.54 2.54)
+    (stroke (width 0) (type default))
+  )
   (bus_entry (at 58.42 36.83) (size 2.54 2.54)
     (stroke (width 0) (type default))
@@
     (stroke (width 0) (type default))
   )
+  (bus (pts (xy 62.23 111.76) (xy 62.23 114.3))
+    (stroke (width 0) (type default))
+  )
   (wire (pts (xy 199.39 26.67) (xy 189.23 26.67))
     (stroke (width 0) (type default))
@@
     (stroke (width 0) (type default))
   )
+  (wire (pts (xy 64.77 116.84) (xy 68.58 116.84))
+    (stroke (width 0) (type default))
+  )
   (bus (pts (xy 58.42 44.45) (xy 58.42 46.99))
     (stroke (width 0) (type default))
@@
     (stroke (width 0) (type default))
   )
+  (bus (pts (xy 62.23 109.22) (xy 62.23 111.76))
+    (stroke (width 0) (type default))
+  )
   (wire (pts (xy 185.42 64.77) (xy 179.07 64.77))
     (stroke (width 0) (type default))
@@
     (stroke (width 0) (type default))
   )
+  (wire (pts (xy 64.77 114.3) (xy 68.58 114.3))
+    (stroke (width 0) (type default))
+  )
   (bus (pts (xy 231.14 92.71) (xy 231.14 115.57))
     (stroke (width 0) (type default))
@@
     (effects (font (size 1.27 1.27)) (justify left bottom))
   )
+  (label "FLASH.IO3" (at 68.58 116.84 0) (fields_autoplaced)
+    (effects (font (size 1.27 1.27)) (justify left bottom))
+  )
   (label "DVI.CK+" (at 223.52 96.52 180) (fields_autoplaced)
     (effects (font (size 1.27 1.27)) (justify right bottom))
@@
     (effects (font (size 1.27 1.27)) (justify left bottom))
   )
+  (label "FLASH.IO2" (at 179.07 77.47 0) (fields_autoplaced)
+    (effects (font (size 1.27 1.27)) (justify left bottom))
+  )
   (label "VGA.R0" (at 226.06 118.11 180) (fields_autoplaced)
     (effects (font (size 1.27 1.27)) (justify right bottom))
@@
     (effects (font (size 1.27 1.27)) (justify left bottom))
   )
+  (label "FLASH.IO3" (at 179.07 80.01 0) (fields_autoplaced)
+    (effects (font (size 1.27 1.27)) (justify left bottom))
+  )
   (label "DVI.D2+" (at 223.52 111.76 180) (fields_autoplaced)
     (effects (font (size 1.27 1.27)) (justify right bottom))
@@
   (label "VGA.B1" (at 226.06 135.89 180) (fields_autoplaced)
     (effects (font (size 1.27 1.27)) (justify right bottom))
+  )
+  (label "FLASH.IO2" (at 68.58 114.3 0) (fields_autoplaced)
+    (effects (font (size 1.27 1.27)) (justify left bottom))
   )
   (label "OUT_BUS.D2" (at 63.5 44.45 0) (fields_autoplaced)
@@
       (effects (font (size 1.27 1.27)) (justify left top))
     )
-    (pin "FLASH{CS# CLK IO[0..1]}" bidirectional (at 57.15 101.6 0)
+    (pin "FLASH{CS# CLK IO[0..3]}" bidirectional (at 57.15 101.6 0)
       (effects (font (size 1.27 1.27)) (justify right))
     )

Commit message: prepared first versions of PCBs
Parts:
- removed C207: 100n, Capacitor_SMD:C_0402_1005Metric_Pad0.74x0.62mm_HandSolder, symbol Device:C
- removed C214: 1u, Capacitor_SMD:C_0402_1005Metric_Pad0.74x0.62mm_HandSolder, symbol Device:C
- removed U4: RP2040, footprints:QFN40P700X700X90-57N, symbol RP2040:RP2040
- added C2, C4, C7: 4.7u, Capacitor_SMD:C_0402_1005Metric_Pad0.74x0.62mm_HandSolder, symbol Device:C
- added L1: 3.3u, Inductor_SMD:L_0805_2012Metric_Pad1.15x1.40mm_HandSolder, symbol Device:L
- added R30: 33, Resistor_SMD:R_0402_1005Metric_Pad0.72x0.64mm_HandSolder, symbol Device:R
- added U2: RP2350_60QFN, RP2350_60QFN_minimal:RP2350-QFN-60-1EP_7x7_P0.4mm_EP3.4x3.4mm_ThermalVias, symbol MCU_RaspberryPi_RP2350:RP2350_60QFN
- C6: renamed from C208; value 1u -> 4.7u
- renumbered C205 to C10, C202 to C11, C209 to C12, C210 to C13, C211 to C14, C212 to C15, C213 to C16, C204 to C3, C206 to C5, C201 to C8, C203 to C9, J201 to J4, R201 to R31, Y201 to Y1
Connections:
- net +1V1: now also C4.1, L1.1, U2.23 (DVDD), U2.39 (DVDD), U2.50 (VREG_FB), U2.6 (DVDD)
- net +3V3: now also C2.1, R30.1, U2.1 (IOVDD), U2.11 (IOVDD), U2.20 (IOVDD), U2.30 (IOVDD), U2.38 (IOVDD), U2.44 (ADC_AVDD), U2.45 (IOVDD), U2.49 (VREG_VIN), U2.53 (USB_OTP_VDD), U2.54 (QSPI_IOVDD)
- net DEBUG.SWCLK: now also U2.24 (SWCLK)
- net DEBUG.SWD: now also U2.25 (SWD)
- net DVI.CK+: now also U2.29 (GPIO18)
- net DVI.CK-: now also U2.31 (GPIO19)
- net DVI.D0+: now also U2.16 (GPIO12)
- net DVI.D0-: now also U2.17 (GPIO13)
- net DVI.D1+: now also U2.18 (GPIO14)
- net DVI.D1-: now also U2.19 (GPIO15)
- net DVI.D2+: now also U2.27 (GPIO16)
- net DVI.D2-: now also U2.28 (GPIO17)
- net GND: now also C2.2, C4.2, C7.2, U2.47 (VREG_PGND), U2.61 (GND)
- net MCU_I2C.CLOCK: now also U2.15 (GPIO11)
- net MCU_I2C.DATA: now also U2.14 (GPIO10)
- net OSC_IN: now also U2.21 (XIN)
- net OSC_OUT: now also U2.22 (XOUT)
- net VGA.B0: now also U2.35 (GPIO23)
- net VGA.B1: now also U2.34 (GPIO22)
- net VGA.G0: now also U2.40 (GPIO26_ADC0)
- net VGA.G1: now also U2.37 (GPIO25)
- net VGA.G2: now also U2.36 (GPIO24)
- net VGA.HSYNC: now also U2.32 (GPIO20)
- net VGA.R0: now also U2.43 (GPIO29_ADC3)
- net VGA.R1: now also U2.42 (GPIO28_ADC2)
- net VGA.R2: now also U2.41 (GPIO27_ADC1)
- net VGA.VSYNC: now also U2.33 (GPIO21)
- new net BUS.CLK: U2.13 (GPIO9)
- new net BUS.CS#: U2.12 (GPIO8)
- new net BUS.D0: U2.2 (GPIO0)
- new net BUS.D1: U2.3 (GPIO1)
- new net BUS.D2: U2.4 (GPIO2)
- new net BUS.D3: U2.5 (GPIO3)
- new net BUS.D4: U2.7 (GPIO4)
- new net BUS.D5: U2.8 (GPIO5)
- new net BUS.D6: U2.9 (GPIO6)
- new net BUS.D7: U2.10 (GPIO7)
- new net BUS.RE#: U2.26 (RUN)
- new net QSPI.CLK: U2.56 (QSPI_SCLK)
- new net QSPI.CS#: U2.60 (QSPI_SS)
- new net QSPI.IO0: U2.57 (QSPI_SD0)
- new net QSPI.IO1: U2.59 (QSPI_SD1)
- new net QSPI.IO2: U2.58 (QSPI_SD2)
- new net QSPI.IO3: U2.55 (QSPI_SD3)
- new net VREG_AVDD: C7.1, R30.2, U2.46 (VREG_AVDD)
- new net VREG_LX: L1.2, U2.48 (VREG_LX)
- no-connect marks 3 -> 2
Other:
- removed sheet Render Engine
- added sheet BUS connector (bus_connector.kicad_sch)
- sheet Memory ports: added QSPI{CS# CLK IO[0..3]}; removed FLASH{CS# CLK IO[0..3]}
- moved on the sheet: C10, C12, C13, C14, C15, C16, C9, J4
