File: gpu_extension/memory_render_engine.kicad_sch (KiCad schematic)
At the start: 9 parts, among them U402 W25Q128JVS, U5 APS6408L-3OBM-BA

Commit message: version 1.0
Parts:
- removed C405 (x3): 100n, Capacitor_SMD:C_0402_1005Metric_Pad0.74x0.62mm_HandSolder, symbol Device:C
- removed C406: 1u, Capacitor_SMD:C_0402_1005Metric_Pad0.74x0.62mm_HandSolder, symbol Device:C
- removed U5: APS6408L-3OBM-BA, BGA24C100P5X5_600X800X120, symbol APS6408L-3OBM-BA:APS6408L-3OBM-BA
- added C405: 100n, Capacitor_SMD:C_0402_1005Metric_Pad0.74x0.62mm_HandSolder, symbol Device:C
- added U2: IPS1604, Package_SO:SOP-8_3.9x4.9mm_P1.27mm, symbol ips1604:IPS1604
- C402: footprint Capacitor_SMD:C_0603_1608Metric_Pad1.08x0.95mm_HandSolder -> Capacitor_SMD:C_0402_1005Metric_Pad0.74x0.62mm_HandSolder
- R402: footprint Resistor_SMD:R_0603_1608Metric_Pad0.98x0.95mm_HandSolder -> Resistor_SMD:R_0402_1005Metric_Pad0.72x0.64mm_HandSolder
Connections:
- net +3V3: now also C405.1, U2.8 (VDD)
- net GND: now also C405.2, U2.4 (VSS)
- net PSRAM.CE#: now also U2.1 (CE#)
- net PSRAM.CLK: now also U2.6 (SCLK)
- net PSRAM.IO0: now also U2.5 (SI/SIO0)
- net PSRAM.IO1: now also U2.2 (SO/SIO1)
- net PSRAM.IO2: now also U2.3 (SIO2)
- net PSRAM.IO3: now also U2.7 (SIO3)
- no-connect marks 2 -> 0

Commit message: prepared first versions of PCBs
Parts:
- renumbered C402 to C403, C405 to C409, R402 to R403, R404 to R405, U402 to U403
