File: gpu_extension/render.kicad_sch (KiCad schematic)
At the start: 18 parts, among them J201 Conn_01x03_Male, U4 RP2040, Y201 ECS-120-8-36-CGN-TR

Commit message: version 1.0
Connections:
- net PSRAM.IO4 is gone; now on net PSRAM.CLK: U4.6 (GPIO4)
- net PSRAM.IO5 is gone; now on net PSRAM.CE#: U4.7 (GPIO5)
- net PSRAM.CE#: no longer U4.13 (GPIO10)
- net PSRAM.CLK: no longer U4.12 (GPIO9)
- net PSRAM.IO6: no longer names the net of U4.8 (GPIO6)
- net PSRAM.IO7: no longer names the net of U4.9 (GPIO7)
- net PSRAM.RWDS: no longer names the net of U4.11 (GPIO8)
- no-connect marks 2 -> 7
Other:
- sheet Memory Render Engine ports: added PSRAM{CE# CLK IO[0..3] RWDS}; removed PSRAM{CE# CLK IO[0..7] RWDS}

Commit message: prepared first versions of PCBs
Parts:
- renumbered C204 to C215, C206 to C216, C208 to C217, C201 to C218, C207 to C219, C203 to C220, C205 to C221, C209 to C222, C202 to C223, C210 to C224, C211 to C225, C212 to C226, C213 to C227, C214 to C228, J201 to J202, R201 to R202, U4 to U6, Y201 to Y202
Other:
- removed sheet BUS connector
