File: gpu_vga_extension/RP2040.kicad_sch (KiCad schematic)
At the start: 18 parts, among them J201 Conn_01x03_Male, U4 RP2040, Y201 ECS-120-8-36-CGN-TR

Commit message: Rename KiCad files and sheets to match what they contain
- mainboard: rp2040_core.kicad_sch -> rp2350_core.kicad_sch and the
  sheet "RP2040 Core" -> "RP2350 Core"; the sheet holds the RP2350.
  Hierarchical net names, footprint sheet properties and the net-class
  patterns in the .kicad_pro follow the new sheet name.
- gpu_vga_extension, gpu_dvi_card: both projects were still called
  gpu_extension; name each after its directory, including the
  (project ...) instance blocks in every sheet.
- gpu_vga_extension: dvi.kicad_sch -> vga.kicad_sch and the sheet
  "DVI connector" -> "VGA connector"; it holds the VGA connector and DAC.
- bus_adapter_20pin: the project inside was bus_adapter_10pin; rename
  the directory and files to bus_adapter_20pin.

kicad-cli ERC and DRC with schematic parity give the same entries before
and after (names aside) for all four projects. Existing gerbers keep
their old file names until the boards are plotted again.

Co-Authored-By: Claude Opus 5 (1M context) <noreply@anthropic.com>
Other:
- sheet DVI connector renamed VGA connector
- sheet VGA connector: file dvi.kicad_sch -> vga.kicad_sch
Changed lines of the file:
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@@
     (pin "2")
     (instances
-      (project "gpu_extension"
+      (project "gpu_vga_extension"
         (path "/125be418-c5a0-4917-8634-47021fa57275/f0969bf3-d19a-4dd7-b14e-11dc331478c5"
           (reference "C212") (unit 1)
@@
     (pin "2")
     (instances
-      (project "gpu_extension"
+      (project "gpu_vga_extension"
         (path "/125be418-c5a0-4917-8634-47021fa57275/f0969bf3-d19a-4dd7-b14e-11dc331478c5"
           (reference "C202") (unit 1)
@@
     (pin "9")
     (instances
-      (project "gpu_extension"
+      (project "gpu_vga_extension"
         (path "/125be418-c5a0-4917-8634-47021fa57275/f0969bf3-d19a-4dd7-b14e-11dc331478c5"
           (reference "U4") (unit 1)
@@
     (pin "1")
     (instances
-      (project "gpu_extension"
+      (project "gpu_vga_extension"
         (path "/125be418-c5a0-4917-8634-47021fa57275/f0969bf3-d19a-4dd7-b14e-11dc331478c5"
           (reference "#PWR0140") (unit 1)
@@
     (pin "2")
     (instances
-      (project "gpu_extension"
+      (project "gpu_vga_extension"
         (path "/125be418-c5a0-4917-8634-47021fa57275/f0969bf3-d19a-4dd7-b14e-11dc331478c5"
           (reference "C210") (unit 1)
@@
     (pin "2")
     (instances
-      (project "gpu_extension"
+      (project "gpu_vga_extension"
         (path "/125be418-c5a0-4917-8634-47021fa57275/f0969bf3-d19a-4dd7-b14e-11dc331478c5"
           (reference "C211") (unit 1)
@@
     (pin "1")
     (instances
-      (project "gpu_extension"
+      (project "gpu_vga_extension"
         (path "/125be418-c5a0-4917-8634-47021fa57275/f0969bf3-d19a-4dd7-b14e-11dc331478c5"
           (reference "#PWR0115") (unit 1)
@@
     (pin "1")
     (instances
-      (project "gpu_extension"
+      (project "gpu_vga_extension"
         (path "/125be418-c5a0-4917-8634-47021fa57275/f0969bf3-d19a-4dd7-b14e-11dc331478c5"
           (reference "#PWR0105") (unit 1)
@@
     (pin "2")
     (instances
-      (project "gpu_extension"
+      (project "gpu_vga_extension"
         (path "/125be418-c5a0-4917-8634-47021fa57275/f0969bf3-d19a-4dd7-b14e-11dc331478c5"
           (reference "C204") (unit 1)
@@
     (pin "1")
     (instances
-      (project "gpu_extension"
+      (project "gpu_vga_extension"
         (path "/125be418-c5a0-4917-8634-47021fa57275/f0969bf3-d19a-4dd7-b14e-11dc331478c5"
           (reference "#PWR0101") (unit 1)
@@
     (pin "2")
     (instances
-      (project "gpu_extension"
+      (project "gpu_vga_extension"
         (path "/125be418-c5a0-4917-8634-47021fa57275/f0969bf3-d19a-4dd7-b14e-11dc331478c5"
           (reference "C208") (unit 1)
@@
     (pin "2")
     (instances
-      (project "gpu_extension"
+      (project "gpu_vga_extension"
         (path "/125be418-c5a0-4917-8634-47021fa57275/f0969bf3-d19a-4dd7-b14e-11dc331478c5"
           (reference "C207") (unit 1)
@@
     (pin "1")
     (instances
-      (project "gpu_extension"
+      (project "gpu_vga_extension"
         (path "/125be418-c5a0-4917-8634-47021fa57275/f0969bf3-d19a-4dd7-b14e-11dc331478c5"
           (reference "#PWR0104") (unit 1)
@@
     (pin "1")
     (instances
-      (project "gpu_extension"
+      (project "gpu_vga_extension"
         (path "/125be418-c5a0-4917-8634-47021fa57275/f0969bf3-d19a-4dd7-b14e-11dc331478c5"
           (reference "#PWR0106") (unit 1)
@@
     (pin "2")
     (instances
-      (project "gpu_extension"
+      (project "gpu_vga_extension"
         (path "/125be418-c5a0-4917-8634-47021fa57275/f0969bf3-d19a-4dd7-b14e-11dc331478c5"
           (reference "C205") (unit 1)
@@
     (pin "4")
     (instances
-      (project "gpu_extension"
+      (project "gpu_vga_extension"
         (path "/125be418-c5a0-4917-8634-47021fa57275/f0969bf3-d19a-4dd7-b14e-11dc331478c5"
           (reference "Y201") (unit 1)
@@
     (pin "2")
     (instances
-      (project "gpu_extension"
+      (project "gpu_vga_extension"
         (path "/125be418-c5a0-4917-8634-47021fa57275/f0969bf3-d19a-4dd7-b14e-11dc331478c5"
           (reference "C213") (unit 1)
@@
     (pin "1")
     (instances
-      (project "gpu_extension"
+      (project "gpu_vga_extension"
         (path "/125be418-c5a0-4917-8634-47021fa57275/f0969bf3-d19a-4dd7-b14e-11dc331478c5"
           (reference "#PWR0110") (unit 1)
@@
     (pin "2")
     (instances
-      (project "gpu_extension"
+      (project "gpu_vga_extension"
         (path "/125be418-c5a0-4917-8634-47021fa57275/f0969bf3-d19a-4dd7-b14e-11dc331478c5"
           (reference "C201") (unit 1)
@@
     (pin "1")
     (instances
-      (project "gpu_extension"
+      (project "gpu_vga_extension"
         (path "/125be418-c5a0-4917-8634-47021fa57275/f0969bf3-d19a-4dd7-b14e-11dc331478c5"
           (reference "#PWR0141") (unit 1)
@@
     (pin "1")
     (instances
-      (project "gpu_extension"
+      (project "gpu_vga_extension"
         (path "/125be418-c5a0-4917-8634-47021fa57275/f0969bf3-d19a-4dd7-b14e-11dc331478c5"
           (reference "#PWR0107") (unit 1)
@@
     (pin "2")
     (instances
-      (project "gpu_extension"
+      (project "gpu_vga_extension"
         (path "/125be418-c5a0-4917-8634-47021fa57275/f0969bf3-d19a-4dd7-b14e-11dc331478c5"
           (reference "C209") (unit 1)
@@
     (pin "1")
     (instances
-      (project "gpu_extension"
+      (project "gpu_vga_extension"
         (path "/125be418-c5a0-4917-8634-47021fa57275/f0969bf3-d19a-4dd7-b14e-11dc331478c5"
           (reference "#PWR0109") (unit 1)
@@
     (pin "1")
     (instances
-      (project "gpu_extension"
+      (project "gpu_vga_extension"
         (path "/125be418-c5a0-4917-8634-47021fa57275/f0969bf3-d19a-4dd7-b14e-11dc331478c5"
           (reference "#PWR0102") (unit 1)
@@
     (pin "2")
     (instances
-      (project "gpu_extension"
+      (project "gpu_vga_extension"
         (path "/125be418-c5a0-4917-8634-47021fa57275/f0969bf3-d19a-4dd7-b14e-11dc331478c5"
           (reference "C214") (unit 1)
@@
     (pin "2")
     (instances
-      (project "gpu_extension"
+      (project "gpu_vga_extension"
         (path "/125be418-c5a0-4917-8634-47021fa57275/f0969bf3-d19a-4dd7-b14e-11dc331478c5"
           (reference "C206") (unit 1)
@@
     (pin "1")
     (instances
-      (project "gpu_extension"
+      (project "gpu_vga_extension"
         (path "/125be418-c5a0-4917-8634-47021fa57275/f0969bf3-d19a-4dd7-b14e-11dc331478c5"
           (reference "#PWR0142") (unit 1)
@@
     (pin "1")
     (instances
-      (project "gpu_extension"
+      (project "gpu_vga_extension"
         (path "/125be418-c5a0-4917-8634-47021fa57275/f0969bf3-d19a-4dd7-b14e-11dc331478c5"
           (reference "#FLG0102") (unit 1)
@@
     (pin "1")
     (instances
-      (project "gpu_extension"
+      (project "gpu_vga_extension"
         (path "/125be418-c5a0-4917-8634-47021fa57275/f0969bf3-d19a-4dd7-b14e-11dc331478c5"
           (reference "#PWR0103") (unit 1)
@@
     (pin "2")
     (instances
-      (project "gpu_extension"
+      (project "gpu_vga_extension"
         (path "/125be418-c5a0-4917-8634-47021fa57275/f0969bf3-d19a-4dd7-b14e-11dc331478c5"
           (reference "R201") (unit 1)
@@
     (pin "1")
     (instances
-      (project "gpu_extension"
+      (project "gpu_vga_extension"
         (path "/125be418-c5a0-4917-8634-47021fa57275/f0969bf3-d19a-4dd7-b14e-11dc331478c5"
           (reference "#FLG0104") (unit 1)
@@
     (pin "3")
     (instances
-      (project "gpu_extension"
+      (project "gpu_vga_extension"
         (path "/125be418-c5a0-4917-8634-47021fa57275/f0969bf3-d19a-4dd7-b14e-11dc331478c5"
           (reference "J201") (unit 1)
@@
     (pin "2")
     (instances
-      (project "gpu_extension"
+      (project "gpu_vga_extension"
         (path "/125be418-c5a0-4917-8634-47021fa57275/f0969bf3-d19a-4dd7-b14e-11dc331478c5"
           (reference "C203") (unit 1)
@@
     (pin "1")
     (instances
-      (project "gpu_extension"
+      (project "gpu_vga_extension"
         (path "/125be418-c5a0-4917-8634-47021fa57275/f0969bf3-d19a-4dd7-b14e-11dc331478c5"
           (reference "#PWR0108") (unit 1)
@@
     )
     (instances
-      (project "gpu_extension"
+      (project "gpu_vga_extension"
         (path "/125be418-c5a0-4917-8634-47021fa57275/f0969bf3-d19a-4dd7-b14e-11dc331478c5" (page ""))
       )
@@
     )
     (instances
-      (project "gpu_extension"
+      (project "gpu_vga_extension"
         (path "/125be418-c5a0-4917-8634-47021fa57275/f0969bf3-d19a-4dd7-b14e-11dc331478c5" (page ""))
       )
@@
     (stroke (width 0.1524) (type solid))
     (fill (color 0 0 0 0.0000))
-    (property "Sheetname" "DVI connector" (at 213.36 95.8084 0)
+    (property "Sheetname" "VGA connector" (at 213.36 95.8084 0)
       (effects (font (size 1.27 1.27)) (justify left bottom))
     )
-    (property "Sheetfile" "dvi.kicad_sch" (at 213.36 107.2646 0)
+    (property "Sheetfile" "vga.kicad_sch" (at 213.36 107.2646 0)
       (effects (font (size 1.27 1.27)) (justify left top))
     )
@@
     )
     (instances
-      (project "gpu_extension"
+      (project "gpu_vga_extension"
         (path "/125be418-c5a0-4917-8634-47021fa57275/f0969bf3-d19a-4dd7-b14e-11dc331478c5" (page ""))
       )
