File: gpu_vga_extension/gpu_vga_extension.kicad_sch (KiCad schematic)
At the start: 22 parts, among them J1 Conn_01x03_Pin, J4 Conn_01x03_Male, U2 RP2350_60QFN, Y1 ECS-120-8-36-CGN-TR

Commit message: Rename KiCad files and sheets to match what they contain
- mainboard: rp2040_core.kicad_sch -> rp2350_core.kicad_sch and the
  sheet "RP2040 Core" -> "RP2350 Core"; the sheet holds the RP2350.
  Hierarchical net names, footprint sheet properties and the net-class
  patterns in the .kicad_pro follow the new sheet name.
- gpu_vga_extension, gpu_dvi_card: both projects were still called
  gpu_extension; name each after its directory, including the
  (project ...) instance blocks in every sheet.
- gpu_vga_extension: dvi.kicad_sch -> vga.kicad_sch and the sheet
  "DVI connector" -> "VGA connector"; it holds the VGA connector and DAC.
- bus_adapter_20pin: the project inside was bus_adapter_10pin; rename
  the directory and files to bus_adapter_20pin.

kicad-cli ERC and DRC with schematic parity give the same entries before
and after (names aside) for all four projects. Existing gerbers keep
their old file names until the boards are plotted again.

Co-Authored-By: Claude Opus 5 (1M context) <noreply@anthropic.com>
Other:
- sheet DVI connector renamed VGA connector
- sheet VGA connector: file dvi.kicad_sch -> vga.kicad_sch
Changed lines of the file:
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@@
 		)
 		(instances
-			(project "gpu_extension"
+			(project "gpu_vga_extension"
 				(path "/125be418-c5a0-4917-8634-47021fa57275"
 					(reference "C14")
@@
 		)
 		(instances
-			(project "gpu_extension"
+			(project "gpu_vga_extension"
 				(path "/125be418-c5a0-4917-8634-47021fa57275"
 					(reference "#FLG04")
@@
 		)
 		(instances
-			(project "gpu_extension"
+			(project "gpu_vga_extension"
 				(path "/125be418-c5a0-4917-8634-47021fa57275"
 					(reference "C8")
@@
 		)
 		(instances
-			(project "gpu_extension"
+			(project "gpu_vga_extension"
 				(path "/125be418-c5a0-4917-8634-47021fa57275"
 					(reference "C11")
@@
 		)
 		(instances
-			(project "gpu_extension"
+			(project "gpu_vga_extension"
 				(path "/125be418-c5a0-4917-8634-47021fa57275"
 					(reference "#PWR034")
@@
 		)
 		(instances
-			(project "gpu_extension"
+			(project "gpu_vga_extension"
 				(path "/125be418-c5a0-4917-8634-47021fa57275"
 					(reference "R31")
@@
 		)
 		(instances
-			(project "gpu_extension"
+			(project "gpu_vga_extension"
 				(path "/125be418-c5a0-4917-8634-47021fa57275"
 					(reference "J4")
@@
 		)
 		(instances
-			(project "gpu_extension"
+			(project "gpu_vga_extension"
 				(path "/125be418-c5a0-4917-8634-47021fa57275"
 					(reference "#PWR031")
@@
 		)
 		(instances
-			(project "gpu_extension"
+			(project "gpu_vga_extension"
 				(path "/125be418-c5a0-4917-8634-47021fa57275"
 					(reference "C9")
@@
 		)
 		(instances
-			(project "gpu_extension"
+			(project "gpu_vga_extension"
 				(path "/125be418-c5a0-4917-8634-47021fa57275"
 					(reference "C12")
@@
 		)
 		(instances
-			(project "gpu_extension"
+			(project "gpu_vga_extension"
 				(path "/125be418-c5a0-4917-8634-47021fa57275"
 					(reference "#PWR037")
@@
 		)
 		(instances
-			(project "gpu_extension"
+			(project "gpu_vga_extension"
 				(path "/125be418-c5a0-4917-8634-47021fa57275"
 					(reference "C4")
@@
 		)
 		(instances
-			(project "gpu_extension"
+			(project "gpu_vga_extension"
 				(path "/125be418-c5a0-4917-8634-47021fa57275"
 					(reference "Y1")
@@
 		)
 		(instances
-			(project "gpu_extension"
+			(project "gpu_vga_extension"
 				(path "/125be418-c5a0-4917-8634-47021fa57275"
 					(reference "C2")
@@
 		)
 		(instances
-			(project "gpu_extension"
+			(project "gpu_vga_extension"
 				(path "/125be418-c5a0-4917-8634-47021fa57275"
 					(reference "#PWR028")
@@
 		)
 		(instances
-			(project "gpu_extension"
+			(project "gpu_vga_extension"
 				(path "/125be418-c5a0-4917-8634-47021fa57275"
 					(reference "#PWR038")
@@
 		)
 		(instances
-			(project "gpu_extension"
+			(project "gpu_vga_extension"
 				(path "/125be418-c5a0-4917-8634-47021fa57275"
 					(reference "C6")
@@
 		)
 		(instances
-			(project "gpu_extension"
+			(project "gpu_vga_extension"
 				(path "/125be418-c5a0-4917-8634-47021fa57275"
 					(reference "C15")
@@
 		)
 		(instances
-			(project "gpu_extension"
+			(project "gpu_vga_extension"
 				(path "/125be418-c5a0-4917-8634-47021fa57275"
 					(reference "#PWR035")
@@
 		)
 		(instances
-			(project "gpu_extension"
+			(project "gpu_vga_extension"
 				(path "/125be418-c5a0-4917-8634-47021fa57275"
 					(reference "C10")
@@
 		)
 		(instances
-			(project "gpu_extension"
+			(project "gpu_vga_extension"
 				(path "/125be418-c5a0-4917-8634-47021fa57275"
 					(reference "#FLG05")
@@
 		)
 		(instances
-			(project "gpu_extension"
+			(project "gpu_vga_extension"
 				(path "/125be418-c5a0-4917-8634-47021fa57275"
 					(reference "C13")
@@
 		)
 		(instances
-			(project "gpu_extension"
+			(project "gpu_vga_extension"
 				(path "/125be418-c5a0-4917-8634-47021fa57275"
 					(reference "#PWR039")
@@
 		)
 		(instances
-			(project "gpu_extension"
+			(project "gpu_vga_extension"
 				(path "/125be418-c5a0-4917-8634-47021fa57275"
 					(reference "C16")
@@
 		)
 		(instances
-			(project "gpu_extension"
+			(project "gpu_vga_extension"
 				(path "/125be418-c5a0-4917-8634-47021fa57275"
 					(reference "C3")
@@
 		)
 		(instances
-			(project "gpu_extension"
+			(project "gpu_vga_extension"
 				(path "/125be418-c5a0-4917-8634-47021fa57275"
 					(reference "#PWR027")
@@
 		)
 		(instances
-			(project "gpu_extension"
+			(project "gpu_vga_extension"
 				(path "/125be418-c5a0-4917-8634-47021fa57275"
 					(reference "#PWR029")
@@
 		)
 		(instances
-			(project "gpu_extension"
+			(project "gpu_vga_extension"
 				(path "/125be418-c5a0-4917-8634-47021fa57275"
 					(reference "C5")
@@
 			(color 0 0 0 0.0000)
 		)
-		(property "Sheetname" "DVI connector"
+		(property "Sheetname" "VGA connector"
 			(at 55.88 93.2684 0)
 			(effects
@@
 			)
 		)
-		(property "Sheetfile" "dvi.kicad_sch"
+		(property "Sheetfile" "vga.kicad_sch"
 			(at 55.88 111.0746 0)
 			(effects
@@
 		)
 		(instances
-			(project "gpu_extension"
+			(project "gpu_vga_extension"
 				(path "/125be418-c5a0-4917-8634-47021fa57275"
 					(page "1")
@@
 		)
 		(instances
-			(project "gpu_extension"
+			(project "gpu_vga_extension"
 				(path "/125be418-c5a0-4917-8634-47021fa57275"
 					(page "3")
@@
 		)
 		(instances
-			(project "gpu_extension"
+			(project "gpu_vga_extension"
 				(path "/125be418-c5a0-4917-8634-47021fa57275"
 					(page "2")
